File: hardware/tscircuit/c5-buses.kicad_pcb (KiCad board)
At the start: 2 copper layers, 120 x 90 mm, 10 parts

Commit message: hw(rf,c5-buses): resolve SP4T sourcing — SKY13414 (in stock) + RFSW_C
PE42440 isn't stocked at JLCPCB; swapped to the in-stock SKY13414-485LF (C255353),
engine-pulled footprint. It uses 3-line control (V1/V2/V3 = RFSW_A/RFSW_B/RFSW_C);
added RFSW_C on PCA9555 #2 P07 (c5-buses). Switch common -> CC1101 radio, RF1..RF4 ->
per-band matches -> shared antenna; EP + unused pads grounded. Both sheets KiCad DRC
0 unconnected / 0 shorts / 0 parity. Docs (rf EN+RU) updated.

Co-Authored-By: Claude Opus 4.8 <noreply@anthropic.com>
Connections:
- U13 pad 11: (no net) -> RFSW_C
Changed lines of the file:
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@@
   (net 69 "JACK_DET")
   (net 70 "RFSW_B")
-  (net 71 "HC138_A")
-  (net 72 "HC138_B")
+  (net 71 "RFSW_C")
+  (net 72 "HC138_A")
+  (net 73 "HC138_B")
   (footprint
     "tscircuit:chip"
@@
       (size 1.499997 0.8999982)
       (layers F.Cu F.Paste F.Mask)
-      (net 71 "HC138_A")
+      (net 72 "HC138_A")
     )
     (pad "13" smd rect
@@
       (size 0.8999982 1.499997)
       (layers F.Cu F.Paste F.Mask)
-      (net 72 "HC138_B")
+      (net 73 "HC138_B")
     )
     (pad "18" smd rect
@@
       (layers F.Cu F.Paste F.Mask)
       (roundrect_rratio 0.5)
-      (net 71 "HC138_A")
+      (net 72 "HC138_A")
     )
     (pad "2" smd roundrect
@@
       (layers F.Cu F.Paste F.Mask)
       (roundrect_rratio 0.5)
-      (net 72 "HC138_B")
+      (net 73 "HC138_B")
     )
     (pad "3" smd roundrect
@@
       (size 1.6500093999999998 0.39999919999999994)
       (layers F.Cu F.Paste F.Mask)
+      (net 71 "RFSW_C")
     )
     (pad "10" smd rect
@@
     (width 0.15)
     (layer F.Cu)
-    (net 72)
+    (net 73)
   )
   (segment
@@
     (width 0.15)
     (layer F.Cu)
-    (net 72)
+    (net 73)
   )
   (segment
@@
     (width 0.15)
     (layer F.Cu)
-    (net 72)
+    (net 73)
   )
   (segment
@@
     (width 0.15)
     (layer F.Cu)
-    (net 72)
+    (net 73)
   )
   (segment
@@
     (width 0.15)
     (layer F.Cu)
-    (net 72)
+    (net 73)
   )
   (segment
@@
     (width 0.15)
     (layer F.Cu)
-    (net 72)
+    (net 73)
   )
   (segment
@@
     (width 0.15)
     (layer F.Cu)
-    (net 72)
+    (net 73)
   )
   (segment
@@
     (width 0.15)
     (layer F.Cu)
-    (net 72)
+    (net 73)
   )
   (segment
@@
     (width 0.15)
     (layer F.Cu)
-    (net 72)
+    (net 73)
   )
   (segment
@@
     (width 0.15)
     (layer F.Cu)
-    (net 72)
+    (net 73)
   )
   (segment
@@
     (width 0.15)
     (layer F.Cu)
-    (net 72)
+    (net 73)
   )
   (segment
@@
     (width 0.15)
     (layer F.Cu)
-    (net 71)
+    (net 72)
   )
   (segment
@@
     (width 0.15)
     (layer F.Cu)
-    (net 71)
+    (net 72)
   )
   (segment
