File: hardware/tscircuit/audio.kicad_pcb (KiCad board)
At the start: 2 copper layers, 80 x 60 mm, 24 parts

Commit message: review onboard audio path options
Parts:
- added Cd33: 100nF, tscircuit:capacitor_cap0402, F.Cu at (78.1, 93.4)
- added Rpu_jack: 10kΩ, tscircuit:resistor_res0402, F.Cu at (103.5, 86.8)
- moved RsumR 11.8 mm to (107.3, 86.8)
- moved RsumL 2.25 mm to (100.7, 86.8)
- moved LS1 0.28 mm to (122.7, 84.0)
Connections:
- RsumL pad 1: .U30 > .pin2 to .RsumL > .pin1 -> .U30 > .pin1 to .RsumL > .pin1
- RsumR pad 1: .U30 > .pin1 to .RsumR > .pin1 -> .U30 > .pin16 to .RsumR > .pin1
- U30 pad 1: .U30 > .pin1 to .RsumR > .pin1 -> .U30 > .pin1 to .RsumL > .pin1
- U30 pad 16: (no net) -> .U30 > .pin16 to .RsumR > .pin1
- U30 pad 2: .U30 > .pin2 to .RsumL > .pin1 -> (no net)
Routing:
- net .U30 > .pin1 to .RsumL > .pin1: track 0.00 -> 35.6 mm, vias 0 -> 2
- net V3V3: track 0.00 -> 33.2 mm, vias 0 -> 2
- net .U30 > .pin2 to .RsumL > .pin1: track 30.9 -> 0.00 mm, vias 2 -> 0
- net JACK_DET: track 0.00 -> 30.8 mm, vias 0 -> 2
- net .U30 > .pin16 to .RsumR > .pin1: track 0.00 -> 24.4 mm, vias 0 -> 2
- net .U30 > .pin1 to .RsumR > .pin1: track 20.5 -> 0.00 mm, vias 2 -> 0
- net SI_AUDIO: track 45.3 -> 35.9 mm, vias 4 -> 2
- net GND: track 115.8 -> 121.9 mm, vias 6 -> 8
- net V3V3A: track 15.3 -> 17.3 mm, vias 2 -> 0
- net SPK_M: track 24.6 -> 26.3 mm, vias 4 -> 2
- net V5: track 19.1 -> 20.1 mm
- net .U30 > .RCLK to .Y1 > .OSC1: track 25.3 -> 26.2 mm
- net .Cjk2 > .pin2 to .J30 > .R: track 6.11 -> 5.37 mm, vias 1 -> 0
- net .Cjk1 > .pin2 to .J30 > .L: track 7.46 -> 8.20 mm, vias 0 -> 1
- net .Cinp > .pin2 to .U32 > .IN_POS: track 27.3 -> 26.8 mm
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