File: hardware/ecad/kicad/L2-DISP-ADP-001-A/L2-DISP-ADP-001-A.kicad_sch (KiCad schematic)
At the start: 0 parts

Commit message: complete H2.4.1 display adapter schematic
Parts:
- added J1: Hirose DF40C-40DP-0.4V(51), Connector_Hirose_DF40:Hirose_DF40C-40DP-0.4V_2x20-1MP_P0.4mm, symbol Leshy2:ADP00_DISPLAY_ADAPTER_PLUG
- added J2: Hirose FH34SRJ-40S-0.5SH(99), Leshy2:FH34SRJ-40S-0.5SH-99, symbol Leshy2:ADP00_DISPLAY_PANEL_CONNECTOR
Connections:
- new net 3V3_MAIN: J1.39 (PIN_39), J1.6 (PIN_6), J1.7 (PIN_7), J2.39 (PIN_39), J2.6 (PIN_6), J2.7 (PIN_7)
- new net DISPLAY_SD_SPI_D0: J1.13 (PIN_13), J2.13 (PIN_13)
- new net DISPLAY_SD_SPI_D1: J1.10 (PIN_10), J2.10 (PIN_10)
- new net DISPLAY_SD_SPI_SCK: J1.11 (PIN_11), J2.11 (PIN_11)
- new net LCD_CS_N: J1.9 (PIN_9), J2.9 (PIN_9)
- new net LCD_LEDA_PROTECTED: J1.33 (PIN_33), J2.33 (PIN_33)
- new net LCD_LEDK: J1.34 (PIN_34), J1.35 (PIN_35), J1.36 (PIN_36), J2.34 (PIN_34), J2.35 (PIN_35), J2.36 (PIN_36)
- new net LCD_NC_14: J1.14 (PIN_14), J2.14 (PIN_14)
- new net LCD_NC_25: J1.25 (PIN_25), J2.25 (PIN_25)
- new net LCD_NC_26: J1.26 (PIN_26), J2.26 (PIN_26)
- new net LCD_NC_27: J1.27 (PIN_27), J2.27 (PIN_27)
- new net LCD_NC_28: J1.28 (PIN_28), J2.28 (PIN_28)
- new net LCD_NC_29: J1.29 (PIN_29), J2.29 (PIN_29)
- new net LCD_NC_30: J1.30 (PIN_30), J2.30 (PIN_30)
- new net LCD_NC_31: J1.31 (PIN_31), J2.31 (PIN_31)
- new net LCD_NC_32: J1.32 (PIN_32), J2.32 (PIN_32)
- new net LCD_QSPI_D2: J1.17 (PIN_17), J2.17 (PIN_17)
- new net LCD_QSPI_D3: J1.18 (PIN_18), J2.18 (PIN_18)
- new net LCD_RD_NC: J1.12 (PIN_12), J2.12 (PIN_12)
- new net LCD_RST_N: J1.15 (PIN_15), J2.15 (PIN_15)
- new net LCD_TE_NC: J1.8 (PIN_8), J2.8 (PIN_8)
- new net LCD_TOUCH_INT_RAW_N: J1.3 (PIN_3), J2.3 (PIN_3)
- new net POWER_GROUND: J1.16 (PIN_16), J1.19 (PIN_19), J1.20 (PIN_20), J1.21 (PIN_21), J1.22 (PIN_22), J1.23 (PIN_23), J1.24 (PIN_24), J1.37 (PIN_37), J1.38 (PIN_38), J1.40 (PIN_40), J1.5 (PIN_5), J2.16 (PIN_16), J2.19 (PIN_19), J2.20 (PIN_20), J2.21 (PIN_21), J2.22 (PIN_22), J2.23 (PIN_23), J2.24 (PIN_24), J2.37 (PIN_37), J2.38 (PIN_38), J2.40 (PIN_40), J2.5 (PIN_5)
- new net SYS_I2C_SCL: J1.1 (PIN_1), J2.1 (PIN_1)
- new net SYS_I2C_SDA: J1.2 (PIN_2), J2.2 (PIN_2)
- new net TOUCH_RST_N: J1.4 (PIN_4), J2.4 (PIN_4)
- no-connect marks 0 -> 2
Other:
- title: (none) -> Leshy2 — passive 40-contact display adapter
