File: hardware/ecad/kicad/LESHY2-LORA-CAP-01/LESHY2-LORA-CAP-01.kicad_sch (KiCad schematic)
At the start: 0 parts

Commit message: complete H2.4.2 LoRa Cap root
Parts:
- added J1: Samtec TSW-107-07-G-D, Connector_PinHeader_2.54mm:PinHeader_2x07_P2.54mm_Vertical, symbol Leshy2:CAP00_CAP_HEADER
Connections:
- new net CAP_10_RADIO_CONTROL/GND: J1.6 (PIN_6)
- new net CAP_10_RADIO_CONTROL/LORA_BUSY: J1.10 (PIN_10)
- new net CAP_10_RADIO_CONTROL/LORA_DIO1: J1.9 (PIN_9)
- new net CAP_10_RADIO_CONTROL/LORA_MISO: J1.13 (PIN_13)
- new net CAP_10_RADIO_CONTROL/LORA_MOSI: J1.12 (PIN_12)
- new net CAP_10_RADIO_CONTROL/LORA_NRESET: J1.8 (PIN_8)
- new net CAP_10_RADIO_CONTROL/LORA_NSS: J1.14 (PIN_14)
- new net CAP_10_RADIO_CONTROL/LORA_SCK: J1.11 (PIN_11)
- new net CAP_20_POWER_BUS/5V_IN: J1.7 (PIN_7)
- new net CAP_20_POWER_BUS/IDENTITY_SCL: J1.3 (PIN_3)
- new net CAP_20_POWER_BUS/IDENTITY_SDA: J1.4 (PIN_4)
- new net CAP_30_TX_EVIDENCE/EXT_TX_EVIDENCE_N: J1.5 (PIN_5)
- no-connect marks 0 -> 2
Other:
- added sheet CAP_10_RADIO_CONTROL (CAP_10_RADIO_CONTROL.kicad_sch)
- added sheet CAP_20_POWER_BUS (CAP_20_POWER_BUS.kicad_sch)
- added sheet CAP_30_TX_EVIDENCE (CAP_30_TX_EVIDENCE.kicad_sch)
- title: (none) -> Leshy2 — optional LoRa Cap and exact 14-contact host boundary
