File: hardware/ecad/kicad/LESHY2-LORA-CAP-01/CAP_30_TX_EVIDENCE.kicad_sch (KiCad schematic)
At the start: 0 parts

Commit message: complete H2.4.2 LoRa Cap root
Connections:
- no-connect marks 0 -> 4
Changed lines of the file:
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@@
 	(generator_version "10.0")
 	(paper "A4")
+	(hierarchical_label "CAP_3V3"
+		(shape bidirectional)
+		(at 20.32 20.32 0)
+		(effects (font (size 1.27 1.27)))
+	)
+	(wire
+		(pts (xy 20.32 20.32) (xy 25.40 20.32))
+		(stroke (width 0) (type default))
+	)
+	(no_connect (at 25.40 20.32)
+	)
+	(hierarchical_label "GND"
+		(shape bidirectional)
+		(at 20.32 25.40 0)
+		(effects (font (size 1.27 1.27)))
+	)
+	(wire
+		(pts (xy 20.32 25.40) (xy 25.40 25.40))
+		(stroke (width 0) (type default))
+	)
+	(no_connect (at 25.40 25.40)
+	)
+	(hierarchical_label "RF_FORWARD_LEVEL"
+		(shape bidirectional)
+		(at 190.50 20.32 180)
+		(effects (font (size 1.27 1.27)) (justify right))
+	)
+	(wire
+		(pts (xy 190.50 20.32) (xy 185.42 20.32))
+		(stroke (width 0) (type default))
+	)
+	(no_connect (at 185.42 20.32)
+	)
+	(hierarchical_label "EXT_TX_EVIDENCE_N"
+		(shape bidirectional)
+		(at 190.50 25.40 180)
+		(effects (font (size 1.27 1.27)) (justify right))
+	)
+	(wire
+		(pts (xy 190.50 25.40) (xy 185.42 25.40))
+		(stroke (width 0) (type default))
+	)
+	(no_connect (at 185.42 25.40)
+	)
 	(sheet_instances
 		(path "/"

Commit message: complete H2.4 LoRa Cap schematics
Parts:
- added C1: TDK C1005X7R1H104K050BB, Capacitor_SMD:C_0402_1005Metric, symbol Leshy2:CAP30_EVIDENCE_COMPARATOR_BYPASS
- added C2: TDK C1005X7R1H104K050BB, Capacitor_SMD:C_0402_1005Metric, symbol Leshy2:CAP30_EVIDENCE_TIMING_CAPACITOR
- added C3: TDK C1005X7R1H104K050BB, Capacitor_SMD:C_0402_1005Metric, symbol Leshy2:CAP30_EVIDENCE_MONOSTABLE_BYPASS
- added C4: TDK C1005X7R1H104K050BB, Capacitor_SMD:C_0402_1005Metric, symbol Leshy2:CAP30_EVIDENCE_DRIVER_BYPASS
- added R1: Yageo RC0402FR-07220KL, Resistor_SMD:R_0402_1005Metric, symbol Leshy2:CAP30_EVIDENCE_THRESHOLD_TOP
- added R2: Yageo RC0402FR-0710KL, Resistor_SMD:R_0402_1005Metric, symbol Leshy2:CAP30_EVIDENCE_THRESHOLD_BOTTOM
- added R3: Yageo RC0402FR-0710KL, Resistor_SMD:R_0402_1005Metric, symbol Leshy2:CAP30_EVIDENCE_COMPARATOR_PULLUP
- added R4: Yageo RC0402FR-07133KL, Resistor_SMD:R_0402_1005Metric, symbol Leshy2:CAP30_EVIDENCE_TIMING_RESISTOR
- added U1: TLV1821DCKR, Package_TO_SOT_SMD:Texas_R-PDSO-G5_DCK-5, symbol Leshy2:CAP30_EVIDENCE_COMPARATOR
- added U2: SN74LVC1G123DCTR, Package_SO:SSOP-8_2.95x2.8mm_P0.65mm, symbol Leshy2:CAP30_EVIDENCE_MONOSTABLE
- added U3: Texas Instruments SN74LVC1G06DCKR, Package_TO_SOT_SMD:Texas_R-PDSO-G5_DCK-5, symbol Leshy2:CAP30_EVIDENCE_DRIVER
Connections:
- net CAP_3V3: now also C1.1 (END_1), C3.1 (END_1), C4.1 (END_1), R1.1 (END_1), R3.1 (END_1), R4.1 (END_1), U1.5 (VPLUS), U2.3 (CLR_N), U2.8 (VCC), U3.5 (VCC)
- net EXT_TX_EVIDENCE_N: now also U3.4 (Y)
- net GND: now also C1.2 (END_2), C3.2 (END_2), C4.2 (END_2), R2.2 (END_2), U1.2 (VMINUS), U2.1 (A), U2.4 (GND), U3.3 (GND)
- net RF_FORWARD_LEVEL: now also U1.3 (IN_P)
- new net EVIDENCE_PULSE_HIGH: U2.5 (Q), U3.2 (A)
- new net EVIDENCE_TIMING_POSITIVE: C2.1 (END_1), R4.2 (END_2), U2.7 (REXT_CEXT)
- new net EVIDENCE_TIMING_RETURN: C2.2 (END_2), U2.6 (CEXT)
- new net RF_DETECTED_HIGH: R3.2 (END_2), U1.1 (OUT), U2.2 (B)
- new net RF_EVIDENCE_THRESHOLD: R1.2 (END_2), R2.1 (END_1), U1.4 (IN_N)
- no-connect marks 4 -> 1
Other:
- title: (none) -> Leshy2 LoRa Cap — independent physical-TX evidence pulse

Commit message: complete H2 schematic review package
Parts:
- renumbered C1 to C30001, C2 to C30002, C3 to C30003, C4 to C30004, R1 to R30001, R2 to R30002, R3 to R30003, R4 to R30004, U1 to U30001, U2 to U30002, U3 to U30003
Changed lines of the file:
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@@
 		(on_board yes)
 		(dnp no)
-		(property "Reference" "U1"
+		(property "Reference" "U30001"
 			(at 40.64 40.64 0)
 			(show_name no)
@@
 			(project "LESHY2-LORA-CAP-01"
 				(path "/08a28aac-c71c-5199-be87-354daca6d9cb"
-					(reference "U1")
+					(reference "U30001")
 					(unit 1)
 				)
@@
 		(on_board yes)
 		(dnp no)
-		(property "Reference" "R1"
+		(property "Reference" "R30001"
 			(at 99.06 36.83 0)
 			(show_name no)
@@
 			(project "LESHY2-LORA-CAP-01"
 				(path "/08a28aac-c71c-5199-be87-354daca6d9cb"
-					(reference "R1")
+					(reference "R30001")
 					(unit 1)
 				)
@@
 		(on_board yes)
 		(dnp no)
-		(property "Reference" "R2"
+		(property "Reference" "R30002"
 			(at 157.48 36.83 0)
 			(show_name no)
@@
 			(project "LESHY2-LORA-CAP-01"
 				(path "/08a28aac-c71c-5199-be87-354daca6d9cb"
-					(reference "R2")
+					(reference "R30002")
 					(unit 1)
 				)
@@
 		(on_board yes)
 		(dnp no)
-		(property "Reference" "R3"
+		(property "Reference" "R30003"
 			(at 215.90 36.83 0)
 			(show_name no)
@@
 			(project "LESHY2-LORA-CAP-01"
 				(path "/08a28aac-c71c-5199-be87-354daca6d9cb"
-					(reference "R3")
+					(reference "R30003")
 					(unit 1)
 				)
@@
 		(on_board yes)
 		(dnp no)
-		(property "Reference" "C1"
+		(property "Reference" "C30001"
 			(at 274.32 36.83 0)
 			(show_name no)
@@
 			(project "LESHY2-LORA-CAP-01"
 				(path "/08a28aac-c71c-5199-be87-354daca6d9cb"
-					(reference "C1")
+					(reference "C30001")
 					(unit 1)
 				)
@@
 		(on_board yes)
 		(dnp no)
-		(property "Reference" "U2"
+		(property "Reference" "U30002"
 			(at 99.06 64.25 0)
 			(show_name no)
@@
 			(project "LESHY2-LORA-CAP-01"
 				(path "/08a28aac-c71c-5199-be87-354daca6d9cb"
-					(reference "U2")
+					(reference "U30002")
 					(unit 1)
 				)
@@
 		(on_board yes)
 		(dnp no)
-		(property "Reference" "R4"
+		(property "Reference" "R30004"
 			(at 157.48 62.23 0)
 			(show_name no)
@@
 			(project "LESHY2-LORA-CAP-01"
 				(path "/08a28aac-c71c-5199-be87-354daca6d9cb"
-					(reference "R4")
+					(reference "R30004")
 					(unit 1)
 				)
@@
 		(on_board yes)
 		(dnp no)
-		(property "Reference" "C2"
+		(property "Reference" "C30002"
 			(at 215.90 62.23 0)
 			(show_name no)
@@
 			(project "LESHY2-LORA-CAP-01"
 				(path "/08a28aac-c71c-5199-be87-354daca6d9cb"
-					(reference "C2")
+					(reference "C30002")
 					(unit 1)
 				)
@@
 		(on_board yes)
 		(dnp no)
-		(property "Reference" "C3"
+		(property "Reference" "C30003"
 			(at 274.32 62.23 0)
 			(show_name no)
@@
 			(project "LESHY2-LORA-CAP-01"
 				(path "/08a28aac-c71c-5199-be87-354daca6d9cb"
-					(reference "C3")
+					(reference "C30003")
 					(unit 1)
 				)
@@
 		(on_board yes)
 		(dnp no)
-		(property "Reference" "U3"
+		(property "Reference" "U30003"
 			(at 40.64 68.58 0)
 			(show_name no)
@@
 			(project "LESHY2-LORA-CAP-01"
 				(path "/08a28aac-c71c-5199-be87-354daca6d9cb"
-					(reference "U3")
+					(reference "U30003")
 					(unit 1)
 				)
@@
 		(on_board yes)
 		(dnp no)
-		(property "Reference" "C4"
+		(property "Reference" "C30004"
 			(at 157.48 87.63 0)
 			(show_name no)
@@
 			(project "LESHY2-LORA-CAP-01"
 				(path "/08a28aac-c71c-5199-be87-354daca6d9cb"
-					(reference "C4")
-					(unit 1)
-				)
+					(reference "C30004")
+					(unit 1)
+				)

Commit message: Optimize H1 display and stocked BOM routes
Parts:
- C30001, C30002, C30003, C30004: value TDK C1005X7R1H104K050BB -> Yageo CC0402KRX7R9BB104
Changed lines of the file:
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@@
 			(effects (font (size 1.27 1.27)))
 		)
-		(property "Value" "TDK C1005X7R1H104K050BB"
+		(property "Value" "Yageo CC0402KRX7R9BB104"
 			(at 274.32 46.99 0)
 			(show_name no)
@@
 			(effects (font (size 1.27 1.27)))
 		)
-		(property "Value" "TDK C1005X7R1H104K050BB"
+		(property "Value" "Yageo CC0402KRX7R9BB104"
 			(at 215.90 72.39 0)
 			(show_name no)
@@
 			(effects (font (size 1.27 1.27)))
 		)
-		(property "Value" "TDK C1005X7R1H104K050BB"
+		(property "Value" "Yageo CC0402KRX7R9BB104"
 			(at 274.32 72.39 0)
 			(show_name no)
@@
 			(effects (font (size 1.27 1.27)))
 		)
-		(property "Value" "TDK C1005X7R1H104K050BB"
+		(property "Value" "Yageo CC0402KRX7R9BB104"
 			(at 157.48 97.79 0)
 			(show_name no)

Commit message: Replace six pre-order resistor identities
Parts:
- R30004: value Yageo RC0402FR-07133KL -> UNI-ROYAL 0402WGF1333TCE
Changed lines of the file:
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@@
 			(effects (font (size 1.27 1.27)))
 		)
-		(property "Value" "Yageo RC0402FR-07133KL"
+		(property "Value" "UNI-ROYAL 0402WGF1333TCE"
 			(at 157.48 72.39 0)
 			(show_name no)
