File: hardware/ecad/kicad/LESHY2-RF/RF_03_MAIN_RAILS_DOMAIN_GATES.kicad_sch (KiCad schematic)
At the start: 69 parts, among them Q3001 Diodes Incorporated MMBT3904-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, U3001 74LVC1G32GV,125, U3002 Texas Instruments SN74LVC2G08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, U3003 Texas Instruments TPS629203DR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, U3004 Texas Instruments TPS25961DRVR, U3005 Texas Instruments TPS564252DR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, U3006 Texas Instruments TPS25974LRP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, U3007 Texas Instruments TPS564252DR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, U3008 Texas Instruments TPS259470LR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, U3009 SN74LVC1G07DCKR

Commit message: review H3.6.2 single-fault containment
Connections:
- net EXT_ANY_5V_EN_SAFE: no longer U3002.2 (1B), U3002.6 (2B)
- new net FAULT_ASSERT_N: U3002.2 (1B), U3002.6 (2B)
Changed lines of the file:
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@@
 	(hierarchical_label "EXT_ANY_5V_EN_SAFE"
 		(shape bidirectional)
-		(at 276.86 45.72 0)
-		(effects (font (size 1.27 1.27)))
-	)
-	(label "EXT_ANY_5V_EN_SAFE"
-		(at 312.42 45.72 180)
-		(effects (font (size 1.27 1.27)) (justify right bottom))
-	)
-	(label "EXT_ANY_5V_EN_SAFE"
 		(at 231.14 172.72 180)
 		(effects (font (size 1.27 1.27)) (justify right bottom))
@@
 		(effects (font (size 1.27 1.27)))
 	)
+	(hierarchical_label "FAULT_ASSERT_N"
+		(shape bidirectional)
+		(at 276.86 45.72 0)
+		(effects (font (size 1.27 1.27)))
+	)
+	(label "FAULT_ASSERT_N"
+		(at 312.42 45.72 180)
+		(effects (font (size 1.27 1.27)) (justify right bottom))
+	)
 	(label "MAIN_3V3_FB"
