File: hardware/ecad/kicad/LESHY2-RF/LESHY2-RF.kicad_sch (KiCad schematic)
At the start: 0 parts

Commit message: complete exact H2.3.1 RF power hierarchy
Other:
- added sheet RF_01_USB_PD_CHARGE (RF_01_USB_PD_CHARGE.kicad_sch)
- added sheet RF_02_PACK_SAFETY_AON (RF_02_PACK_SAFETY_AON.kicad_sch)
- added sheet RF_03_MAIN_RAILS_DOMAIN_GATES (RF_03_MAIN_RAILS_DOMAIN_GATES.kicad_sch)
- added sheet RF_30_RP2354_CORE_SERVICE (RF_30_RP2354_CORE_SERVICE.kicad_sch)
- added sheet RF_31_NRF24_X3 (RF_31_NRF24_X3.kicad_sch)
- added sheet RF_32_SUBGHZ_VOICE (RF_32_SUBGHZ_VOICE.kicad_sch)
- added sheet RF_34_U214_M5_EXT (RF_34_U214_M5_EXT.kicad_sch)
- added sheet RF_35_REAR_CONTROLS (RF_35_REAR_CONTROLS.kicad_sch)
- added sheet RF_36_AUDIO_IO_AMP (RF_36_AUDIO_IO_AMP.kicad_sch)
- added sheet RF_40_INTERBOARD_M1 (RF_40_INTERBOARD_M1.kicad_sch)
- added sheet RF_50_TX_SAFETY_EVIDENCE (RF_50_TX_SAFETY_EVIDENCE.kicad_sch)
- added sheet RF_60_TESTPOINTS_MANUFACTURING (RF_60_TESTPOINTS_MANUFACTURING.kicad_sch)

Commit message: complete exact H2.3.2 USB PD charging
Other:
- sheet RF_01_USB_PD_CHARGE ports: added none; removed AON_BUCK_EN
- sheet RF_03_MAIN_RAILS_DOMAIN_GATES ports: added none; removed AON_BUCK_EN

Commit message: complete exact H2.3.3 pack safety
Other:
- sheet RF_02_PACK_SAFETY_AON ports: added 3V3_MAIN; removed none
Changed lines of the file:
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@@
 			(effects (font (size 1.27 1.27)) (justify left top))
 		)
-		(pin "PACK_ADMISSION_VDD" bidirectional
+		(pin "3V3_MAIN" bidirectional
 			(at 274.32 78.74 0)
 			(effects (font (size 1.27 1.27)))
 		)
-		(pin "POWER_COMMAND_OFF_N" bidirectional
+		(pin "PACK_ADMISSION_VDD" bidirectional
 			(at 274.32 81.28 0)
 			(effects (font (size 1.27 1.27)))
 		)
-		(pin "POWER_GROUND" bidirectional
+		(pin "POWER_COMMAND_OFF_N" bidirectional
 			(at 274.32 83.82 0)
 			(effects (font (size 1.27 1.27)))
 		)
-		(pin "PROTECTED_PACK_POSITIVE" bidirectional
+		(pin "POWER_GROUND" bidirectional
 			(at 274.32 86.36 0)
 			(effects (font (size 1.27 1.27)))
 		)
-		(pin "SYS_I2C_SCL" bidirectional
+		(pin "PROTECTED_PACK_POSITIVE" bidirectional
 			(at 274.32 88.90 0)
 			(effects (font (size 1.27 1.27)))
 		)
-		(pin "SYS_I2C_SDA" bidirectional
+		(pin "SYS_I2C_SCL" bidirectional
 			(at 274.32 91.44 0)
 			(effects (font (size 1.27 1.27)))
 		)
-		(pin "SYS_INT_N" bidirectional
+		(pin "SYS_I2C_SDA" bidirectional
 			(at 274.32 93.98 0)
 			(effects (font (size 1.27 1.27)))
 		)
+		(pin "SYS_INT_N" bidirectional
+			(at 274.32 96.52 0)
+			(effects (font (size 1.27 1.27)))
+		)
 		(instances
 			(project "LESHY2-RF"
@@
 	)
 	(wire
+		(pts (xy 274.32 78.74) (xy 299.72 78.74))
+		(stroke (width 0) (type default))
+	)
+	(junction (at 299.72 78.74)
+		(diameter 0)
+		(color 0 0 0 0)
+	)
+	(wire
 		(pts (xy 274.32 129.54) (xy 299.72 129.54))
 		(stroke (width 0) (type default))
@@
 	)
 	(wire
-		(pts (xy 299.72 129.54) (xy 299.72 883.92))
+		(pts (xy 299.72 78.74) (xy 299.72 883.92))
 		(stroke (width 0) (type default))
 	)
@@
 	)
 	(wire
-		(pts (xy 274.32 78.74) (xy 477.52 78.74))
+		(pts (xy 274.32 81.28) (xy 477.52 81.28))
 		(stroke (width 0) (type default))
 	)
-	(junction (at 477.52 78.74)
+	(junction (at 477.52 81.28)
 		(diameter 0)
 		(color 0 0 0 0)
@@
 	)
 	(wire
-		(pts (xy 477.52 78.74) (xy 477.52 985.52))
+		(pts (xy 477.52 81.28) (xy 477.52 985.52))
 		(stroke (width 0) (type default))
 	)
@@
 	)
 	(wire
-		(pts (xy 274.32 81.28) (xy 482.60 81.28))
+		(pts (xy 274.32 83.82) (xy 482.60 83.82))
 		(stroke (width 0) (type default))
 	)
-	(junction (at 482.60 81.28)
+	(junction (at 482.60 83.82)
 		(diameter 0)
 		(color 0 0 0 0)
@@
 	)
 	(wire
-		(pts (xy 482.60 81.28) (xy 482.60 990.60))
+		(pts (xy 482.60 83.82) (xy 482.60 990.60))
 		(stroke (width 0) (type default))
 	)
@@
 	)
 	(wire
-		(pts (xy 274.32 83.82) (xy 487.68 83.82))
+		(pts (xy 274.32 86.36) (xy 487.68 86.36))
 		(stroke (width 0) (type default))
 	)
-	(junction (at 487.68 83.82)
+	(junction (at 487.68 86.36)
 		(diameter 0)
 		(color 0 0 0 0)
@@
 	)
 	(wire
-		(pts (xy 274.32 86.36) (xy 492.76 86.36))
+		(pts (xy 274.32 88.90) (xy 492.76 88.90))
 		(stroke (width 0) (type default))
 	)
-	(junction (at 492.76 86.36)
+	(junction (at 492.76 88.90)
 		(diameter 0)
 		(color 0 0 0 0)
 	)
 	(wire
-		(pts (xy 492.76 35.56) (xy 492.76 86.36))
+		(pts (xy 492.76 35.56) (xy 492.76 88.90))
 		(stroke (width 0) (type default))
 	)
@@
 	)
 	(wire
-		(pts (xy 274.32 88.90) (xy 543.56 88.90))
+		(pts (xy 274.32 91.44) (xy 543.56 91.44))
 		(stroke (width 0) (type default))
 	)
-	(junction (at 543.56 88.90)
+	(junction (at 543.56 91.44)
 		(diameter 0)
 		(color 0 0 0 0)
@@
 	)
 	(wire
-		(pts (xy 274.32 91.44) (xy 546.10 91.44))
+		(pts (xy 274.32 93.98) (xy 546.10 93.98))
 		(stroke (width 0) (type default))
 	)
-	(junction (at 546.10 91.44)
+	(junction (at 546.10 93.98)
 		(diameter 0)
 		(color 0 0 0 0)
@@
 	)
 	(wire
-		(pts (xy 274.32 93.98) (xy 548.64 93.98))
+		(pts (xy 274.32 96.52) (xy 548.64 96.52))
 		(stroke (width 0) (type default))
 	)
-	(junction (at 548.64 93.98)
+	(junction (at 548.64 96.52)
 		(diameter 0)
 		(color 0 0 0 0)

Commit message: complete exact H2.3.4 power rails
Other:
- sheet RF_03_MAIN_RAILS_DOMAIN_GATES ports: added POWER_FAULT_N; removed none
- sheet RF_32_SUBGHZ_VOICE ports: added POWER_FAULT_N; removed none
- sheet RF_34_U214_M5_EXT ports: added POWER_FAULT_N; removed none

Commit message: complete exact H2.3.13 RF testpoint sheet
Other:
- sheet RF_02_PACK_SAFETY_AON ports: added PACK_ADMISSION_NRST_N, PACK_ADMISSION_SWCLK, PACK_ADMISSION_SWDIO, PACK_ADMISSION_UART_RX, PACK_ADMISSION_UART_TX, PACK_FIXTURE_3V3; removed none
- sheet RF_03_MAIN_RAILS_DOMAIN_GATES ports: added MAIN_RAW_3V3_PG_N; removed none
- sheet RF_32_SUBGHZ_VOICE ports: added VOICE_RAW_4V_PG_N, VOICE_UPDATE_FIXTURE; removed none
- sheet RF_50_TX_SAFETY_EVIDENCE ports: added ANY_TX_AON_N, EVIDENCE_MASK_INT_N_TP, SAFETY_CONTROLLER_NRST_N, SAFETY_SERVICE_UART_RX, SAFETY_SERVICE_UART_TX, SAFETY_SWCLK, SAFETY_SWDIO; removed none
- sheet RF_60_TESTPOINTS_MANUFACTURING ports: added 3V3_MAIN, ANY_TX_AON_N, AON_SAFE_3V3, EVIDENCE_MASK_INT_N_TP, EV_N2_NRF0, EV_N3_NRF1, EV_N4_NRF2, EV_N5_CC, EV_N6_VOICE, EV_N8_LORA_EXT, MAIN_RAW_3V3_PG_N, PACK_ADMISSION_NRST_N, PACK_ADMISSION_SWCLK, PACK_ADMISSION_SWDIO, PACK_ADMISSION_UART_RX, PACK_ADMISSION_UART_TX, PACK_FIXTURE_3V3, POWER_FAULT_N, POWER_GROUND, POWER_ZONE_TEMP_ADC, RF_ZONE_TEMP_ADC, RP_RESET_N, RUN_PERMIT, SAFETY_CONTROLLER_NRST_N, SAFETY_SERVICE_UART_RX, SAFETY_SERVICE_UART_TX, SAFETY_SWCLK, SAFETY_SWDIO, VOICE_RAW_4V_PG_N, VOICE_UPDATE_FIXTURE; removed none

Commit message: complete H2 schematic review package
Other:
- sheet RF_01_USB_PD_CHARGE ports: added PD_EEPROM_WP, PD_LOCAL_I2C_SCL, PD_LOCAL_I2C_SDA; removed none
- sheet RF_30_RP2354_CORE_SERVICE ports: added RP_SERVICE_VBUS_SENSE_ONLY; removed none
- sheet RF_50_TX_SAFETY_EVIDENCE ports: added FAULT_ASSERT_N, RUN_EDGE, RUN_LOOP_RAW, SAFETY_WATCHDOG_WDI; removed none
- sheet RF_60_TESTPOINTS_MANUFACTURING ports: added CC_PWR_EN_SAFE, EXT_ANY_5V_EN_SAFE, FAULT_ASSERT_N, FAULT_LATCH_SENSE_AON, NRF0_CE_SAFE, NRF1_CE_SAFE, NRF2_CE_SAFE, NRF_GROUP_PWR_EN_SAFE, PD_EEPROM_WP, PD_LOCAL_I2C_SCL, PD_LOCAL_I2C_SDA, POR_N, RP_ANY_TX_N, RP_SERVICE_VBUS_SENSE_ONLY, RUN_EDGE, RUN_LOOP_RAW, SAFETY_WATCHDOG_WDI, SYS_I2C_SCL, SYS_I2C_SDA, SYS_INT_N, VOICE_DOMAIN_EN_SAFE, VOICE_PTT_SAFE_N; removed none

Commit message: review H3.6.2 single-fault containment
Other:
- sheet RF_03_MAIN_RAILS_DOMAIN_GATES ports: added FAULT_ASSERT_N; removed none
- sheet RF_31_NRF24_X3 ports: added FAULT_ASSERT_N, NRF_GROUP_PWR_EN_PRIMARY; removed none
- sheet RF_32_SUBGHZ_VOICE ports: added CC_PWR_EN_PRIMARY, FAULT_ASSERT_N, VOICE_EFUSE_BACKUP_EN_N; removed none
- sheet RF_40_INTERBOARD_M1 ports: added FAULT_ASSERT_N; removed RF_RESET_KILL_GATE
- sheet RF_50_TX_SAFETY_EVIDENCE ports: added CC_PWR_EN_PRIMARY, NRF_GROUP_PWR_EN_PRIMARY, VOICE_EFUSE_BACKUP_EN_N; removed NRF_GROUP_PWR_EN_SAFE, RF_RESET_KILL_GATE

Commit message: Reclose H2 through H4 on dual SA818S architecture
Other:
- sheet RF_32_SUBGHZ_VOICE ports: added RX_VOICE_AFOUT_SELECTED, SYS_I2C_SCL, SYS_I2C_SDA, SYS_INT_N, VOICE_U_RF_SAMPLE, VOICE_V_DETECT_FILTER, VOICE_V_DETECT_V, VOICE_V_RF_SAMPLE; removed RX_SA518_AFOUT_ISOLATED, VOICE_RF_SAMPLE, VOICE_UPDATE_FIXTURE
- sheet RF_40_INTERBOARD_M1 ports: added RX_VOICE_AFOUT_SELECTED; removed RX_SA518_AFOUT_ISOLATED
- sheet RF_50_TX_SAFETY_EVIDENCE ports: added VOICE_U_RF_SAMPLE, VOICE_V_DETECT_FILTER, VOICE_V_DETECT_V, VOICE_V_RF_SAMPLE; removed VOICE_RF_SAMPLE
- sheet RF_60_TESTPOINTS_MANUFACTURING ports: added none; removed VOICE_UPDATE_FIXTURE
