File: hardware/ecad/kicad/LESHY2-RF/RF_30_RP2354_CORE_SERVICE.kicad_sch (KiCad schematic)
At the start: 0 parts

Commit message: complete exact H2.3.1 RF power hierarchy
Connections:
- no-connect marks 0 -> 51

Commit message: complete exact H2.3.5 RP2354 core
Parts:
- added C1: TDK C1005X5R0J475K050BC, Capacitor_SMD:C_0402_1005Metric, symbol Leshy2:RF30_RP_VREG_VIN_BULK
- added C10: TDK C1005X7R1H104K050BB, Capacitor_SMD:C_0402_1005Metric, symbol Leshy2:RF30_RP_IOVDD5_BYPASS
- added C11: TDK C1005X7R1H104K050BB, Capacitor_SMD:C_0402_1005Metric, symbol Leshy2:RF30_RP_IOVDD15_BYPASS
- added C12: TDK C1005X7R1H104K050BB, Capacitor_SMD:C_0402_1005Metric, symbol Leshy2:RF30_RP_IOVDD24_BYPASS
- added C13: TDK C1005X7R1H104K050BB, Capacitor_SMD:C_0402_1005Metric, symbol Leshy2:RF30_RP_IOVDD29_BYPASS
- added C14: TDK C1005X7R1H104K050BB, Capacitor_SMD:C_0402_1005Metric, symbol Leshy2:RF30_RP_IOVDD41_BYPASS
- added C15: TDK C1005X7R1H104K050BB, Capacitor_SMD:C_0402_1005Metric, symbol Leshy2:RF30_RP_IOVDD50_BYPASS
- added C16: TDK C1005X7R1H104K050BB, Capacitor_SMD:C_0402_1005Metric, symbol Leshy2:RF30_RP_IOVDD60_BYPASS
- added C17: TDK C1005X7R1H104K050BB, Capacitor_SMD:C_0402_1005Metric, symbol Leshy2:RF30_RP_IOVDD76_BYPASS
- added C18: TDK C1005X7R1H104K050BB, Capacitor_SMD:C_0402_1005Metric, symbol Leshy2:RF30_RP_ADC_AVDD_BYPASS
- added C19: TDK C1005X7R1H104K050BB, Capacitor_SMD:C_0402_1005Metric, symbol Leshy2:RF30_RP_USB_OTP_VDD_BYPASS
- added C2: TDK C1005X5R0J475K050BC, Capacitor_SMD:C_0402_1005Metric, symbol Leshy2:RF30_RP_VREG_OUTPUT_BULK
- added C20: TDK C1005X7R1H104K050BB, Capacitor_SMD:C_0402_1005Metric, symbol Leshy2:RF30_RP_QSPI_IOVDD_BYPASS
- added C21: TDK C1005X7R1H104K050BB, Capacitor_SMD:C_0402_1005Metric, symbol Leshy2:RF30_RP_SERVICE_USB_SWITCH_BYPASS
- added C3: TDK C1005X5R0J475K050BC, Capacitor_SMD:C_0402_1005Metric, symbol Leshy2:RF30_RP_VREG_AVDD_FILTER_CAP
- added C4: TDK C1005X5R0J475K050BC, Capacitor_SMD:C_0402_1005Metric, symbol Leshy2:RF30_RP_DVDD_REMOTE_BULK
- added C5: Murata GJM1555C1H150JB01D, Capacitor_SMD:C_0402_1005Metric, symbol Leshy2:RF30_RP_CLOCK_LOAD_XIN
- added C6: Murata GJM1555C1H150JB01D, Capacitor_SMD:C_0402_1005Metric, symbol Leshy2:RF30_RP_CLOCK_LOAD_XOUT
- added C7: TDK C1005X7R1H104K050BB, Capacitor_SMD:C_0402_1005Metric, symbol Leshy2:RF30_RP_DVDD10_BYPASS
- added C8: TDK C1005X7R1H104K050BB, Capacitor_SMD:C_0402_1005Metric, symbol Leshy2:RF30_RP_DVDD32_BYPASS
- added C9: TDK C1005X7R1H104K050BB, Capacitor_SMD:C_0402_1005Metric, symbol Leshy2:RF30_RP_DVDD51_BYPASS
- added D1: Texas Instruments TPD2EUSB30ADRTR, Package_TO_SOT_SMD:SOT-23, symbol Leshy2:RF30_RP_SERVICE_USB_ESD
- added D2: Texas Instruments TPD4E05U06DQAR, Package_SON:USON-10_2.5x1.0mm_P0.5mm, symbol Leshy2:RF30_RP_DBG_ESD
- added J1: GCT USB4105-GF-A, Connector_USB:USB_C_Receptacle_GCT_USB4105-xx-A_16P_TopMnt_Horizontal, symbol Leshy2:RF30_RP_SERVICE_USB_CONNECTOR
- added J2: Samtec FTSH-105-01-L-DV-K-P-TR, Leshy2:FTSH-105-01-L-DV-K-P-TR, symbol Leshy2:RF30_RP_DBG_HEADER
- added L1: Abracon AOTA-B201610S3R3-101-T, Inductor_SMD:L_Murata_DFE201610P, symbol Leshy2:RF30_RP_VREG_INDUCTOR
- added R1: Yageo RC0402FR-0733RL, Resistor_SMD:R_0402_1005Metric, symbol Leshy2:RF30_RP_VREG_AVDD_FILTER_RES
- added R10: Yageo RC0402FR-071KL, Resistor_SMD:R_0402_1005Metric, symbol Leshy2:RF30_RP_DBG_BOOT_SERIES
- added R11: Yageo RC0402FR-07470RL, Resistor_SMD:R_0402_1005Metric, symbol Leshy2:RF30_RP_DBG0_SERIES
- added R12: Yageo RC0402FR-07470RL, Resistor_SMD:R_0402_1005Metric, symbol Leshy2:RF30_RP_DBG1_SERIES
- added R13: Yageo RC0402FR-0710KL, Resistor_SMD:R_0402_1005Metric, symbol Leshy2:RF30_RP_DBG_ID0_STRAP
- added R14: Yageo RC0402FR-0710KL, Resistor_SMD:R_0402_1005Metric, symbol Leshy2:RF30_RP_DBG_ID1_STRAP
- added R15: Yageo RC0402FR-0710KL, Resistor_SMD:R_0402_1005Metric, symbol Leshy2:RF30_RP_BOOT_PULLUP
- added R16: Yageo RC0402FR-0710KL, Resistor_SMD:R_0402_1005Metric, symbol Leshy2:RF30_RP_RESET_PULLUP
- added R17: Yageo RC0402FR-0710KL, Resistor_SMD:R_0402_1005Metric, symbol Leshy2:RF30_RP_ANY_TX_MAIN_PULLUP
- added R2: Yageo RC0402FR-071KL, Resistor_SMD:R_0402_1005Metric, symbol Leshy2:RF30_RP_CLOCK_SERIES
- added R3: Yageo RC0402FR-075K1L, Resistor_SMD:R_0402_1005Metric, symbol Leshy2:RF30_RP_SERVICE_USB_CC1_RD
- added R4: Yageo RC0402FR-075K1L, Resistor_SMD:R_0402_1005Metric, symbol Leshy2:RF30_RP_SERVICE_USB_CC2_RD
- added R5: Yageo RC0402FR-071ML, Resistor_SMD:R_0402_1005Metric, symbol Leshy2:RF30_RP_SERVICE_USB_VBUS_BLEEDER
- added R6: Panasonic ERJ-2RKF27R0X, Resistor_SMD:R_0402_1005Metric, symbol Leshy2:RF30_RP_SERVICE_USB_DM_SERIES
- added R7: Panasonic ERJ-2RKF27R0X, Resistor_SMD:R_0402_1005Metric, symbol Leshy2:RF30_RP_SERVICE_USB_DP_SERIES
- added R8: Yageo RC0402FR-071KL, Resistor_SMD:R_0402_1005Metric, symbol Leshy2:RF30_RP_DBG_VTREF_SERIES
- added R9: Yageo RC0402FR-071KL, Resistor_SMD:R_0402_1005Metric, symbol Leshy2:RF30_RP_DBG_RESET_SERIES
- added SW1: Alps Alpine SKRTLAE010, Button_Switch_SMD:SW_Push_1P1T-MP_NO_Horizontal_Alps_SKRTLAE010, symbol Leshy2:RF30_RP_RESET_BUTTON
- added SW2: Alps Alpine SKRTLAE010, Button_Switch_SMD:SW_Push_1P1T-MP_NO_Horizontal_Alps_SKRTLAE010, symbol Leshy2:RF30_RP_BOOT_BUTTON
- added U1: SC1512-A4, Package_DFN_QFN:QFN-80-1EP_10x10mm_P0.4mm_EP3.4x3.4mm, symbol Leshy2:RF30_RP
- added U2: onsemi FSUSB42MUX, Package_SO:MSOP-10_3x3mm_P0.5mm, symbol Leshy2:RF30_RP_SERVICE_USB_SWITCH
- added Y1: Abracon ABM8-272-T3, Crystal:Crystal_SMD_Abracon_ABM8G-4Pin_3.2x2.5mm, symbol Leshy2:RF30_RP_CLOCK
Connections:
- net 3V3_MAIN: now also C1.1 (END_1), C10.1 (END_1), C11.1 (END_1), C12.1 (END_1), C13.1 (END_1), C14.1 (END_1), C15.1 (END_1), C16.1 (END_1), C17.1 (END_1), C18.1 (END_1), C19.1 (END_1), C20.1 (END_1), C21.1 (END_1), R1.1 (END_1), R14.2 (END_2), R15.1 (END_1), R16.1 (END_1), R17.1 (END_1), R8.2 (END_2), U1.15 (IOVDD_15), U1.24 (IOVDD_24), U1.29 (IOVDD_29), U1.41 (IOVDD_41), U1.5 (IOVDD_5), U1.50 (IOVDD_50), U1.59 (ADC_AVDD), U1.60 (IOVDD_60), U1.64 (VREG_VIN), U1.68 (USB_OTP_VDD), U1.69 (QSPI_IOVDD), U1.76 (IOVDD_76), U2.1 (VCC)
- net CC_CSN_N: now also U1.7 (GPIO9)
- net CC_GDO0: now also U1.8 (GPIO10)
- net CC_GDO2: now also U1.9 (GPIO11)
- net CC_MISO: now also U1.48 (GPIO39)
- net CC_MOSI: now also U1.54 (GPIO43)
- net CC_PWR_EN: now also U1.23 (GPIO23)
- net CC_SCK: now also U1.53 (GPIO42)
- net NRF0_CE_REQ: now also U1.78 (GPIO1)
- net NRF0_CSN_N: now also U1.77 (GPIO0)
- net NRF0_IRQ_N: now also U1.79 (GPIO2)
- net NRF0_MISO: now also U1.38 (GPIO30)
- net NRF0_MOSI: now also U1.40 (GPIO32)
- net NRF0_SCK: now also U1.39 (GPIO31)
- net NRF1_CE_REQ: now also U1.1 (GPIO4)
- net NRF1_CSN_N: now also U1.80 (GPIO3)
- net NRF1_IRQ_N: now also U1.2 (GPIO5)
- net NRF1_MISO: now also U1.42 (GPIO33)
- net NRF1_MOSI: now also U1.44 (GPIO35)
- net NRF1_SCK: now also U1.43 (GPIO34)
- net NRF2_CE_REQ: now also U1.4 (GPIO7)
- net NRF2_CSN_N: now also U1.3 (GPIO6)
- net NRF2_IRQ_N: now also U1.6 (GPIO8)
- net NRF2_MISO: now also U1.45 (GPIO36)
- net NRF2_MOSI: now also U1.47 (GPIO38)
- net NRF2_SCK: now also U1.46 (GPIO37)
- net NRF_GROUP_PWR_EN: now also U1.14 (GPIO15)
- net POWER_GROUND: now also C1.2 (END_2), C10.2 (END_2), C11.2 (END_2), C12.2 (END_2), C13.2 (END_2), C14.2 (END_2), C15.2 (END_2), C16.2 (END_2), C17.2 (END_2), C18.2 (END_2), C19.2 (END_2), C2.2 (END_2), C20.2 (END_2), C21.2 (END_2), C3.2 (END_2), C4.2 (END_2), C5.2 (END_2), C6.2 (END_2), C7.2 (END_2), C8.2 (END_2), C9.2 (END_2), D1.3 (GND), D2.3 (GND_3), D2.8 (GND_8), J1.A1 (A1_GND), J1.A12 (A12_GND), J1.B1 (B1_GND), J1.B12 (B12_GND), J1.SH (SHIELD), J2.2 (P2), J2.7 (P7), J2.9 (P9), R13.2 (END_2), R3.2 (END_2), R4.2 (END_2), R5.2 (END_2), SW1.2 (NO), SW2.2 (NO), U1.62 (VREG_PGND), U1.81 (GND_EP), U2.10 (OE), U2.2 (SEL), U2.5 (GND), Y1.2 (GND_2), Y1.4 (GND_4)
- net PTT_BUTTON_N: now also U1.21 (GPIO21)
- net RP_ALERT_N: now also U1.19 (GPIO19)
- net RP_ANY_TX_N: now also R17.2 (END_2), U1.22 (GPIO22)
- net RP_RESET_N: now also R16.2 (END_2), R9.2 (END_2), U1.35 (RUN)
- net S3_RP_IPC_CS_N: now also U1.26 (GPIO25)
- net S3_RP_IPC_MISO: now also U1.28 (GPIO27)
- net S3_RP_IPC_MOSI: now also U1.25 (GPIO24)
- net S3_RP_IPC_SCK: now also U1.27 (GPIO26)
- net U214_HOST_BUSY: now also U1.11 (GPIO12)
- net U214_HOST_GPS_RX: now also U1.52 (GPIO41)
- net U214_HOST_GPS_TX: now also U1.49 (GPIO40)
- net U214_HOST_IRQ: now also U1.12 (GPIO13)
- net U214_HOST_MISO: now also U1.55 (GPIO44)
- net U214_HOST_MOSI: now also U1.57 (GPIO46)
- net U214_HOST_NSS_N: now also U1.58 (GPIO47)
- net U214_HOST_RST_N: now also U1.13 (GPIO14)
- net U214_HOST_SCK: now also U1.56 (GPIO45)
- net U214_I2C_SCL_IN: now also U1.37 (GPIO29)
- net U214_I2C_SDA_IN: now also U1.36 (GPIO28)
- net VOICE_AUDIO_ON_N: now also U1.20 (GPIO20)
- net VOICE_PTT_REQ_N: now also U1.18 (GPIO18)
- net VOICE_UART_RX: now also U1.17 (GPIO17)
- net VOICE_UART_TX: now also U1.16 (GPIO16)
- new net RP_CORE_1V1: C2.1 (END_1), C4.1 (END_1), C7.1 (END_1), C8.1 (END_1), C9.1 (END_1), L1.1 (END_1), U1.10 (DVDD_10), U1.32 (DVDD_32), U1.51 (DVDD_51), U1.65 (VREG_FB)
- new net RP_DBG0_CONNECTOR: D2.4 (D2_PLUS), J2.5 (P5), R11.1 (END_1)
- new net RP_DBG1_CONNECTOR: D2.5 (D2_MINUS), J2.6 (P6), R12.1 (END_1)
- new net RP_DBG_BOOT_CONNECTOR_N: D2.2 (D1_MINUS), J2.4 (P4), R10.1 (END_1), SW2.1 (C1), SW2.3 (C2)
- new net RP_DBG_ID0: J2.8 (P8), R13.1 (END_1)
- new net RP_DBG_ID1: J2.10 (P10), R14.1 (END_1)
- new net RP_DBG_RESET_CONNECTOR_N: D2.1 (D1_PLUS), J2.3 (P3), R9.1 (END_1), SW1.1 (C1), SW1.3 (C2)
- new net RP_DBG_VTREF_SENSE: J2.1 (P1), R8.1 (END_1)
- new net RP_SERVICE_CC1: J1.A5 (A5_CC1), R3.1 (END_1)
- new net RP_SERVICE_CC2: J1.B5 (B5_CC2), R4.1 (END_1)
- new net RP_SERVICE_USB_DM_CONNECTOR: D1.2 (D_MINUS), J1.A7 (A7_DM), J1.B7 (B7_DM), U2.4 (D_MINUS)
- new net RP_SERVICE_USB_DM_SWITCHED: R6.1 (END_1), U2.6 (HSD1_MINUS)
- new net RP_SERVICE_USB_DP_CONNECTOR: D1.1 (D_PLUS), J1.A6 (A6_DP), J1.B6 (B6_DP), U2.3 (D_PLUS)
- new net RP_SERVICE_USB_DP_SWITCHED: R7.1 (END_1), U2.7 (HSD1_PLUS)
- new net RP_SERVICE_VBUS_SENSE_ONLY: J1.A4 (A4_VBUS), J1.A9 (A9_VBUS), J1.B4 (B4_VBUS), J1.B9 (B9_VBUS), R5.1 (END_1)
- new net RP_SWCLK: R12.2 (END_2), U1.33 (SWCLK)
- new net RP_SWDIO: R11.2 (END_2), U1.34 (SWDIO)
- new net RP_USB_BOOT_N: R10.2 (END_2), R15.2 (END_2), U1.75 (QSPI_SS_USB_BOOT)
- new net RP_USB_DM: R6.2 (END_2), U1.66 (USB_DM)
- new net RP_USB_DP: R7.2 (END_2), U1.67 (USB_DP)
- new net RP_VREG_AVDD_FILTERED: C3.1 (END_1), R1.2 (END_2), U1.61 (VREG_AVDD)
- new net RP_VREG_LX_SW: L1.2 (END_2), U1.63 (VREG_LX)
- new net RP_XIN: C5.1 (END_1), U1.30 (XIN), Y1.1 (X1)
- new net RP_XOUT: R2.2 (END_2), U1.31 (XOUT)
- new net RP_XOUT_CRYSTAL: C6.1 (END_1), R2.1 (END_1), Y1.3 (X2)
- no-connect marks 51 -> 13
Other:
- title: (none) -> Leshy2 — exact RP2354B core, clock, USB and recovery

Commit message: complete H2 schematic review package
Parts:
- renumbered C1 to C30001, C2 to C30002, C3 to C30003, C4 to C30004, C5 to C30005, C6 to C30006, C7 to C30007, C8 to C30008, C9 to C30009, C10 to C30010, C11 to C30011, C12 to C30012, C13 to C30013, C14 to C30014, C15 to C30015, C16 to C30016, C17 to C30017, C18 to C30018, C19 to C30019, C20 to C30020, C21 to C30021, D1 to D30001, D2 to D30002, J1 to J30001, J2 to J30002, L1 to L30001, R1 to R30001, R2 to R30002, R3 to R30003, R4 to R30004, R5 to R30005, R6 to R30006, R7 to R30007, R8 to R30008, R9 to R30009, R10 to R30010, R11 to R30011, R12 to R30012, R13 to R30013, R14 to R30014, R15 to R30015, R16 to R30016, R17 to R30017, SW1 to SW30001, SW2 to SW30002, U1 to U30001, U2 to U30002, Y1 to Y30001

Commit message: Optimize H1 display and stocked BOM routes
Parts:
- C30007, C30008, C30009, C30010, C30011, C30012, C30013, C30014, C30015, C30016, C30017, C30018, C30019, C30020, C30021: value TDK C1005X7R1H104K050BB -> Yageo CC0402KRX7R9BB104
Changed lines of the file:
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@@
 			(effects (font (size 1.27 1.27)))
 		)
-		(property "Value" "TDK C1005X7R1H104K050BB"
+		(property "Value" "Yageo CC0402KRX7R9BB104"
 			(at 457.20 74.93 0)
 			(show_name no)
@@
 			(effects (font (size 1.27 1.27)))
 		)
-		(property "Value" "TDK C1005X7R1H104K050BB"
+		(property "Value" "Yageo CC0402KRX7R9BB104"
 			(at 538.48 74.93 0)
 			(show_name no)
@@
 			(effects (font (size 1.27 1.27)))
 		)
-		(property "Value" "TDK C1005X7R1H104K050BB"
+		(property "Value" "Yageo CC0402KRX7R9BB104"
 			(at 132.08 100.33 0)
 			(show_name no)
@@
 			(effects (font (size 1.27 1.27)))
 		)
-		(property "Value" "TDK C1005X7R1H104K050BB"
+		(property "Value" "Yageo CC0402KRX7R9BB104"
 			(at 213.36 100.33 0)
 			(show_name no)
@@
 			(effects (font (size 1.27 1.27)))
 		)
-		(property "Value" "TDK C1005X7R1H104K050BB"
+		(property "Value" "Yageo CC0402KRX7R9BB104"
 			(at 294.64 100.33 0)
 			(show_name no)
@@
 			(effects (font (size 1.27 1.27)))
 		)
-		(property "Value" "TDK C1005X7R1H104K050BB"
+		(property "Value" "Yageo CC0402KRX7R9BB104"
 			(at 375.92 100.33 0)
 			(show_name no)
@@
 			(effects (font (size 1.27 1.27)))
 		)
-		(property "Value" "TDK C1005X7R1H104K050BB"
+		(property "Value" "Yageo CC0402KRX7R9BB104"
 			(at 457.20 100.33 0)
 			(show_name no)
@@
 			(effects (font (size 1.27 1.27)))
 		)
-		(property "Value" "TDK C1005X7R1H104K050BB"
+		(property "Value" "Yageo CC0402KRX7R9BB104"
 			(at 538.48 100.33 0)
 			(show_name no)
@@
 			(effects (font (size 1.27 1.27)))
 		)
-		(property "Value" "TDK C1005X7R1H104K050BB"
+		(property "Value" "Yageo CC0402KRX7R9BB104"
 			(at 132.08 125.73 0)
 			(show_name no)
@@
 			(effects (font (size 1.27 1.27)))
 		)
-		(property "Value" "TDK C1005X7R1H104K050BB"
+		(property "Value" "Yageo CC0402KRX7R9BB104"
 			(at 213.36 125.73 0)
 			(show_name no)
@@
 			(effects (font (size 1.27 1.27)))
 		)
-		(property "Value" "TDK C1005X7R1H104K050BB"
+		(property "Value" "Yageo CC0402KRX7R9BB104"
 			(at 294.64 125.73 0)
 			(show_name no)
@@
 			(effects (font (size 1.27 1.27)))
 		)
-		(property "Value" "TDK C1005X7R1H104K050BB"
+		(property "Value" "Yageo CC0402KRX7R9BB104"
 			(at 375.92 125.73 0)
 			(show_name no)
@@
 			(effects (font (size 1.27 1.27)))
 		)
-		(property "Value" "TDK C1005X7R1H104K050BB"
+		(property "Value" "Yageo CC0402KRX7R9BB104"
 			(at 457.20 125.73 0)
 			(show_name no)
@@
 			(effects (font (size 1.27 1.27)))
 		)
-		(property "Value" "TDK C1005X7R1H104K050BB"
+		(property "Value" "Yageo CC0402KRX7R9BB104"
 			(at 538.48 125.73 0)
 			(show_name no)
@@
 			(effects (font (size 1.27 1.27)))
 		)
-		(property "Value" "TDK C1005X7R1H104K050BB"
+		(property "Value" "Yageo CC0402KRX7R9BB104"
 			(at 375.92 151.13 0)
 			(show_name no)
