File: hardware/ecad/kicad/LESHY2-RF/RF_31_NRF24_X3.kicad_sch (KiCad schematic)
At the start: 0 parts

Commit message: complete exact H2.3.1 RF power hierarchy
Connections:
- no-connect marks 0 -> 33

Commit message: complete exact H2.3.6 three-radio nRF24 sheet
Parts:
- added C1: TDK C1608X7R1C105K080AC, Capacitor_SMD:C_0603_1608Metric, symbol Leshy2:RF31_NRF_POWER_INPUT_CAP
- added C10: TDK C1005X7R1H104K050BB, Capacitor_SMD:C_0402_1005Metric, symbol Leshy2:RF31_NRF1_RETURN_BUFFER_BYPASS
- added C11: Murata GRM188R60J106ME47D, Capacitor_SMD:C_0603_1608Metric, symbol Leshy2:RF31_NRF1_MODULE_BULK_CAP
- added C12: TDK C1005X7R1H104K050BB, Capacitor_SMD:C_0402_1005Metric, symbol Leshy2:RF31_NRF1_MODULE_HF_CAP
- added C13: Murata GRM1555C1H121JA01D, Capacitor_SMD:C_0402_1005Metric, symbol Leshy2:RF31_NRF1_DETECTOR_FILTER
- added C14: TDK C1005X7R1H104K050BB, Capacitor_SMD:C_0402_1005Metric, symbol Leshy2:RF31_NRF1_DETECTOR_BYPASS
- added C15: TDK C1005X7R1H104K050BB, Capacitor_SMD:C_0402_1005Metric, symbol Leshy2:RF31_NRF2_HOST_BUFFER_BYPASS
- added C16: TDK C1005X7R1H104K050BB, Capacitor_SMD:C_0402_1005Metric, symbol Leshy2:RF31_NRF2_RETURN_BUFFER_BYPASS
- added C17: Murata GRM188R60J106ME47D, Capacitor_SMD:C_0603_1608Metric, symbol Leshy2:RF31_NRF2_MODULE_BULK_CAP
- added C18: TDK C1005X7R1H104K050BB, Capacitor_SMD:C_0402_1005Metric, symbol Leshy2:RF31_NRF2_MODULE_HF_CAP
- added C19: Murata GRM1555C1H121JA01D, Capacitor_SMD:C_0402_1005Metric, symbol Leshy2:RF31_NRF2_DETECTOR_FILTER
- added C2: TDK C1608X7R1C105K080AC, Capacitor_SMD:C_0603_1608Metric, symbol Leshy2:RF31_NRF_EVIDENCE_HOLD_CAP
- added C20: TDK C1005X7R1H104K050BB, Capacitor_SMD:C_0402_1005Metric, symbol Leshy2:RF31_NRF2_DETECTOR_BYPASS
- added C3: TDK C1005X7R1H104K050BB, Capacitor_SMD:C_0402_1005Metric, symbol Leshy2:RF31_NRF0_HOST_BUFFER_BYPASS
- added C4: TDK C1005X7R1H104K050BB, Capacitor_SMD:C_0402_1005Metric, symbol Leshy2:RF31_NRF0_RETURN_BUFFER_BYPASS
- added C5: Murata GRM188R60J106ME47D, Capacitor_SMD:C_0603_1608Metric, symbol Leshy2:RF31_NRF0_MODULE_BULK_CAP
- added C6: TDK C1005X7R1H104K050BB, Capacitor_SMD:C_0402_1005Metric, symbol Leshy2:RF31_NRF0_MODULE_HF_CAP
- added C7: Murata GRM1555C1H121JA01D, Capacitor_SMD:C_0402_1005Metric, symbol Leshy2:RF31_NRF0_DETECTOR_FILTER
- added C8: TDK C1005X7R1H104K050BB, Capacitor_SMD:C_0402_1005Metric, symbol Leshy2:RF31_NRF0_DETECTOR_BYPASS
- added C9: TDK C1005X7R1H104K050BB, Capacitor_SMD:C_0402_1005Metric, symbol Leshy2:RF31_NRF1_HOST_BUFFER_BYPASS
- added D1: Diodes Incorporated BAT54-7-F, Package_TO_SOT_SMD:SOT-23, symbol Leshy2:RF31_NRF_EVIDENCE_HOLD_DIODE
- added J1: GCT RFPC-SMA31-FN-175-A, Leshy2:RFPC-SMA31-FN-175-A, symbol Leshy2:RF31_NRF0_EXTERNAL_SMA
- added J2: GCT RFPC-SMA31-FN-175-A, Leshy2:RFPC-SMA31-FN-175-A, symbol Leshy2:RF31_NRF1_EXTERNAL_SMA
- added J3: GCT RFPC-SMA31-FN-175-A, Leshy2:RFPC-SMA31-FN-175-A, symbol Leshy2:RF31_NRF2_EXTERNAL_SMA
- added J4: Hirose U.FL-R-SMT-1(10), Connector_Coaxial:U.FL_Hirose_U.FL-R-SMT-1_Vertical, symbol Leshy2:RF31_NRF0_RF_BOARD_CONNECTOR
- added J5: Hirose U.FL-R-SMT-1(10), Connector_Coaxial:U.FL_Hirose_U.FL-R-SMT-1_Vertical, symbol Leshy2:RF31_NRF1_RF_BOARD_CONNECTOR
- added J6: Hirose U.FL-R-SMT-1(10), Connector_Coaxial:U.FL_Hirose_U.FL-R-SMT-1_Vertical, symbol Leshy2:RF31_NRF2_RF_BOARD_CONNECTOR
- added R1: Yageo RC0402FR-0710KL, Resistor_SMD:R_0402_1005Metric, symbol Leshy2:RF31_NRF_POWER_ON_PULLDOWN
- added R10: Yageo RC0402FR-0710KL, Resistor_SMD:R_0402_1005Metric, symbol Leshy2:RF31_NRF0_HOST_CSN_PULLUP
- added R11: Yageo RC0402FR-0710KL, Resistor_SMD:R_0402_1005Metric, symbol Leshy2:RF31_NRF0_HOST_SCK_PULLDOWN
- added R12: Yageo RC0402FR-0710KL, Resistor_SMD:R_0402_1005Metric, symbol Leshy2:RF31_NRF0_HOST_MOSI_PULLDOWN
- added R13: Yageo RC0402FR-0710KL, Resistor_SMD:R_0402_1005Metric, symbol Leshy2:RF31_NRF0_HOST_MISO_PULLDOWN
- added R14: Yageo RC0402FR-0710KL, Resistor_SMD:R_0402_1005Metric, symbol Leshy2:RF31_NRF0_HOST_IRQ_PULLUP
- added R15: Yageo RC0402FR-0710KL, Resistor_SMD:R_0402_1005Metric, symbol Leshy2:RF31_NRF0_MODULE_CE_PULLDOWN
- added R16: Yageo RC0402FR-0710KL, Resistor_SMD:R_0402_1005Metric, symbol Leshy2:RF31_NRF0_MODULE_CSN_PULLUP
- added R17: Yageo RC0402FR-0710KL, Resistor_SMD:R_0402_1005Metric, symbol Leshy2:RF31_NRF0_MODULE_SCK_PULLDOWN
- added R18: Yageo RC0402FR-0710KL, Resistor_SMD:R_0402_1005Metric, symbol Leshy2:RF31_NRF0_MODULE_MOSI_PULLDOWN
- added R19: Yageo RC0402FR-0710KL, Resistor_SMD:R_0402_1005Metric, symbol Leshy2:RF31_NRF0_MODULE_MISO_PULLDOWN
- added R2: Yageo RC0402FR-0710KL, Resistor_SMD:R_0402_1005Metric, symbol Leshy2:RF31_NRF_EVIDENCE_HOLD_PULLDOWN
- added R20: Yageo RC0402FR-0710KL, Resistor_SMD:R_0402_1005Metric, symbol Leshy2:RF31_NRF0_MODULE_IRQ_PULLUP
- added R21: Yageo RC0402FR-0749R9L, Resistor_SMD:R_0402_1005Metric, symbol Leshy2:RF31_NRF0_COUPLER_TERMINATION
- added R22: Yageo RC0402FR-0752R3L, Resistor_SMD:R_0402_1005Metric, symbol Leshy2:RF31_NRF0_DETECTOR_MATCH
- added R23: Panasonic ERJ-2RKF22R0X, Resistor_SMD:R_0402_1005Metric, symbol Leshy2:RF31_NRF1_CE_SERIES
- added R24: Panasonic ERJ-2RKF22R0X, Resistor_SMD:R_0402_1005Metric, symbol Leshy2:RF31_NRF1_CSN_SERIES
- added R25: Panasonic ERJ-2RKF22R0X, Resistor_SMD:R_0402_1005Metric, symbol Leshy2:RF31_NRF1_SCK_SERIES
- added R26: Panasonic ERJ-2RKF22R0X, Resistor_SMD:R_0402_1005Metric, symbol Leshy2:RF31_NRF1_MOSI_SERIES
- added R27: Panasonic ERJ-2RKF22R0X, Resistor_SMD:R_0402_1005Metric, symbol Leshy2:RF31_NRF1_MISO_SERIES
- added R28: Panasonic ERJ-2RKF22R0X, Resistor_SMD:R_0402_1005Metric, symbol Leshy2:RF31_NRF1_IRQ_SERIES
- added R29: Yageo RC0402FR-0710KL, Resistor_SMD:R_0402_1005Metric, symbol Leshy2:RF31_NRF1_HOST_CE_PULLDOWN
- added R3: Panasonic ERJ-2RKF22R0X, Resistor_SMD:R_0402_1005Metric, symbol Leshy2:RF31_NRF0_CE_SERIES
- added R30: Yageo RC0402FR-0710KL, Resistor_SMD:R_0402_1005Metric, symbol Leshy2:RF31_NRF1_HOST_CSN_PULLUP
- added R31: Yageo RC0402FR-0710KL, Resistor_SMD:R_0402_1005Metric, symbol Leshy2:RF31_NRF1_HOST_SCK_PULLDOWN
- added R32: Yageo RC0402FR-0710KL, Resistor_SMD:R_0402_1005Metric, symbol Leshy2:RF31_NRF1_HOST_MOSI_PULLDOWN
- added R33: Yageo RC0402FR-0710KL, Resistor_SMD:R_0402_1005Metric, symbol Leshy2:RF31_NRF1_HOST_MISO_PULLDOWN
- added R34: Yageo RC0402FR-0710KL, Resistor_SMD:R_0402_1005Metric, symbol Leshy2:RF31_NRF1_HOST_IRQ_PULLUP
- added R35: Yageo RC0402FR-0710KL, Resistor_SMD:R_0402_1005Metric, symbol Leshy2:RF31_NRF1_MODULE_CE_PULLDOWN
- added R36: Yageo RC0402FR-0710KL, Resistor_SMD:R_0402_1005Metric, symbol Leshy2:RF31_NRF1_MODULE_CSN_PULLUP
- added R37: Yageo RC0402FR-0710KL, Resistor_SMD:R_0402_1005Metric, symbol Leshy2:RF31_NRF1_MODULE_SCK_PULLDOWN
- added R38: Yageo RC0402FR-0710KL, Resistor_SMD:R_0402_1005Metric, symbol Leshy2:RF31_NRF1_MODULE_MOSI_PULLDOWN
- added R39: Yageo RC0402FR-0710KL, Resistor_SMD:R_0402_1005Metric, symbol Leshy2:RF31_NRF1_MODULE_MISO_PULLDOWN
- added R4: Panasonic ERJ-2RKF22R0X, Resistor_SMD:R_0402_1005Metric, symbol Leshy2:RF31_NRF0_CSN_SERIES
- added R40: Yageo RC0402FR-0710KL, Resistor_SMD:R_0402_1005Metric, symbol Leshy2:RF31_NRF1_MODULE_IRQ_PULLUP
- added R41: Yageo RC0402FR-0749R9L, Resistor_SMD:R_0402_1005Metric, symbol Leshy2:RF31_NRF1_COUPLER_TERMINATION
- added R42: Yageo RC0402FR-0752R3L, Resistor_SMD:R_0402_1005Metric, symbol Leshy2:RF31_NRF1_DETECTOR_MATCH
- added R43: Panasonic ERJ-2RKF22R0X, Resistor_SMD:R_0402_1005Metric, symbol Leshy2:RF31_NRF2_CE_SERIES
- added R44: Panasonic ERJ-2RKF22R0X, Resistor_SMD:R_0402_1005Metric, symbol Leshy2:RF31_NRF2_CSN_SERIES
- added R45: Panasonic ERJ-2RKF22R0X, Resistor_SMD:R_0402_1005Metric, symbol Leshy2:RF31_NRF2_SCK_SERIES
- added R46: Panasonic ERJ-2RKF22R0X, Resistor_SMD:R_0402_1005Metric, symbol Leshy2:RF31_NRF2_MOSI_SERIES
- added R47: Panasonic ERJ-2RKF22R0X, Resistor_SMD:R_0402_1005Metric, symbol Leshy2:RF31_NRF2_MISO_SERIES
- added R48: Panasonic ERJ-2RKF22R0X, Resistor_SMD:R_0402_1005Metric, symbol Leshy2:RF31_NRF2_IRQ_SERIES
- added R49: Yageo RC0402FR-0710KL, Resistor_SMD:R_0402_1005Metric, symbol Leshy2:RF31_NRF2_HOST_CE_PULLDOWN
- added R5: Panasonic ERJ-2RKF22R0X, Resistor_SMD:R_0402_1005Metric, symbol Leshy2:RF31_NRF0_SCK_SERIES
- added R50: Yageo RC0402FR-0710KL, Resistor_SMD:R_0402_1005Metric, symbol Leshy2:RF31_NRF2_HOST_CSN_PULLUP
- added R51: Yageo RC0402FR-0710KL, Resistor_SMD:R_0402_1005Metric, symbol Leshy2:RF31_NRF2_HOST_SCK_PULLDOWN
- added R52: Yageo RC0402FR-0710KL, Resistor_SMD:R_0402_1005Metric, symbol Leshy2:RF31_NRF2_HOST_MOSI_PULLDOWN
- added R53: Yageo RC0402FR-0710KL, Resistor_SMD:R_0402_1005Metric, symbol Leshy2:RF31_NRF2_HOST_MISO_PULLDOWN
- added R54: Yageo RC0402FR-0710KL, Resistor_SMD:R_0402_1005Metric, symbol Leshy2:RF31_NRF2_HOST_IRQ_PULLUP
- added R55: Yageo RC0402FR-0710KL, Resistor_SMD:R_0402_1005Metric, symbol Leshy2:RF31_NRF2_MODULE_CE_PULLDOWN
- added R56: Yageo RC0402FR-0710KL, Resistor_SMD:R_0402_1005Metric, symbol Leshy2:RF31_NRF2_MODULE_CSN_PULLUP
- added R57: Yageo RC0402FR-0710KL, Resistor_SMD:R_0402_1005Metric, symbol Leshy2:RF31_NRF2_MODULE_SCK_PULLDOWN
- added R58: Yageo RC0402FR-0710KL, Resistor_SMD:R_0402_1005Metric, symbol Leshy2:RF31_NRF2_MODULE_MOSI_PULLDOWN
- added R59: Yageo RC0402FR-0710KL, Resistor_SMD:R_0402_1005Metric, symbol Leshy2:RF31_NRF2_MODULE_MISO_PULLDOWN
- added R6: Panasonic ERJ-2RKF22R0X, Resistor_SMD:R_0402_1005Metric, symbol Leshy2:RF31_NRF0_MOSI_SERIES
- added R60: Yageo RC0402FR-0710KL, Resistor_SMD:R_0402_1005Metric, symbol Leshy2:RF31_NRF2_MODULE_IRQ_PULLUP
- added R61: Yageo RC0402FR-0749R9L, Resistor_SMD:R_0402_1005Metric, symbol Leshy2:RF31_NRF2_COUPLER_TERMINATION
- added R62: Yageo RC0402FR-0752R3L, Resistor_SMD:R_0402_1005Metric, symbol Leshy2:RF31_NRF2_DETECTOR_MATCH
- added R7: Panasonic ERJ-2RKF22R0X, Resistor_SMD:R_0402_1005Metric, symbol Leshy2:RF31_NRF0_MISO_SERIES
- added R8: Panasonic ERJ-2RKF22R0X, Resistor_SMD:R_0402_1005Metric, symbol Leshy2:RF31_NRF0_IRQ_SERIES
- added R9: Yageo RC0402FR-0710KL, Resistor_SMD:R_0402_1005Metric, symbol Leshy2:RF31_NRF0_HOST_CE_PULLDOWN
- added U1: Ebyte E01-ML01IPX, Leshy2:Ebyte-E01-ML01IPX, symbol Leshy2:RF31_NRF0
- added U10: Nexperia 74LVC126APW,118, Package_SO:TSSOP-14_4.4x5mm_P0.65mm, symbol Leshy2:RF31_NRF2_HOST_BUFFER
- added U11: Nexperia 74LVC2G126DC,125, Package_SO:VSSOP-8_2.3x2mm_P0.5mm, symbol Leshy2:RF31_NRF2_RETURN_BUFFER
- added U12: TTM Technologies DC2337J5010AHF, Leshy2:DC2337J5010AHF, symbol Leshy2:RF31_NRF2_COUPLER
- added U13: Texas Instruments TPS22919DCKR, Package_TO_SOT_SMD:SOT-363_SC-70-6, symbol Leshy2:RF31_NRF_POWER_SWITCH
- added U2: Ebyte E01-ML01IPX, Leshy2:Ebyte-E01-ML01IPX, symbol Leshy2:RF31_NRF1
- added U3: Ebyte E01-ML01IPX, Leshy2:Ebyte-E01-ML01IPX, symbol Leshy2:RF31_NRF2
- added U4: Nexperia 74LVC126APW,118, Package_SO:TSSOP-14_4.4x5mm_P0.65mm, symbol Leshy2:RF31_NRF0_HOST_BUFFER
- added U5: Nexperia 74LVC2G126DC,125, Package_SO:VSSOP-8_2.3x2mm_P0.5mm, symbol Leshy2:RF31_NRF0_RETURN_BUFFER
- added U6: TTM Technologies DC2337J5010AHF, Leshy2:DC2337J5010AHF, symbol Leshy2:RF31_NRF0_COUPLER
- added U7: Nexperia 74LVC126APW,118, Package_SO:TSSOP-14_4.4x5mm_P0.65mm, symbol Leshy2:RF31_NRF1_HOST_BUFFER
- added U8: Nexperia 74LVC2G126DC,125, Package_SO:VSSOP-8_2.3x2mm_P0.5mm, symbol Leshy2:RF31_NRF1_RETURN_BUFFER
- added U9: TTM Technologies DC2337J5010AHF, Leshy2:DC2337J5010AHF, symbol Leshy2:RF31_NRF1_COUPLER
- added W1: TE Connectivity 2118651-2, symbol Leshy2:RF31_NRF0_RF_JUMPER
- added W2: TE Connectivity 2118651-2, symbol Leshy2:RF31_NRF1_RF_JUMPER
- added W3: TE Connectivity 2118651-2, symbol Leshy2:RF31_NRF2_RF_JUMPER
- added X1: Ebyte E01-ML01IPX factory IPEX (nrf0), symbol Leshy2:RF31_NRF0_FACTORY_IPEX
- added X2: Ebyte E01-ML01IPX factory IPEX (nrf1), symbol Leshy2:RF31_NRF1_FACTORY_IPEX
- added X3: Ebyte E01-ML01IPX factory IPEX (nrf2), symbol Leshy2:RF31_NRF2_FACTORY_IPEX
Connections:
- net 3V3_MAIN: now also C1.1 (END_1), R10.2 (END_2), R14.2 (END_2), R30.2 (END_2), R34.2 (END_2), R50.2 (END_2), R54.2 (END_2), U13.1 (IN)
- net AON_SAFE_3V3: now also C14.1 (END_1), C20.1 (END_1), C8.1 (END_1)
- net NRF0_CE_SAFE: now also R9.1 (END_1), U4.2 (1A)
- net NRF0_CSN_N: now also R10.1 (END_1), U4.5 (2A)
- net NRF0_DETECT_FILTER: now also C7.1 (END_1)
- net NRF0_DETECT_V: now also C7.2 (END_2)
- net NRF0_FORWARD_RF_SAMPLE: now also R22.1 (END_1), U6.2 (COUPLED_FWD)
- net NRF0_IRQ_N: now also R14.1 (END_1), R8.2 (END_2)
- net NRF0_MISO: now also R13.1 (END_1), R7.2 (END_2)
- net NRF0_MOSI: now also R12.1 (END_1), U4.12 (4A)
- net NRF0_SCK: now also R11.1 (END_1), U4.9 (3A)
- net NRF1_CE_SAFE: now also R29.1 (END_1), U7.2 (1A)
- net NRF1_CSN_N: now also R30.1 (END_1), U7.5 (2A)
- net NRF1_DETECT_FILTER: now also C13.1 (END_1)
- net NRF1_DETECT_V: now also C13.2 (END_2)
- net NRF1_FORWARD_RF_SAMPLE: now also R42.1 (END_1), U9.2 (COUPLED_FWD)
- net NRF1_IRQ_N: now also R28.2 (END_2), R34.1 (END_1)
- net NRF1_MISO: now also R27.2 (END_2), R33.1 (END_1)
- net NRF1_MOSI: now also R32.1 (END_1), U7.12 (4A)
- net NRF1_SCK: now also R31.1 (END_1), U7.9 (3A)
- net NRF2_CE_SAFE: now also R49.1 (END_1), U10.2 (1A)
- net NRF2_CSN_N: now also R50.1 (END_1), U10.5 (2A)
- net NRF2_DETECT_FILTER: now also C19.1 (END_1)
- net NRF2_DETECT_V: now also C19.2 (END_2)
- net NRF2_FORWARD_RF_SAMPLE: now also R62.1 (END_1), U12.2 (COUPLED_FWD)
- net NRF2_IRQ_N: now also R48.2 (END_2), R54.1 (END_1)
- net NRF2_MISO: now also R47.2 (END_2), R53.1 (END_1)
- net NRF2_MOSI: now also R52.1 (END_1), U10.12 (4A)
- net NRF2_SCK: now also R51.1 (END_1), U10.9 (3A)
- net NRF_EVIDENCE_HOLD: now also C2.1 (END_1), D1.3 (K), R2.1 (END_1)
- net NRF_GROUP_PWR_EN_SAFE: now also D1.1 (A), R1.1 (END_1), U13.3 (ON)
- net POWER_GROUND: now also C1.2 (END_2), C10.2 (END_2), C11.2 (END_2), C12.2 (END_2), C15.2 (END_2), C16.2 (END_2), C17.2 (END_2), C18.2 (END_2), C3.2 (END_2), C4.2 (END_2), C5.2 (END_2), C6.2 (END_2), C9.2 (END_2), J1.2 (GROUND_TOP_LEFT), J1.3 (GROUND_TOP_RIGHT), J1.4 (GROUND_BOTTOM_LEFT), J1.5 (GROUND_BOTTOM_RIGHT), J2.2 (GROUND_TOP_LEFT), J2.3 (GROUND_TOP_RIGHT), J2.4 (GROUND_BOTTOM_LEFT), J2.5 (GROUND_BOTTOM_RIGHT), J3.2 (GROUND_TOP_LEFT), J3.3 (GROUND_TOP_RIGHT), J3.4 (GROUND_BOTTOM_LEFT), J3.5 (GROUND_BOTTOM_RIGHT), J4.2 (SHELL), J5.2 (SHELL), J6.2 (SHELL), R1.2 (END_2), R11.2 (END_2), R12.2 (END_2), R13.2 (END_2), R15.2 (END_2), R17.2 (END_2), R18.2 (END_2), R19.2 (END_2), R21.2 (END_2), R22.2 (END_2), R29.2 (END_2), R31.2 (END_2), R32.2 (END_2), R33.2 (END_2), R35.2 (END_2), R37.2 (END_2), R38.2 (END_2), R39.2 (END_2), R41.2 (END_2), R42.2 (END_2), R49.2 (END_2), R51.2 (END_2), R52.2 (END_2), R53.2 (END_2), R55.2 (END_2), R57.2 (END_2), R58.2 (END_2), R59.2 (END_2), R61.2 (END_2), R62.2 (END_2), R9.2 (END_2), U1.8 (GND), U10.7 (GND), U11.4 (GND), U12.3 (GND_3), U12.4 (GND_4), U13.2 (GND), U2.8 (GND), U3.8 (GND), U4.7 (GND), U5.4 (GND), U6.3 (GND_3), U6.4 (GND_4), U7.7 (GND), U8.4 (GND), U9.3 (GND_3), U9.4 (GND_4)
- net SAFETY_GROUND: now also C14.2 (END_2), C2.2 (END_2), C20.2 (END_2), C8.2 (END_2), R2.2 (END_2)
- new net NRF0_CE_BUFFERED: R3.1 (END_1), U4.3 (1Y)
- new net NRF0_CE_MODULE: R15.1 (END_1), R3.2 (END_2), U1.2 (CE)
- new net NRF0_CSN_BUFFERED_N: R4.1 (END_1), U4.6 (2Y)
- new net NRF0_CSN_MODULE_N: R16.1 (END_1), R4.2 (END_2), U1.3 (CSN)
- new net NRF0_EXTERNAL_RF_50R: J1.1 (RF), U6.6 (RF_OUT)
- new net NRF0_IRQ_BUFFERED_N: R8.1 (END_1), U5.3 (2Y)
- new net NRF0_IRQ_MODULE_N: R20.1 (END_1), U1.7 (IRQ), U5.5 (2A)
- new net NRF0_MISO_BUFFERED: R7.1 (END_1), U5.6 (1Y)
- new net NRF0_MISO_MODULE: R19.1 (END_1), U1.6 (MISO), U5.2 (1A)
- new net NRF0_MODULE_RF_50R: J4.1 (CENTER), U6.1 (RF_IN), W1.A (END_A), W1.B (END_B), X1.1 (FACTORY_IPEX)
- new net NRF0_MOSI_BUFFERED: R6.1 (END_1), U4.11 (4Y)
- new net NRF0_MOSI_MODULE: R18.1 (END_1), R6.2 (END_2), U1.5 (MOSI)
- new net NRF0_REVERSE_ISOLATED_PORT: R21.1 (END_1), U6.5 (ISOLATED_REVERSE)
- new net NRF0_SCK_BUFFERED: R5.1 (END_1), U4.8 (3Y)
- new net NRF0_SCK_MODULE: R17.1 (END_1), R5.2 (END_2), U1.4 (SCK)
- new net NRF1_CE_BUFFERED: R23.1 (END_1), U7.3 (1Y)
- new net NRF1_CE_MODULE: R23.2 (END_2), R35.1 (END_1), U2.2 (CE)
- new net NRF1_CSN_BUFFERED_N: R24.1 (END_1), U7.6 (2Y)
- new net NRF1_CSN_MODULE_N: R24.2 (END_2), R36.1 (END_1), U2.3 (CSN)
- new net NRF1_EXTERNAL_RF_50R: J2.1 (RF), U9.6 (RF_OUT)
- new net NRF1_IRQ_BUFFERED_N: R28.1 (END_1), U8.3 (2Y)
- new net NRF1_IRQ_MODULE_N: R40.1 (END_1), U2.7 (IRQ), U8.5 (2A)
- new net NRF1_MISO_BUFFERED: R27.1 (END_1), U8.6 (1Y)
- new net NRF1_MISO_MODULE: R39.1 (END_1), U2.6 (MISO), U8.2 (1A)
- new net NRF1_MODULE_RF_50R: J5.1 (CENTER), U9.1 (RF_IN), W2.A (END_A), W2.B (END_B), X2.1 (FACTORY_IPEX)
- new net NRF1_MOSI_BUFFERED: R26.1 (END_1), U7.11 (4Y)
- new net NRF1_MOSI_MODULE: R26.2 (END_2), R38.1 (END_1), U2.5 (MOSI)
- new net NRF1_REVERSE_ISOLATED_PORT: R41.1 (END_1), U9.5 (ISOLATED_REVERSE)
- new net NRF1_SCK_BUFFERED: R25.1 (END_1), U7.8 (3Y)
- new net NRF1_SCK_MODULE: R25.2 (END_2), R37.1 (END_1), U2.4 (SCK)
- new net NRF2_CE_BUFFERED: R43.1 (END_1), U10.3 (1Y)
- new net NRF2_CE_MODULE: R43.2 (END_2), R55.1 (END_1), U3.2 (CE)
- new net NRF2_CSN_BUFFERED_N: R44.1 (END_1), U10.6 (2Y)
- new net NRF2_CSN_MODULE_N: R44.2 (END_2), R56.1 (END_1), U3.3 (CSN)
- new net NRF2_EXTERNAL_RF_50R: J3.1 (RF), U12.6 (RF_OUT)
- new net NRF2_IRQ_BUFFERED_N: R48.1 (END_1), U11.3 (2Y)
- new net NRF2_IRQ_MODULE_N: R60.1 (END_1), U11.5 (2A), U3.7 (IRQ)
- new net NRF2_MISO_BUFFERED: R47.1 (END_1), U11.6 (1Y)
- new net NRF2_MISO_MODULE: R59.1 (END_1), U11.2 (1A), U3.6 (MISO)
- new net NRF2_MODULE_RF_50R: J6.1 (CENTER), U12.1 (RF_IN), W3.A (END_A), W3.B (END_B), X3.1 (FACTORY_IPEX)
- new net NRF2_MOSI_BUFFERED: R46.1 (END_1), U10.11 (4Y)
- new net NRF2_MOSI_MODULE: R46.2 (END_2), R58.1 (END_1), U3.5 (MOSI)
- new net NRF2_REVERSE_ISOLATED_PORT: R61.1 (END_1), U12.5 (ISOLATED_REVERSE)
- new net NRF2_SCK_BUFFERED: R45.1 (END_1), U10.8 (3Y)
- new net NRF2_SCK_MODULE: R45.2 (END_2), R57.1 (END_1), U3.4 (SCK)
- new net NRF_QOD: C10.1 (END_1), C11.1 (END_1), C12.1 (END_1), C15.1 (END_1), C16.1 (END_1), C17.1 (END_1), C18.1 (END_1), C3.1 (END_1), C4.1 (END_1), C5.1 (END_1), C6.1 (END_1), C9.1 (END_1), R16.2 (END_2), R20.2 (END_2), R36.2 (END_2), R40.2 (END_2), R56.2 (END_2), R60.2 (END_2), U1.1 (VCC), U10.1 (1OE), U10.10 (3OE), U10.13 (4OE), U10.14 (VCC), U10.4 (2OE), U11.1 (1OE), U11.7 (2OE), U11.8 (VCC), U13.5 (QOD), U13.6 (VOUT), U2.1 (VCC), U3.1 (VCC), U4.1 (1OE), U4.10 (3OE), U4.13 (4OE), U4.14 (VCC), U4.4 (2OE), U5.1 (1OE), U5.7 (2OE), U5.8 (VCC), U7.1 (1OE), U7.10 (3OE), U7.13 (4OE), U7.14 (VCC), U7.4 (2OE), U8.1 (1OE), U8.7 (2OE), U8.8 (VCC)
- no-connect marks 33 -> 2
Other:
- title: (none) -> Leshy2 — three independent full-function nRF24 paths

Commit message: complete H2 schematic review package
Parts:
- renumbered C1 to C31001, C2 to C31002, C3 to C31003, C4 to C31004, C5 to C31005, C6 to C31006, C7 to C31007, C8 to C31008, C9 to C31009, C10 to C31010, C11 to C31011, C12 to C31012, C13 to C31013, C14 to C31014, C15 to C31015, C16 to C31016, C17 to C31017, C18 to C31018, C19 to C31019, C20 to C31020, D1 to D31001, J1 to J31001, J2 to J31002, J3 to J31003, J4 to J31004, J5 to J31005, J6 to J31006, R1 to R31001, R2 to R31002, R3 to R31003, R4 to R31004, R5 to R31005, R6 to R31006, R7 to R31007, R8 to R31008, R9 to R31009, R10 to R31010, R11 to R31011, R12 to R31012, R13 to R31013, R14 to R31014, R15 to R31015, R16 to R31016, R17 to R31017, R18 to R31018, R19 to R31019, R20 to R31020, R21 to R31021, R22 to R31022, R23 to R31023, R24 to R31024, R25 to R31025, R26 to R31026, R27 to R31027, R28 to R31028, R29 to R31029, R30 to R31030, R31 to R31031, R32 to R31032, R33 to R31033, R34 to R31034, R35 to R31035, R36 to R31036, R37 to R31037, R38 to R31038, R39 to R31039, R40 to R31040, R41 to R31041, R42 to R31042, R43 to R31043, R44 to R31044, R45 to R31045, R46 to R31046, R47 to R31047, R48 to R31048, R49 to R31049, R50 to R31050, R51 to R31051, R52 to R31052, R53 to R31053, R54 to R31054, R55 to R31055, R56 to R31056, R57 to R31057, R58 to R31058, R59 to R31059, R60 to R31060, R61 to R31061, R62 to R31062, U1 to U31001, U2 to U31002, U3 to U31003, U4 to U31004, U5 to U31005, U6 to U31006, U7 to U31007, U8 to U31008, U9 to U31009, U10 to U31010, U11 to U31011, U12 to U31012, U13 to U31013, W1 to W31001, W2 to W31002, W3 to W31003, X1 to X31001, X2 to X31002, X3 to X31003

Commit message: review H3.6.2 single-fault containment
Parts:
- added C31021: TDK C1005X7R1H104K050BB, Capacitor_SMD:C_0402_1005Metric, symbol Leshy2:RF31_NRF_BACKUP_GATE_BYPASS
- added U31014: SN74LVC1G08DCKR, Package_TO_SOT_SMD:SOT-353_SC-70-5, symbol Leshy2:RF31_NRF_BACKUP_GATE
Connections:
- net AON_SAFE_3V3: now also C31021.1 (END_1), U31014.5 (VCC)
- net NRF_GROUP_PWR_EN_SAFE: now also U31014.4 (Y)
- net SAFETY_GROUND: now also C31021.2 (END_2), U31014.3 (GND)
- new net FAULT_ASSERT_N: U31014.2 (B)
- new net NRF_GROUP_PWR_EN_PRIMARY: U31014.1 (A)
Other:
- moved on the sheet: X31001, X31002, X31003
Changed lines of the file:
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@@
+	)
+	(symbol
+		(lib_id "Leshy2:RF31_NRF_BACKUP_GATE")
+		(at 574.04 340.36 0)
+		(unit 1)
+		(exclude_from_sim no)
+		(in_bom yes)
+		(on_board yes)
+		(dnp no)
+		(property "Reference" "U31014"
+			(at 574.04 335.28 0)
+			(show_name no)
+			(do_not_autoplace no)
+			(effects (font (size 1.27 1.27)))
+		)
+		(property "Value" "SN74LVC1G08DCKR"
+			(at 574.04 345.44 0)
+			(show_name no)
+			(do_not_autoplace no)
+			(effects (font (size 1.27 1.27)))
+		)
+		(property "Footprint" "Package_TO_SOT_SMD:SOT-353_SC-70-5"
+			(at 574.04 340.36 0)
+			(show_name no)
+			(do_not_autoplace no)
+			(hide yes)
+			(effects (font (size 1.27 1.27)))
+		)
+		(property "Datasheet" "~"
+			(at 574.04 340.36 0)
+			(show_name no)
+			(do_not_autoplace no)
+			(hide yes)
+			(effects (font (size 1.27 1.27)))
+		)
+		(property "Description" "independent FAULT_ASSERT_N nRF rail qualifier"
+			(at 574.04 340.36 0)
+			(show_name no)
+			(do_not_autoplace no)
+			(hide yes)
+			(effects (font (size 1.27 1.27)))
+		)
+		(pin "1"
+		)
+		(pin "2"
+		)
+		(pin "3"
+		)
+		(pin "4"
+		)
+		(pin "5"
+		)
+		(instances
+			(project "LESHY2-RF"
+				(path "/5ff0ce01-98fc-5b57-807d-50b7149d832d"
+					(reference "U31014")
+					(unit 1)
+				)
+			)
+		)
+	)
+	(symbol
+		(lib_id "Leshy2:RF31_NRF_BACKUP_GATE_BYPASS")
+		(at 309.88 341.63 0)
+		(unit 1)
+		(exclude_from_sim no)
+		(in_bom yes)
+		(on_board yes)
+		(dnp no)
+		(property "Reference" "C31021"
+			(at 309.88 336.55 0)
+			(show_name no)
+			(do_not_autoplace no)
+			(effects (font (size 1.27 1.27)))
+		)
+		(property "Value" "TDK C1005X7R1H104K050BB"
+			(at 309.88 346.71 0)
+			(show_name no)
+			(do_not_autoplace no)
+			(effects (font (size 1.27 1.27)))
+		)
+		(property "Footprint" "Capacitor_SMD:C_0402_1005Metric"
+			(at 309.88 341.63 0)
+			(show_name no)
+			(do_not_autoplace no)
+			(hide yes)
+			(effects (font (size 1.27 1.27)))
+		)
+		(property "Datasheet" "~"
+			(at 309.88 341.63 0)
+			(show_name no)
+			(do_not_autoplace no)
+			(hide yes)
+			(effects (font (size 1.27 1.27)))
+		)
+		(property "Description" "100nf_10pct_50v_x7r_0402_converter_hf_input_capacitor"
+			(at 309.88 341.63 0)
+			(show_name no)
+			(do_not_autoplace no)
+			(hide yes)
+			(effects (font (size 1.27 1.27)))
+		)
+		(pin "1"
+		)
+		(pin "2"
+		)
+		(instances
+			(project "LESHY2-RF"
+				(path "/5ff0ce01-98fc-5b57-807d-50b7149d832d"
+					(reference "C31021")
+					(unit 1)
+				)
+			)
+		)
 	)
 	(symbol
 		(lib_id "Leshy2:RF31_NRF0_FACTORY_IPEX")
-		(at 574.04 339.09 0)
+		(at 375.92 341.63 0)
 		(unit 1)
 		(exclude_from_sim no)
@@
 		(dnp no)
 		(property "Reference" "X31001"
-			(at 574.04 334.01 0)
+			(at 375.92 336.55 0)
 			(show_name no)
 			(do_not_autoplace no)
@@
 		)
 		(property "Value" "Ebyte E01-ML01IPX factory IPEX (nrf0)"
-			(at 574.04 344.17 0)
+			(at 375.92 346.71 0)
 			(show_name no)
 			(do_not_autoplace no)
@@
 		)
 		(property "Footprint" ""
-			(at 574.04 339.09 0)
+			(at 375.92 341.63 0)
 			(show_name no)
 			(do_not_autoplace no)
@@
 		)
 		(property "Datasheet" "~"
-			(at 574.04 339.09 0)
+			(at 375.92 341.63 0)
 			(show_name no)
 			(do_not_autoplace no)
@@
 		)
 		(property "Description" "non-PCB factory micro-coax assembly boundary"
-			(at 574.04 339.09 0)
+			(at 375.92 341.63 0)
 			(show_name no)
 			(do_not_autoplace no)
@@
 	(symbol
 		(lib_id "Leshy2:RF31_NRF1_FACTORY_IPEX")
-		(at 309.88 341.63 0)
+		(at 111.76 351.79 0)
 		(unit 1)
 		(exclude_from_sim no)
@@
 		(dnp no)
 		(property "Reference" "X31002"
-			(at 309.88 336.55 0)
+			(at 111.76 346.71 0)
 			(show_name no)
 			(do_not_autoplace no)
@@
 		)
 		(property "Value" "Ebyte E01-ML01IPX factory IPEX (nrf1)"
-			(at 309.88 346.71 0)
+			(at 111.76 356.87 0)
 			(show_name no)
 			(do_not_autoplace no)
@@
 		)
 		(property "Footprint" ""
-			(at 309.88 341.63 0)
+			(at 111.76 351.79 0)
 			(show_name no)
 			(do_not_autoplace no)
@@
 		)
 		(property "Datasheet" "~"
-			(at 309.88 341.63 0)
+			(at 111.76 351.79 0)
 			(show_name no)
 			(do_not_autoplace no)
@@
 		)
 		(property "Description" "non-PCB factory micro-coax assembly boundary"
-			(at 309.88 341.63 0)
+			(at 111.76 351.79 0)
 			(show_name no)
 			(do_not_autoplace no)
@@
 	(symbol
 		(lib_id "Leshy2:RF31_NRF2_FACTORY_IPEX")
-		(at 375.92 341.63 0)
+		(at 177.80 351.79 0)
 		(unit 1)
 		(exclude_from_sim no)
@@
 		(dnp no)
 		(property "Reference" "X31003"
-			(at 375.92 336.55 0)
+			(at 177.80 346.71 0)
 			(show_name no)
 			(do_not_autoplace no)
@@
 		)
 		(property "Value" "Ebyte E01-ML01IPX factory IPEX (nrf2)"
-			(at 375.92 346.71 0)
+			(at 177.80 356.87 0)
 			(show_name no)
 			(do_not_autoplace no)
@@
 		)
 		(property "Footprint" ""
-			(at 375.92 341.63 0)
+			(at 177.80 351.79 0)
 			(show_name no)
 			(do_not_autoplace no)
@@
 		)
 		(property "Datasheet" "~"
-			(at 375.92 341.63 0)
+			(at 177.80 351.79 0)
 			(show_name no)
 			(do_not_autoplace no)
@@
 		)
 		(property "Description" "non-PCB factory micro-coax assembly boundary"
-			(at 375.92 341.63 0)
+			(at 177.80 351.79 0)
 			(show_name no)
 			(do_not_autoplace no)
@@
 		(effects (font (size 1.27 1.27)))
 	)
+	(label "AON_SAFE_3V3"
+		(at 591.82 340.36 180)
+		(effects (font (size 1.27 1.27)) (justify right bottom))
+	)
+	(label "AON_SAFE_3V3"
+		(at 292.10 340.36 0)
+		(effects (font (size 1.27 1.27)))
+	)
+	(hierarchical_label "FAULT_ASSERT_N"
+		(shape bidirectional)
+		(at 556.26 340.36 0)
+		(effects (font (size 1.27 1.27)))
+	)
 	(no_connect (at 160.02 73.66)
 	)
@@
 	)
 	(label "NRF0_MODULE_RF_50R"
-		(at 556.26 337.82 0)
+		(at 358.14 340.36 0)
 		(effects (font (size 1.27 1.27)))
 	)
@@
 	)
 	(label "NRF1_MODULE_RF_50R"
-		(at 292.10 340.36 0)
+		(at 93.98 350.52 0)
 		(effects (font (size 1.27 1.27)))
 	)
@@
 	)
 	(label "NRF2_MODULE_RF_50R"
-		(at 358.14 340.36 0)
+		(at 160.02 350.52 0)
 		(effects (font (size 1.27 1.27)))
 	)
@@
 		(effects (font (size 1.27 1.27)))
 	)
+	(hierarchical_label "NRF_GROUP_PWR_EN_PRIMARY"
+		(shape bidirectional)
+		(at 556.26 337.82 0)
+		(effects (font (size 1.27 1.27)))
+	)
 	(hierarchical_label "NRF_GROUP_PWR_EN_SAFE"
 		(shape bidirectional)
@@
 		(effects (font (size 1.27 1.27)))
 	)
+	(label "NRF_GROUP_PWR_EN_SAFE"
+		(at 591.82 337.82 180)
+		(effects (font (size 1.27 1.27)) (justify right bottom))
+	)
 	(label "NRF_QOD"
 		(at 226.06 43.18 0)
@@
 		(effects (font (size 1.27 1.27)) (justify right bottom))
 	)
+	(label "SAFETY_GROUND"
+		(at 556.26 342.90 0)
+		(effects (font (size 1.27 1.27)))
+	)
+	(label "SAFETY_GROUND"
+		(at 327.66 340.36 180)
+		(effects (font (size 1.27 1.27)) (justify right bottom))
+	)

Commit message: Optimize H1 display and stocked BOM routes
Parts:
- C31003, C31004, C31006, C31008, C31009, C31010, C31012, C31014, C31015, C31016, C31018, C31020, C31021: value TDK C1005X7R1H104K050BB -> Yageo CC0402KRX7R9BB104
- U31005, U31008, U31011: value Nexperia 74LVC2G126DC,125 -> Nexperia 74LVC2G126DP,125; footprint Package_SO:VSSOP-8_2.3x2mm_P0.5mm -> Package_SO:TSSOP-8_3x3mm_P0.65mm
Changed lines of the file:
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@@
 			(effects (font (size 1.27 1.27)))
 		)
-		(property "Value" "Nexperia 74LVC2G126DC,125"
+		(property "Value" "Nexperia 74LVC2G126DP,125"
 			(at 441.96 103.39 0)
 			(show_name no)
@@
 			(effects (font (size 1.27 1.27)))
 		)
-		(property "Footprint" "Package_SO:VSSOP-8_2.3x2mm_P0.5mm"
+		(property "Footprint" "Package_SO:TSSOP-8_3x3mm_P0.65mm"
 			(at 441.96 97.79 0)
 			(show_name no)
@@
 			(effects (font (size 1.27 1.27)))
 		)
-		(property "Value" "TDK C1005X7R1H104K050BB"
+		(property "Value" "Yageo CC0402KRX7R9BB104"
 			(at 508.00 100.33 0)
 			(show_name no)
@@
 			(effects (font (size 1.27 1.27)))
 		)
-		(property "Value" "TDK C1005X7R1H104K050BB"
+		(property "Value" "Yageo CC0402KRX7R9BB104"
 			(at 574.04 100.33 0)
 			(show_name no)
@@
 			(effects (font (size 1.27 1.27)))
 		)
-		(property "Value" "TDK C1005X7R1H104K050BB"
+		(property "Value" "Yageo CC0402KRX7R9BB104"
 			(at 111.76 102.87 0)
 			(show_name no)
@@
 			(effects (font (size 1.27 1.27)))
 		)
-		(property "Value" "TDK C1005X7R1H104K050BB"
+		(property "Value" "Yageo CC0402KRX7R9BB104"
 			(at 508.00 176.53 0)
 			(show_name no)
@@
 			(effects (font (size 1.27 1.27)))
 		)
-		(property "Value" "Nexperia 74LVC2G126DC,125"
+		(property "Value" "Nexperia 74LVC2G126DP,125"
 			(at 45.72 182.13 0)
 			(show_name no)
@@
 			(effects (font (size 1.27 1.27)))
 		)
-		(property "Footprint" "Package_SO:VSSOP-8_2.3x2mm_P0.5mm"
+		(property "Footprint" "Package_SO:TSSOP-8_3x3mm_P0.65mm"
 			(at 45.72 176.53 0)
 			(show_name no)
@@
 			(effects (font (size 1.27 1.27)))
 		)
-		(property "Value" "TDK C1005X7R1H104K050BB"
+		(property "Value" "Yageo CC0402KRX7R9BB104"
 			(at 111.76 179.07 0)
 			(show_name no)
@@
 			(effects (font (size 1.27 1.27)))
 		)
-		(property "Value" "TDK C1005X7R1H104K050BB"
+		(property "Value" "Yageo CC0402KRX7R9BB104"
 			(at 177.80 179.07 0)
 			(show_name no)
@@
 			(effects (font (size 1.27 1.27)))
 		)
-		(property "Value" "TDK C1005X7R1H104K050BB"
+		(property "Value" "Yageo CC0402KRX7R9BB104"
 			(at 441.96 181.61 0)
 			(show_name no)
@@
 			(effects (font (size 1.27 1.27)))
 		)
-		(property "Value" "TDK C1005X7R1H104K050BB"
+		(property "Value" "Yageo CC0402KRX7R9BB104"
 			(at 177.80 255.27 0)
 			(show_name no)
@@
 			(effects (font (size 1.27 1.27)))
 		)
-		(property "Value" "Nexperia 74LVC2G126DC,125"
+		(property "Value" "Nexperia 74LVC2G126DP,125"
 			(at 441.96 260.87 0)
 			(show_name no)
@@
 			(effects (font (size 1.27 1.27)))
 		)
-		(property "Footprint" "Package_SO:VSSOP-8_2.3x2mm_P0.5mm"
+		(property "Footprint" "Package_SO:TSSOP-8_3x3mm_P0.65mm"
 			(at 441.96 255.27 0)
 			(show_name no)
@@
 			(effects (font (size 1.27 1.27)))
 		)
-		(property "Value" "TDK C1005X7R1H104K050BB"
+		(property "Value" "Yageo CC0402KRX7R9BB104"
 			(at 45.72 260.35 0)
 			(show_name no)
@@
 			(effects (font (size 1.27 1.27)))
 		)
-		(property "Value" "TDK C1005X7R1H104K050BB"
+		(property "Value" "Yageo CC0402KRX7R9BB104"
 			(at 243.84 260.35 0)
 			(show_name no)
@@
 			(effects (font (size 1.27 1.27)))
 		)
-		(property "Value" "TDK C1005X7R1H104K050BB"
+		(property "Value" "Yageo CC0402KRX7R9BB104"
 			(at 375.92 270.51 0)
 			(show_name no)
@@
 			(effects (font (size 1.27 1.27)))
 		)
-		(property "Value" "TDK C1005X7R1H104K050BB"
+		(property "Value" "Yageo CC0402KRX7R9BB104"
 			(at 243.84 336.55 0)
 			(show_name no)
@@
 			(effects (font (size 1.27 1.27)))
 		)
-		(property "Value" "TDK C1005X7R1H104K050BB"
+		(property "Value" "Yageo CC0402KRX7R9BB104"
 			(at 309.88 346.71 0)
 			(show_name no)
