File: hardware/ecad/kicad/LESHY2-RF/RF_32_SUBGHZ_VOICE.kicad_sch (KiCad schematic)
At the start: 119 parts, among them J32001 GCT RFPC-SMA31-FN-175-A, J32002 GCT RFPC-SMA31-FN-175-A, Q32001 Diodes Incorporated MMBT3904-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, U32001 CC1101RGPR, U32002 Nexperia 74LVC126APW,118, U32003 Nexperia 74LVC126APW,118, U32004 Nexperia 74LVC2G126DC,125, U32005 TTM Technologies B0310J50100A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, U32006 Infineon BGS13SN8E6327XTSA1, U32007 Infineon BGS13SN8E6327XTSA1, U32008 NiceRF SA518, U32009 TPS3808G33DBVR, U32010 Texas Instruments TPS22919DCKR, U32011 Texas Instruments SN74LVC1G12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, U32012 Texas Instruments SN74LVC1G12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, U32013 SN74LVC1G07DCKR, U32014 Texas Instruments SN74LVC2G66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, U32015 Texas Instruments TPS564252DR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, U32016 Texas Instruments TPS25974LRP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, U32017 Texas Instruments TPS22919DCKR, U32018 SN74LVC1G08DCKR, Y32001 Abracon ABM8-26.000MHZ-10-D-1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

Commit message: Reclose H2 through H4 on dual SA818S architecture
Parts:
- removed C32031: TDK C1005X7R1H104K050BB, Capacitor_SMD:C_0402_1005Metric, symbol Leshy2:RF32_VOICE_PTT_ISO_BYPASS
- removed C32032: TDK C1005X7R1H104K050BB, Capacitor_SMD:C_0402_1005Metric, symbol Leshy2:RF32_VOICE_UART_TX_ISO_BYPASS
- removed C32034: TDK C1005X7R1H104K050BB, Capacitor_SMD:C_0402_1005Metric, symbol Leshy2:RF32_VOICE_AUDIO_ISO_BYPASS
- removed U32011: Texas Instruments SN74LVC1G126DCKR, Package_TO_SOT_SMD:Texas_R-PDSO-G5_DCK-5, symbol Leshy2:RF32_VOICE_PTT_ISO
- removed U32012: Texas Instruments SN74LVC1G126DCKR, Package_TO_SOT_SMD:Texas_R-PDSO-G5_DCK-5, symbol Leshy2:RF32_VOICE_UART_TX_ISO
- removed U32014: Texas Instruments SN74LVC2G66DCUR, Package_SO:VSSOP-8_2.3x2mm_P0.5mm, symbol Leshy2:RF32_VOICE_AUDIO_ISO
- added C32026: Murata GRM1555C1H121JA01D, Capacitor_SMD:C_0402_1005Metric, symbol Leshy2:RF32_VOICE_V_DETECTOR_FILTER
- added C32027: TDK C1005X7R1H104K050BB, Capacitor_SMD:C_0402_1005Metric, symbol Leshy2:RF32_VOICE_V_DETECTOR_BYPASS
- added C32029: TDK C1608X7R1C105K080AC, Capacitor_SMD:C_0603_1608Metric, symbol Leshy2:RF32_VOICE_V_MIC_COUPLING
- added C32034: TDK C1005X7R1H104K050BB, Capacitor_SMD:C_0402_1005Metric, symbol Leshy2:RF32_VOICE_BAND_IO_BYPASS
- added C32035: TDK C1005X7R1H104K050BB, Capacitor_SMD:C_0402_1005Metric, symbol Leshy2:RF32_VOICE_BAND_INVERTER_BYPASS
- added C32036: TDK C1005X7R1H104K050BB, Capacitor_SMD:C_0402_1005Metric, symbol Leshy2:RF32_VOICE_PD_GATE_BYPASS
- added C32037: TDK C1005X7R1H104K050BB, Capacitor_SMD:C_0402_1005Metric, symbol Leshy2:RF32_VOICE_CONTROL_MUX_A_BYPASS
- added C32038: TDK C1005X7R1H104K050BB, Capacitor_SMD:C_0402_1005Metric, symbol Leshy2:RF32_VOICE_CONTROL_MUX_B_BYPASS
- added C32039: TDK C1005X7R1H104K050BB, Capacitor_SMD:C_0402_1005Metric, symbol Leshy2:RF32_VOICE_AUDIO_MUX_BYPASS
- added D32003: Nexperia PESD24VY1BSF, Diode_SMD:Nexperia_DSN0603-2_0.6x0.3mm_P0.4mm, symbol Leshy2:RF32_VOICE_V_RF_ESD
- added J32003: GCT RFPC-SMA31-FN-175-A, Leshy2:RFPC-SMA31-FN-175-A, symbol Leshy2:RF32_VOICE_V_EXTERNAL_SMA
- added R32025: Yageo RC0402FR-075K1L, Resistor_SMD:R_0402_1005Metric, symbol Leshy2:RF32_VOICE_V_DETECTOR_SERIES_ATTENUATOR
- added R32026: Yageo RC0402FR-0752R3L, Resistor_SMD:R_0402_1005Metric, symbol Leshy2:RF32_VOICE_V_DETECTOR_MATCH
- added R32030: Yageo RC0402FR-0710KL, Resistor_SMD:R_0402_1005Metric, symbol Leshy2:RF32_VOICE_BAND_SELECT_PULLDOWN
- added R32031: Yageo RC0402FR-0710KL, Resistor_SMD:R_0402_1005Metric, symbol Leshy2:RF32_VOICE_BAND_P1_PULLDOWN
- added R32032: Yageo RC0402FR-0710KL, Resistor_SMD:R_0402_1005Metric, symbol Leshy2:RF32_VOICE_BAND_P2_PULLDOWN
- added R32033: Yageo RC0402FR-0710KL, Resistor_SMD:R_0402_1005Metric, symbol Leshy2:RF32_VOICE_BAND_P3_PULLDOWN
- added R32034: Yageo RC0402FR-0710KL, Resistor_SMD:R_0402_1005Metric, symbol Leshy2:RF32_VOICE_BAND_P4_PULLDOWN
- added R32035: Yageo RC0402FR-0710KL, Resistor_SMD:R_0402_1005Metric, symbol Leshy2:RF32_VOICE_BAND_P5_PULLDOWN
- added R32036: Yageo RC0402FR-0710KL, Resistor_SMD:R_0402_1005Metric, symbol Leshy2:RF32_VOICE_BAND_P6_PULLDOWN
- added R32037: Yageo RC0402FR-0710KL, Resistor_SMD:R_0402_1005Metric, symbol Leshy2:RF32_VOICE_BAND_P7_PULLDOWN
- added R32039: Yageo RC0402FR-0710KL, Resistor_SMD:R_0402_1005Metric, symbol Leshy2:RF32_VOICE_V_PTT_PULLUP
- added R32041: Yageo RC0402FR-07100KL, Resistor_SMD:R_0402_1005Metric, symbol Leshy2:RF32_VOICE_V_UART_RX_PULLDOWN
- added U32009: G-NiceRF SA818S-V, Leshy2:G-NiceRF-SA818S-Official-Package, symbol Leshy2:RF32_VOICE_V
- added U32012: TCA9534APWR, Package_SO:TSSOP-16_4.4x5mm_P0.65mm, symbol Leshy2:RF32_VOICE_BAND_IO
- added U32013: 74LVC2G14GW,125, Package_TO_SOT_SMD:SOT-363_SC-70-6, symbol Leshy2:RF32_VOICE_BAND_INVERTER
- added U32014: Texas Instruments SN74LVC2G08DCUR, Package_SO:VSSOP-8_2.3x2mm_P0.5mm, symbol Leshy2:RF32_VOICE_PD_GATE
- added U32015: Texas Instruments TMUX1136DGSR, Package_SO:TSSOP-10_3x3mm_P0.5mm, symbol Leshy2:RF32_VOICE_CONTROL_MUX_A
- added U32016: Texas Instruments TMUX1136DGSR, Package_SO:TSSOP-10_3x3mm_P0.5mm, symbol Leshy2:RF32_VOICE_CONTROL_MUX_B
- added U32017: Texas Instruments TMUX1136DGSR, Package_SO:TSSOP-10_3x3mm_P0.5mm, symbol Leshy2:RF32_VOICE_AUDIO_MUX
- U32008: value NiceRF SA518 -> G-NiceRF SA818S-U; footprint Leshy2:NiceRF-SA518-Rev1.1-H5-CONTACT-AXIS-RESERVE -> Leshy2:G-NiceRF-SA818S-Official-Package
- renumbered C32026 to C32028, C32027 to C32030, C32028 to C32031, C32029 to C32032, C32030 to C32033, C32033 to C32040, C32035 to C32041, C32036 to C32042, C32037 to C32043, C32038 to C32044, C32039 to C32045, C32040 to C32046, C32041 to C32047, C32042 to C32048, C32043 to C32049, R32025 to R32027, R32026 to R32028, R32027 to R32029, R32028 to R32038, R32029 to R32040, R32030 to R32042, R32031 to R32043, R32032 to R32044, R32033 to R32045, R32034 to R32046, R32035 to R32047, R32036 to R32048, R32037 to R32049, R32038 to R32050, R32039 to R32051, R32040 to R32052, R32041 to R32053, R32042 to R32054, R32043 to R32055, U32009 to U32010, U32010 to U32011, U32013 to U32018, U32015 to U32019, U32016 to U32020, U32017 to U32021, U32018 to U32022
Connections:
- net 3V3_MAIN: now also C32034.1 (END_1), U32012.16 (VCC), U32012.2 (A1)
- net AON_SAFE_3V3: now also C32027.1 (END_1), C32035.1 (END_1), C32036.1 (END_1), U32013.5 (VCC), U32014.8 (VCC)
- net AUDIO_GROUND: now also C32037.2 (END_2), C32038.2 (END_2), C32039.2 (END_2), R32041.2 (END_2), U32015.3 (GND), U32016.3 (GND), U32017.3 (GND)
- net POWER_GROUND: now also C32034.2 (END_2), D32003.2 (K2), J32003.2 (GROUND_TOP_LEFT), J32003.3 (GROUND_TOP_RIGHT), J32003.4 (GROUND_BOTTOM_LEFT), J32003.5 (GROUND_BOTTOM_RIGHT), R32026.2 (END_2), R32030.2 (END_2), R32031.2 (END_2), R32032.2 (END_2), R32033.2 (END_2), R32034.2 (END_2), R32035.2 (END_2), R32036.2 (END_2), R32037.2 (END_2), U32009.10 (GND_10), U32009.9 (GND_9), U32012.1 (A0), U32012.3 (A2), U32012.8 (GND); no longer U32008.19 (GND_19), U32008.20 (GND_20), U32008.8 (GND_8)
- net SAFETY_GROUND: now also C32027.2 (END_2), C32035.2 (END_2), C32036.2 (END_2), U32013.2 (GND), U32013.3 (2A), U32014.4 (GND)
- net VOICE_AUDIO_ON_N: now also U32016.6 (D2); no longer U32008.18 (AUDIO_ON)
- net VOICE_HL_OPEN_DRAIN: now also U32008.7 (HL), U32009.7 (HL); no longer U32008.12 (HL)
- net VOICE_MIC_SELECTED_MAIN: now also U32017.6 (D2)
- net VOICE_PTT_SAFE_N: now also U32016.10 (D1)
- net VOICE_READY: now also U32014.1 (1A), U32014.5 (2A); no longer U32008.13 (PD)
- net VOICE_UART_RX: now also U32015.6 (D2); no longer U32008.2 (UART_TX)
- net VOICE_UART_TX: now also U32015.10 (D1)
- net VVOICE_4V: now also U32008.8 (VCC), U32009.8 (VCC); no longer U32008.11 (VCC)
- net VVOICE_IO_3V3: now also C32037.1 (END_1), C32038.1 (END_1), C32039.1 (END_1), R32039.1 (END_1), U32015.8 (VDD), U32016.8 (VDD), U32017.8 (VDD)
- net VOICE_U_PTT_N: now reaches U32008.5 (PTT)
- net VOICE_U_PTT_N: now also R32038.2 (END_2), U32016.2 (S1A)
- net VOICE_U_PD: now reaches U32008.6 (PD)
- net VOICE_U_PD: now also U32014.7 (1Y)
- net RX_SA518_AFOUT_LOCAL renamed VOICE_U_UART_RX
- net VOICE_U_UART_RX: now also R32040.1 (END_1), U32015.2 (S1A)
- net VOICE_EXTERNAL_RF_50R renamed VOICE_U_EXTERNAL_RF_50R
- net VOICE_U_EXTERNAL_RF_50R: now also U32008.12 (ANT); no longer U32008.7 (ANT)
- net VOICE_MIC_IN renamed VOICE_U_AUDIO_ON_N
- net VOICE_U_AUDIO_ON_N: now also U32016.4 (S2A); no longer C32028.2 (END_2)
- net VOICE_MIC_SELECTED_ISOLATED renamed VOICE_U_MIC_SELECTED
- net VOICE_U_MIC_SELECTED: now also U32017.4 (S2A)
- net VOICE_PTT_MODULE_N: no longer names the net of U32008.14 (NC_14)
- net VOICE_PTT_MODULE_N: no longer R32038.2 (END_2)
- net VOICE_RF_SAMPLE renamed VOICE_U_RF_SAMPLE
- net VOICE_UART_RX_MODULE renamed RX_VOICE_U_AFOUT_LOCAL
- net RX_VOICE_U_AFOUT_LOCAL: now also U32017.2 (S1A); no longer R32040.1 (END_1)
- net VOICE_UPDATE_FIXTURE renamed VOICE_U_UART_TX
- net VOICE_U_UART_TX: now also U32015.4 (S2A)
- new net RX_VOICE_AFOUT_SELECTED: U32017.10 (D1)
- new net RX_VOICE_V_AFOUT_LOCAL: U32009.3 (AFOUT), U32017.9 (S1B)
- new net SYS_I2C_SCL: U32012.14 (SCL)
- new net SYS_I2C_SDA: U32012.15 (SDA)
- new net SYS_INT_N: U32012.13 (INT_N)
- new net VOICE_BAND_RESERVE_P1: R32031.1 (END_1), U32012.5 (P1)
- new net VOICE_BAND_RESERVE_P2: R32032.1 (END_1), U32012.6 (P2)
- new net VOICE_BAND_RESERVE_P3: R32033.1 (END_1), U32012.7 (P3)
- new net VOICE_BAND_RESERVE_P4: R32034.1 (END_1), U32012.9 (P4)
- new net VOICE_BAND_RESERVE_P5: R32035.1 (END_1), U32012.10 (P5)
- new net VOICE_BAND_RESERVE_P6: R32036.1 (END_1), U32012.11 (P6)
- new net VOICE_BAND_RESERVE_P7: R32037.1 (END_1), U32012.12 (P7)
- new net VOICE_U_MIC_IN: C32028.2 (END_2), U32008.18 (MIC_IN)
- new net VOICE_U_SELECT: U32013.6 (1Y), U32014.2 (1B)
- new net VOICE_V_AUDIO_ON_N: U32009.1 (AUDIO_ON), U32016.7 (S2B)
- new net VOICE_V_DETECT_FILTER: C32026.1 (END_1)
- new net VOICE_V_DETECT_V: C32026.2 (END_2)
- new net VOICE_V_EXTERNAL_RF_50R: D32003.1 (K1), J32003.1 (RF), R32025.1 (END_1), U32009.12 (ANT)
- new net VOICE_V_MIC_IN: C32029.2 (END_2), U32009.18 (MIC_IN)
- new net VOICE_V_MIC_SELECTED: C32029.1 (END_1), U32017.7 (S2B)
- new net VOICE_V_PD: U32009.6 (PD), U32014.3 (2Y)
- new net VOICE_V_PTT_N: R32039.2 (END_2), U32009.5 (PTT), U32016.9 (S1B)
- new net VOICE_V_RF_SAMPLE: R32025.2 (END_2), R32026.1 (END_1)
- new net VOICE_V_SELECT: R32030.1 (END_1), U32012.4 (P0), U32013.1 (1A), U32014.6 (2B), U32015.1 (SEL1), U32015.5 (SEL2), U32016.1 (SEL1), U32016.5 (SEL2), U32017.1 (SEL1), U32017.5 (SEL2)
- new net VOICE_V_UART_RX: R32041.1 (END_1), U32009.16 (UART_RX), U32015.9 (S1B)
- new net VOICE_V_UART_TX: U32009.17 (UART_TX), U32015.7 (S2B)
- no-connect marks 11 -> 20
Other:
- title: Leshy2 — independent CC1101 Sub-GHz data and SA518 voice -> Leshy2 — independent CC1101 data plus one-hot SA818S VHF/UHF voice
- moved on the sheet: C32001, C32002, C32003, C32004, C32005, C32006, C32007, C32008, C32009, C32010, C32011, C32012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

Commit message: Optimize H1 display and stocked BOM routes
Parts:
- C32001, C32002, C32003, C32006, C32007, C32008, C32009, C32010, C32011, C32023, C32025, C32027, C32030, C32034, C32035, C32036, C32037, C32038, C32039, C32040, C32042, C32049: value TDK C1005X7R1H104K050BB -> Yageo CC0402KRX7R9BB104
- U32004: value Nexperia 74LVC2G126DC,125 -> Nexperia 74LVC2G126DP,125; footprint Package_SO:VSSOP-8_2.3x2mm_P0.5mm -> Package_SO:TSSOP-8_3x3mm_P0.65mm
Changed lines of the file:
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@@
 			(effects (font (size 1.27 1.27)))
 		)
-		(property "Value" "Nexperia 74LVC2G126DC,125"
+		(property "Value" "Nexperia 74LVC2G126DP,125"
 			(at 375.92 47.51 0)
 			(show_name no)
@@
 			(effects (font (size 1.27 1.27)))
 		)
-		(property "Footprint" "Package_SO:VSSOP-8_2.3x2mm_P0.5mm"
+		(property "Footprint" "Package_SO:TSSOP-8_3x3mm_P0.65mm"
 			(at 375.92 41.91 0)
 			(show_name no)
@@
 			(effects (font (size 1.27 1.27)))
 		)
-		(property "Value" "TDK C1005X7R1H104K050BB"
+		(property "Value" "Yageo CC0402KRX7R9BB104"
 			(at 431.80 44.45 0)
 			(show_name no)
@@
 			(effects (font (size 1.27 1.27)))
 		)
-		(property "Value" "TDK C1005X7R1H104K050BB"
+		(property "Value" "Yageo CC0402KRX7R9BB104"
 			(at 487.68 44.45 0)
 			(show_name no)
@@
 			(effects (font (size 1.27 1.27)))
 		)
-		(property "Value" "TDK C1005X7R1H104K050BB"
+		(property "Value" "Yageo CC0402KRX7R9BB104"
 			(at 543.56 44.45 0)
 			(show_name no)
@@
 			(effects (font (size 1.27 1.27)))
 		)
-		(property "Value" "TDK C1005X7R1H104K050BB"
+		(property "Value" "Yageo CC0402KRX7R9BB104"
 			(at 543.56 67.31 0)
 			(show_name no)
@@
 			(effects (font (size 1.27 1.27)))
 		)
-		(property "Value" "TDK C1005X7R1H104K050BB"
+		(property "Value" "Yageo CC0402KRX7R9BB104"
 			(at 599.44 67.31 0)
 			(show_name no)
@@
 			(effects (font (size 1.27 1.27)))
 		)
-		(property "Value" "TDK C1005X7R1H104K050BB"
+		(property "Value" "Yageo CC0402KRX7R9BB104"
 			(at 40.64 69.85 0)
 			(show_name no)
@@
 			(effects (font (size 1.27 1.27)))
 		)
-		(property "Value" "TDK C1005X7R1H104K050BB"
+		(property "Value" "Yageo CC0402KRX7R9BB104"
 			(at 96.52 69.85 0)
 			(show_name no)
@@
 			(effects (font (size 1.27 1.27)))
 		)
-		(property "Value" "TDK C1005X7R1H104K050BB"
+		(property "Value" "Yageo CC0402KRX7R9BB104"
 			(at 152.40 69.85 0)
 			(show_name no)
@@
 			(effects (font (size 1.27 1.27)))
 		)
-		(property "Value" "TDK C1005X7R1H104K050BB"
+		(property "Value" "Yageo CC0402KRX7R9BB104"
 			(at 375.92 72.39 0)
 			(show_name no)
@@
 			(effects (font (size 1.27 1.27)))
 		)
-		(property "Value" "TDK C1005X7R1H104K050BB"
+		(property "Value" "Yageo CC0402KRX7R9BB104"
 			(at 320.04 171.45 0)
 			(show_name no)
@@
 			(effects (font (size 1.27 1.27)))
 		)
-		(property "Value" "TDK C1005X7R1H104K050BB"
+		(property "Value" "Yageo CC0402KRX7R9BB104"
 			(at 599.44 184.15 0)
 			(show_name no)
@@
 			(effects (font (size 1.27 1.27)))
 		)
-		(property "Value" "TDK C1005X7R1H104K050BB"
+		(property "Value" "Yageo CC0402KRX7R9BB104"
 			(at 543.56 204.47 0)
 			(show_name no)
@@
 			(effects (font (size 1.27 1.27)))
 		)
-		(property "Value" "TDK C1005X7R1H104K050BB"
+		(property "Value" "Yageo CC0402KRX7R9BB104"
 			(at 599.44 207.01 0)
 			(show_name no)
@@
 			(effects (font (size 1.27 1.27)))
 		)
-		(property "Value" "TDK C1005X7R1H104K050BB"
+		(property "Value" "Yageo CC0402KRX7R9BB104"
 			(at 96.52 229.87 0)
 			(show_name no)
@@
 			(effects (font (size 1.27 1.27)))
 		)
-		(property "Value" "TDK C1005X7R1H104K050BB"
+		(property "Value" "Yageo CC0402KRX7R9BB104"
 			(at 96.52 252.73 0)
 			(show_name no)
@@
 			(effects (font (size 1.27 1.27)))
 		)
-		(property "Value" "TDK C1005X7R1H104K050BB"
+		(property "Value" "Yageo CC0402KRX7R9BB104"
 			(at 152.40 255.27 0)
 			(show_name no)
@@
 			(effects (font (size 1.27 1.27)))
 		)
-		(property "Value" "TDK C1005X7R1H104K050BB"
+		(property "Value" "Yageo CC0402KRX7R9BB104"
 			(at 375.92 260.35 0)
 			(show_name no)
@@
 			(effects (font (size 1.27 1.27)))
 		)
-		(property "Value" "TDK C1005X7R1H104K050BB"
+		(property "Value" "Yageo CC0402KRX7R9BB104"
 			(at 320.04 262.89 0)
 			(show_name no)
@@
 			(effects (font (size 1.27 1.27)))
 		)
-		(property "Value" "TDK C1005X7R1H104K050BB"
+		(property "Value" "Yageo CC0402KRX7R9BB104"
 			(at 487.68 267.97 0)
 			(show_name no)
@@
 			(effects (font (size 1.27 1.27)))
 		)
-		(property "Value" "TDK C1005X7R1H104K050BB"
+		(property "Value" "Yageo CC0402KRX7R9BB104"
 			(at 320.04 285.75 0)
 			(show_name no)
@@
 			(effects (font (size 1.27 1.27)))
 		)
-		(property "Value" "TDK C1005X7R1H104K050BB"
+		(property "Value" "Yageo CC0402KRX7R9BB104"
 			(at 96.52 298.45 0)
 			(show_name no)
@@
 			(effects (font (size 1.27 1.27)))
 		)
-		(property "Value" "TDK C1005X7R1H104K050BB"
+		(property "Value" "Yageo CC0402KRX7R9BB104"
 			(at 40.64 344.17 0)
 			(show_name no)
