File: hardware/ecad/kicad/LESHY2-RF/RF_50_TX_SAFETY_EVIDENCE.kicad_sch (KiCad schematic)
At the start: 0 parts

Commit message: complete exact H2.3.1 RF power hierarchy
Connections:
- no-connect marks 0 -> 63

Commit message: complete exact H2.3.12 RF TX safety sheet
Parts:
- added C1: TDK C1608X7R1C105K080AC, Capacitor_SMD:C_0603_1608Metric, symbol Leshy2:RF50_CC_EVIDENCE_HOLD_CAP
- added C10: TDK C1005X7R1H104K050BB, Capacitor_SMD:C_0402_1005Metric, symbol Leshy2:RF50_SAFETY_WATCHDOG_BYPASS
- added C11: TDK C1005X7R1H104K050BB, Capacitor_SMD:C_0402_1005Metric, symbol Leshy2:RF50_SAFE_RUN_FAULT_ISO_BYPASS
- added C12: TDK C1005X7R1H104K050BB, Capacitor_SMD:C_0402_1005Metric, symbol Leshy2:RF50_SAFE_SUPERVISOR_BYPASS
- added C13: TDK C1005X7R1H104K050BB, Capacitor_SMD:C_0402_1005Metric, symbol Leshy2:RF50_SAFE_CONDITIONER_BYPASS
- added C14: TDK C1005X7R1H104K050BB, Capacitor_SMD:C_0402_1005Metric, symbol Leshy2:RF50_SAFE_LATCH_BYPASS
- added C15: TDK C1005X7R1H104K050BB, Capacitor_SMD:C_0402_1005Metric, symbol Leshy2:RF50_SAFE_RESET_BUFFER_BYPASS
- added C16: TDK C1005X7R1H104K050BB, Capacitor_SMD:C_0402_1005Metric, symbol Leshy2:RF50_SAFE_GATE_A_BYPASS
- added C17: TDK C1005X7R1H104K050BB, Capacitor_SMD:C_0402_1005Metric, symbol Leshy2:RF50_SAFE_GATE_B_BYPASS
- added C18: TDK C1005X7R1H104K050BB, Capacitor_SMD:C_0402_1005Metric, symbol Leshy2:RF50_SAFE_PTT_OR_BYPASS
- added C19: TDK C1005X7R1H104K050BB, Capacitor_SMD:C_0402_1005Metric, symbol Leshy2:RF50_EVIDENCE_CMP_B_BYPASS
- added C2: TDK C1608X7R1C105K080AC, Capacitor_SMD:C_0603_1608Metric, symbol Leshy2:RF50_VOICE_EVIDENCE_HOLD_CAP
- added C20: TDK C1005X7R1H104K050BB, Capacitor_SMD:C_0402_1005Metric, symbol Leshy2:RF50_EVIDENCE_CMP_VOICE_BYPASS
- added C21: TDK C1005X7R1H104K050BB, Capacitor_SMD:C_0402_1005Metric, symbol Leshy2:RF50_EVIDENCE_MASK_BYPASS
- added C22: TDK C1005X7R1H104K050BB, Capacitor_SMD:C_0402_1005Metric, symbol Leshy2:RF50_EVIDENCE_MAIN_ISOLATOR_BYPASS
- added C3: TDK C1005X7R1H104K050BB, Capacitor_SMD:C_0402_1005Metric, symbol Leshy2:RF50_POWER_COMMAND_FILTER
- added C4: TDK C1005X7R1H104K050BB, Capacitor_SMD:C_0402_1005Metric, symbol Leshy2:RF50_RUN_LOOP_FILTER
- added C5: Murata GRM188R60J106ME47D, Capacitor_SMD:C_0603_1608Metric, symbol Leshy2:RF50_SAFETY_CONTROLLER_BULK
- added C6: TDK C1005X7R1H104K050BB, Capacitor_SMD:C_0402_1005Metric, symbol Leshy2:RF50_SAFETY_CONTROLLER_BYPASS
- added C7: Murata GRM155R71H103KA88D, Capacitor_SMD:C_0402_1005Metric, symbol Leshy2:RF50_SAFETY_CONTROLLER_RESET_CAP
- added C8: TDK C1005X7R1H104K050BB, Capacitor_SMD:C_0402_1005Metric, symbol Leshy2:RF50_SAFETY_FAULT_REQUEST_ISO_BYPASS
- added C9: TDK C1005X7R1H104K050BB, Capacitor_SMD:C_0402_1005Metric, symbol Leshy2:RF50_SAFETY_S3_RESET_ISO_BYPASS
- added D1: Diodes Incorporated BAT54-7-F, Package_TO_SOT_SMD:SOT-23, symbol Leshy2:RF50_CC_EVIDENCE_HOLD_DIODE
- added D2: Diodes Incorporated BAT54-7-F, Package_TO_SOT_SMD:SOT-23, symbol Leshy2:RF50_VOICE_EVIDENCE_HOLD_DIODE
- added D3: Texas Instruments TPD4E05U06DQAR, Package_SON:USON-10_2.5x1.0mm_P0.5mm, symbol Leshy2:RF50_SAFETY_CONTROL_ESD
- added D4: BAT54ALT1G, Package_TO_SOT_SMD:SOT-23, symbol Leshy2:RF50_EVIDENCE_OR_0
- added D5: BAT54ALT1G, Package_TO_SOT_SMD:SOT-23, symbol Leshy2:RF50_EVIDENCE_OR_1
- added D6: BAT54ALT1G, Package_TO_SOT_SMD:SOT-23, symbol Leshy2:RF50_EVIDENCE_OR_2
- added D7: BAT54ALT1G, Package_TO_SOT_SMD:SOT-23, symbol Leshy2:RF50_EVIDENCE_OR_3
- added D8: BAT54ALT1G, Package_TO_SOT_SMD:SOT-23, symbol Leshy2:RF50_EVIDENCE_OR_4
- added Q1: Diodes Incorporated 2N7002DW-7-F, Package_TO_SOT_SMD:SOT-363_SC-70-6, symbol Leshy2:RF50_SAFE_RESET_SINK_B
- added R1: Yageo RC0402FR-0710KL, Resistor_SMD:R_0402_1005Metric, symbol Leshy2:RF50_CC_EVIDENCE_HOLD_PULLDOWN
- added R10: Yageo RC0402FR-0710KL, Resistor_SMD:R_0402_1005Metric, symbol Leshy2:RF50_SAFETY_WATCHDOG_WDI_PULLDOWN
- added R11: Yageo RC0402FR-0710KL, Resistor_SMD:R_0402_1005Metric, symbol Leshy2:RF50_SAFETY_WATCHDOG_MR_PULLUP
- added R12: Yageo RC0402FR-0710KL, Resistor_SMD:R_0402_1005Metric, symbol Leshy2:RF50_FAULT_ASSERT_PULLUP
- added R13: Yageo RC0402FR-0710KL, Resistor_SMD:R_0402_1005Metric, symbol Leshy2:RF50_SAFE_LATCH_D_PULLDOWN
- added R14: Yageo RC0402FR-0710KL, Resistor_SMD:R_0402_1005Metric, symbol Leshy2:RF50_SAFE_RESET_GATE_PULLUP
- added R15: Yageo RC0402FR-0710KL, Resistor_SMD:R_0402_1005Metric, symbol Leshy2:RF50_EVIDENCE_MASK_SCL_PULLUP
- added R16: Yageo RC0402FR-0710KL, Resistor_SMD:R_0402_1005Metric, symbol Leshy2:RF50_EVIDENCE_MASK_SDA_PULLUP
- added R17: Yageo RC0402FR-0710KL, Resistor_SMD:R_0402_1005Metric, symbol Leshy2:RF50_EVIDENCE_MASK_P11_PULLDOWN
- added R18: Yageo RC0402FR-0710KL, Resistor_SMD:R_0402_1005Metric, symbol Leshy2:RF50_EVIDENCE_MASK_P12_PULLDOWN
- added R19: Yageo RC0402FR-0710KL, Resistor_SMD:R_0402_1005Metric, symbol Leshy2:RF50_EVIDENCE_MASK_P13_PULLDOWN
- added R2: Yageo RC0402FR-0710KL, Resistor_SMD:R_0402_1005Metric, symbol Leshy2:RF50_VOICE_EVIDENCE_HOLD_PULLDOWN
- added R20: Yageo RC0402FR-0710KL, Resistor_SMD:R_0402_1005Metric, symbol Leshy2:RF50_EVIDENCE_MASK_P14_PULLDOWN
- added R21: Yageo RC0402FR-0710KL, Resistor_SMD:R_0402_1005Metric, symbol Leshy2:RF50_EVIDENCE_MASK_P15_PULLDOWN
- added R22: Yageo RC0402FR-0710KL, Resistor_SMD:R_0402_1005Metric, symbol Leshy2:RF50_EVIDENCE_MASK_P16_PULLDOWN
- added R23: Yageo RC0402FR-0710KL, Resistor_SMD:R_0402_1005Metric, symbol Leshy2:RF50_EVIDENCE_MASK_P17_PULLDOWN
- added R24: Yageo RC0402FR-07100KL, Resistor_SMD:R_0402_1005Metric, symbol Leshy2:RF50_NRF0_EVIDENCE_THRESHOLD_TOP
- added R25: Yageo RC0402FR-0710KL, Resistor_SMD:R_0402_1005Metric, symbol Leshy2:RF50_NRF0_EVIDENCE_THRESHOLD_BOTTOM
- added R26: Yageo RC0402FR-071ML, Resistor_SMD:R_0402_1005Metric, symbol Leshy2:RF50_NRF0_EVIDENCE_HYSTERESIS
- added R27: Yageo RC0402FR-0710KL, Resistor_SMD:R_0402_1005Metric, symbol Leshy2:RF50_NRF0_EVIDENCE_OUTPUT_PULLUP
- added R28: Yageo RC0402FR-07100KL, Resistor_SMD:R_0402_1005Metric, symbol Leshy2:RF50_NRF1_EVIDENCE_THRESHOLD_TOP
- added R29: Yageo RC0402FR-0710KL, Resistor_SMD:R_0402_1005Metric, symbol Leshy2:RF50_NRF1_EVIDENCE_THRESHOLD_BOTTOM
- added R3: Yageo RC0402FR-0747KL, Resistor_SMD:R_0402_1005Metric, symbol Leshy2:RF50_POWER_COMMAND_PULLUP
- added R30: Yageo RC0402FR-071ML, Resistor_SMD:R_0402_1005Metric, symbol Leshy2:RF50_NRF1_EVIDENCE_HYSTERESIS
- added R31: Yageo RC0402FR-0710KL, Resistor_SMD:R_0402_1005Metric, symbol Leshy2:RF50_NRF1_EVIDENCE_OUTPUT_PULLUP
- added R32: Yageo RC0402FR-07100KL, Resistor_SMD:R_0402_1005Metric, symbol Leshy2:RF50_NRF2_EVIDENCE_THRESHOLD_TOP
- added R33: Yageo RC0402FR-0710KL, Resistor_SMD:R_0402_1005Metric, symbol Leshy2:RF50_NRF2_EVIDENCE_THRESHOLD_BOTTOM
- added R34: Yageo RC0402FR-071ML, Resistor_SMD:R_0402_1005Metric, symbol Leshy2:RF50_NRF2_EVIDENCE_HYSTERESIS
- added R35: Yageo RC0402FR-0710KL, Resistor_SMD:R_0402_1005Metric, symbol Leshy2:RF50_NRF2_EVIDENCE_OUTPUT_PULLUP
- added R36: Yageo RC0402FR-07100KL, Resistor_SMD:R_0402_1005Metric, symbol Leshy2:RF50_CC_EVIDENCE_THRESHOLD_TOP
- added R37: Yageo RC0402FR-0710KL, Resistor_SMD:R_0402_1005Metric, symbol Leshy2:RF50_CC_EVIDENCE_THRESHOLD_BOTTOM
- added R38: Yageo RC0402FR-071ML, Resistor_SMD:R_0402_1005Metric, symbol Leshy2:RF50_CC_EVIDENCE_HYSTERESIS
- added R39: Yageo RC0402FR-0710KL, Resistor_SMD:R_0402_1005Metric, symbol Leshy2:RF50_CC_EVIDENCE_OUTPUT_PULLUP
- added R4: Yageo RC0402FR-0710KL, Resistor_SMD:R_0402_1005Metric, symbol Leshy2:RF50_RUN_LOOP_PULLUP
- added R40: Yageo RC0402FR-07100KL, Resistor_SMD:R_0402_1005Metric, symbol Leshy2:RF50_VOICE_EVIDENCE_THRESHOLD_TOP
- added R41: Yageo RC0402FR-0710KL, Resistor_SMD:R_0402_1005Metric, symbol Leshy2:RF50_VOICE_EVIDENCE_THRESHOLD_BOTTOM
- added R42: Yageo RC0402FR-071ML, Resistor_SMD:R_0402_1005Metric, symbol Leshy2:RF50_VOICE_EVIDENCE_HYSTERESIS
- added R43: Yageo RC0402FR-0710KL, Resistor_SMD:R_0402_1005Metric, symbol Leshy2:RF50_VOICE_EVIDENCE_OUTPUT_PULLUP
- added R44: Yageo RC0402FR-0710KL, Resistor_SMD:R_0402_1005Metric, symbol Leshy2:RF50_ANY_TX_AON_PULLUP
- added R5: Yageo RC0402FR-0710KL, Resistor_SMD:R_0402_1005Metric, symbol Leshy2:RF50_POWER_FAULT_PULLUP
- added R6: Yageo RC0402FR-0710KL, Resistor_SMD:R_0402_1005Metric, symbol Leshy2:RF50_SAFE_POR_PULLUP
- added R7: Yageo RC0402FR-0747KL, Resistor_SMD:R_0402_1005Metric, symbol Leshy2:RF50_SAFETY_CONTROLLER_RESET_PULLUP
- added R8: Yageo RC0402FR-0710KL, Resistor_SMD:R_0402_1005Metric, symbol Leshy2:RF50_SAFETY_FAULT_REQUEST_PULLDOWN
- added R9: Yageo RC0402FR-0710KL, Resistor_SMD:R_0402_1005Metric, symbol Leshy2:RF50_SAFETY_WATCHDOG_WDO_PULLUP
- added SW1: C&K JS102011SCQN, Leshy2:JS102011SCQN, symbol Leshy2:RF50_POWER_COMMAND_SWITCH
- added U1: TPS3808G33DBVR, Package_TO_SOT_SMD:SOT-23-6, symbol Leshy2:RF50_SAFE_SUPERVISOR
- added U10: SN74LVC08APWR, Package_SO:TSSOP-14_4.4x5mm_P0.65mm, symbol Leshy2:RF50_SAFE_GATE_A
- added U11: SN74LVC08APWR, Package_SO:TSSOP-14_4.4x5mm_P0.65mm, symbol Leshy2:RF50_SAFE_GATE_B
- added U12: 74LVC1G32GV,125, Package_TO_SOT_SMD:SOT-353_SC-70-5, symbol Leshy2:RF50_SAFE_PTT_OR
- added U13: Analog Devices AD8314ACPZ-RL7, Package_CSP:LFCSP-8-1EP_3x2mm_P0.5mm_EP1.6x1.65mm, symbol Leshy2:RF50_DET_NRF0
- added U14: Analog Devices AD8314ACPZ-RL7, Package_CSP:LFCSP-8-1EP_3x2mm_P0.5mm_EP1.6x1.65mm, symbol Leshy2:RF50_DET_NRF1
- added U15: Analog Devices AD8314ACPZ-RL7, Package_CSP:LFCSP-8-1EP_3x2mm_P0.5mm_EP1.6x1.65mm, symbol Leshy2:RF50_DET_NRF2
- added U16: Analog Devices AD8314ACPZ-RL7, Package_CSP:LFCSP-8-1EP_3x2mm_P0.5mm_EP1.6x1.65mm, symbol Leshy2:RF50_DET_CC
- added U17: Analog Devices AD8314ACPZ-RL7, Package_CSP:LFCSP-8-1EP_3x2mm_P0.5mm_EP1.6x1.65mm, symbol Leshy2:RF50_DET_VOICE
- added U18: TLV1824PWR, Package_SO:TSSOP-14_4.4x5mm_P0.65mm, symbol Leshy2:RF50_EVIDENCE_CMP_B
- added U19: TLV1821DCKR, Package_TO_SOT_SMD:SOT-353_SC-70-5, symbol Leshy2:RF50_EVIDENCE_CMP_VOICE
- added U2: Texas Instruments MSPM0C1106SDGS20R, Package_SO:Texas_DGS0020A_TSSOP-20_3x5.1mm_P0.5mm, symbol Leshy2:RF50_SAFETY_CONTROLLER
- added U20: TCA9535PWR, Package_SO:TSSOP-24_4.4x7.8mm_P0.65mm, symbol Leshy2:RF50_EVIDENCE_MASK
- added U21: SN74LVC3G07DCUR, Package_SO:VSSOP-8_2.3x2mm_P0.5mm, symbol Leshy2:RF50_EVIDENCE_MAIN_ISOLATOR
- added U3: SN74LVC1G07DCKR, Package_TO_SOT_SMD:SOT-353_SC-70-5, symbol Leshy2:RF50_SAFETY_FAULT_REQUEST_ISO
- added U4: SN74LVC1G07DCKR, Package_TO_SOT_SMD:SOT-353_SC-70-5, symbol Leshy2:RF50_SAFETY_S3_RESET_ISO
- added U5: Texas Instruments TPS3435CAKAGDDFR, Package_TO_SOT_SMD:Texas_DDF0008A_SOT-8_1.6x2.9mm_P0.65mm, symbol Leshy2:RF50_SAFETY_WATCHDOG
- added U6: SN74LVC1G07DCKR, Package_TO_SOT_SMD:SOT-353_SC-70-5, symbol Leshy2:RF50_SAFE_RUN_FAULT_ISO
- added U7: 74LVC2G14GW,125, Package_TO_SOT_SMD:SOT-363_SC-70-6, symbol Leshy2:RF50_SAFE_CONDITIONER
- added U8: SN74LVC1G74DCUR, Package_SO:VSSOP-8_2.3x2mm_P0.5mm, symbol Leshy2:RF50_SAFE_LATCH
- added U9: Texas Instruments SN74LVC1G06DCKR, Package_TO_SOT_SMD:SOT-353_SC-70-5, symbol Leshy2:RF50_SAFE_RESET_BUFFER
Connections:
- net 3V3_MAIN: now also R14.1 (END_1), R5.1 (END_1)
- net AON_PG_N: now also U1.3 (MR_N)
- net AON_SAFE_3V3: now also C10.1 (END_1), C11.1 (END_1), C12.1 (END_1), C13.1 (END_1), C14.1 (END_1), C15.1 (END_1), C16.1 (END_1), C17.1 (END_1), C18.1 (END_1), C19.1 (END_1), C20.1 (END_1), C21.1 (END_1), C22.1 (END_1), C5.1 (END_1), C6.1 (END_1), C8.1 (END_1), C9.1 (END_1), R11.1 (END_1), R12.1 (END_1), R15.1 (END_1), R16.1 (END_1), R24.1 (END_1), R27.1 (END_1), R28.1 (END_1), R31.1 (END_1), R32.1 (END_1), R35.1 (END_1), R36.1 (END_1), R39.1 (END_1), R4.1 (END_1), R40.1 (END_1), R43.1 (END_1), R44.1 (END_1), R6.1 (END_1), R7.1 (END_1), R9.1 (END_1), U1.5 (SENSE), U1.6 (VDD), U10.14 (VCC), U11.14 (VCC), U12.5 (VCC), U13.8 (VPOS), U14.8 (VPOS), U15.8 (VPOS), U16.8 (VPOS), U17.8 (VPOS), U18.3 (VPLUS), U19.5 (VPLUS), U2.6 (VDD), U20.24 (VCC), U21.8 (VCC), U3.5 (VCC), U4.5 (VCC), U5.6 (WD_EN), U5.8 (VDD), U6.5 (VCC), U7.5 (VCC), U8.8 (VCC), U9.5 (VCC)
- net C5_RF_TX_EVIDENCE_N: now also U21.7 (1Y)
- net CC_DETECT_FILTER: now also U16.4 (FLTR)
- net CC_DETECT_V: now also U16.3 (VSET), U16.6 (V_UP), U18.10 (IN4_N)
- net CC_PWR_EN: now also U11.1 (1A)
- net CC_PWR_EN_SAFE: now also D1.1 (A), U11.3 (1Y)
- net CC_RF_SAMPLE: now also U16.1 (RFIN)
- net EV_N0_S3: now also D4.1 (K1), U20.4 (P00)
- net EV_N1_C5: now also D4.2 (K2), U20.5 (P01), U21.1 (1A)
- net EV_N2_NRF0: now also D5.1 (K1), R26.1 (END_1), R27.2 (END_2), U18.2 (OUT1), U20.6 (P02)
- net EV_N3_NRF1: now also D5.2 (K2), R30.1 (END_1), R31.2 (END_2), U18.1 (OUT2), U20.7 (P03)
- net EV_N4_NRF2: now also D6.1 (K1), R34.1 (END_1), R35.2 (END_2), U18.14 (OUT3), U20.8 (P04)
- net EV_N5_CC: now also D6.2 (K2), R38.1 (END_1), R39.2 (END_2), U18.13 (OUT4), U20.9 (P05)
- net EV_N6_VOICE: now also D7.1 (K1), R42.1 (END_1), R43.2 (END_2), U19.1 (OUT), U20.10 (P06)
- net EV_N7_IR: now also D7.2 (K2), U20.11 (P07), U21.3 (2A)
- net EV_N8_LORA_EXT: now also D8.1 (K1), U20.13 (P10)
- net EXT_ANY_5V_EN_SAFE: now also U11.11 (4Y)
- net EXT_ANY_5V_REQ: now also U11.12 (4A)
- net FAULT_LATCH_SENSE_AON: now also U12.2 (1B), U8.5 (Q)
- net IR_TX_EVIDENCE_N: now also U21.5 (2Y)
- net NRF0_CE_REQ: now also U10.1 (1A)
- net NRF0_CE_SAFE: now also U10.3 (1Y)
- net NRF0_DETECT_FILTER: now also U13.4 (FLTR)
- net NRF0_DETECT_V: now also U13.3 (VSET), U13.6 (V_UP), U18.4 (IN1_N)
- net NRF0_FORWARD_RF_SAMPLE: now also U13.1 (RFIN)
- net NRF1_CE_REQ: now also U10.4 (2A)
- net NRF1_CE_SAFE: now also U10.6 (2Y)
- net NRF1_DETECT_FILTER: now also U14.4 (FLTR)
- net NRF1_DETECT_V: now also U14.3 (VSET), U14.6 (V_UP), U18.6 (IN2_N)
- net NRF1_FORWARD_RF_SAMPLE: now also U14.1 (RFIN)
- net NRF2_CE_REQ: now also U10.9 (3A)
- net NRF2_CE_SAFE: now also U10.8 (3Y)
- net NRF2_DETECT_FILTER: now also U15.4 (FLTR)
- net NRF2_DETECT_V: now also U15.3 (VSET), U15.6 (V_UP), U18.8 (IN3_N)
- net NRF2_FORWARD_RF_SAMPLE: now also U15.1 (RFIN)
- net NRF_EVIDENCE_HOLD: now also U13.2 (ENBL), U14.2 (ENBL), U15.2 (ENBL)
- net NRF_GROUP_PWR_EN: now also U10.12 (4A)
- net NRF_GROUP_PWR_EN_SAFE: now also U10.11 (4Y)
- net PACK_ADMISSION_VDD: now also R3.1 (END_1)
- net POR_N: now also R6.2 (END_2), U1.1 (RESET_N), U8.6 (CLR_N)
- net POWER_COMMAND_OFF_N: now also C3.1 (END_1), R3.2 (END_2), SW1.3 (THROW_B)
- net POWER_FAULT_N: now also R5.2 (END_2), U2.3 (PA30)
- net POWER_GROUND: now also C3.2 (END_2), SW1.2 (COMMON)
- net POWER_ZONE_TEMP_ADC: now also U2.1 (PA26)
- net RF_RESET_KILL_GATE: now also Q1.2 (G1), R14.2 (END_2), U9.4 (Y)
- net RF_ZONE_TEMP_ADC: now also U2.2 (PA27)
- net RP_ANY_TX_N: now also U21.2 (3Y)
- net RP_RESET_N: now also Q1.4 (D1)
- net RUN_PERMIT: now also U10.10 (3B), U10.13 (4B), U10.2 (1B), U10.5 (2B), U11.13 (4B), U11.2 (1B), U11.5 (2B), U8.3 (Q_N), U9.2 (A)
- net S3_RESET_KILL_GATE: now also U7.4 (2Y)
- net SAFETY_GROUND: now also C1.2 (END_2), C10.2 (END_2), C11.2 (END_2), C12.2 (END_2), C13.2 (END_2), C14.2 (END_2), C15.2 (END_2), C16.2 (END_2), C17.2 (END_2), C18.2 (END_2), C19.2 (END_2), C2.2 (END_2), C20.2 (END_2), C21.2 (END_2), C22.2 (END_2), C4.2 (END_2), C5.2 (END_2), C6.2 (END_2), C7.2 (END_2), C8.2 (END_2), C9.2 (END_2), Q1.3 (S1), Q1.5 (G2), Q1.6 (S2), R1.2 (END_2), R10.2 (END_2), R13.2 (END_2), R17.2 (END_2), R18.2 (END_2), R19.2 (END_2), R2.2 (END_2), R20.2 (END_2), R21.2 (END_2), R22.2 (END_2), R23.2 (END_2), R25.2 (END_2), R29.2 (END_2), R33.2 (END_2), R37.2 (END_2), R41.2 (END_2), R8.2 (END_2), U1.2 (GND), U10.7 (GND), U11.10 (3B), U11.7 (GND), U11.9 (3A), U12.3 (GND), U13.5 (COMM), U13.9 (EPAD), U14.5 (COMM), U14.9 (EPAD), U15.5 (COMM), U15.9 (EPAD), U16.5 (COMM), U16.9 (EPAD), U17.5 (COMM), U17.9 (EPAD), U18.12 (VMINUS), U19.2 (VMINUS), U2.7 (VSS), U20.12 (GND), U20.2 (A1), U20.21 (A0), U20.3 (A2), U21.4 (GND), U3.3 (GND), U4.3 (GND), U5.1 (SET0), U5.4 (GND), U5.5 (SET1), U6.3 (GND), U7.2 (GND), U8.4 (GND), U9.3 (GND)
- net SYS_I2C_SCL: now also U2.11 (PA11)
- net SYS_I2C_SDA: now also U2.4 (PA0)
- net UI_ZONE_TEMP_ADC: now also U2.12 (PA16)
- net VOICE_DETECT_FILTER: now also U17.4 (FLTR)
- net VOICE_DETECT_V: now also U17.3 (VSET), U17.6 (V_UP), U19.4 (IN_N)
- net VOICE_DOMAIN_EN_SAFE: now also D2.1 (A), U11.6 (2Y)
- net VOICE_DOMAIN_REQ: now also U11.4 (2A)
- net VOICE_PTT_REQ_N: now also U12.1 (1A)
- net VOICE_PTT_SAFE_N: now also U12.4 (1Y)
- net VOICE_RF_SAMPLE: now also U17.1 (RFIN)
- new net ANY_TX_AON_N: D4.3 (A_COMMON), D5.3 (A_COMMON), D6.3 (A_COMMON), D7.3 (A_COMMON), D8.3 (A_COMMON), R44.2 (END_2), U2.17 (PA22), U21.6 (3A)
- new net CC_EVIDENCE_HOLD: C1.1 (END_1), D1.3 (K), R1.1 (END_1), U16.2 (ENBL)
- new net EVIDENCE_MASK_INT_N_TP: U20.1 (INT_N)
- new net EVIDENCE_MASK_UNUSED_P11: R17.1 (END_1), U20.14 (P11)
- new net EVIDENCE_MASK_UNUSED_P12: R18.1 (END_1), U20.15 (P12)
- new net EVIDENCE_MASK_UNUSED_P13: R19.1 (END_1), U20.16 (P13)
- new net EVIDENCE_MASK_UNUSED_P14: R20.1 (END_1), U20.17 (P14)
- new net EVIDENCE_MASK_UNUSED_P15: R21.1 (END_1), U20.18 (P15)
- new net EVIDENCE_MASK_UNUSED_P16: R22.1 (END_1), U20.19 (P16)
- new net EVIDENCE_MASK_UNUSED_P17: R23.1 (END_1), U20.20 (P17)
- new net EV_THRESH_2_NRF0: R24.2 (END_2), R25.1 (END_1), R26.2 (END_2), U18.5 (IN1_P)
- new net EV_THRESH_3_NRF1: R28.2 (END_2), R29.1 (END_1), R30.2 (END_2), U18.7 (IN2_P)
- new net EV_THRESH_4_NRF2: R32.2 (END_2), R33.1 (END_1), R34.2 (END_2), U18.9 (IN3_P)
- new net EV_THRESH_5_CC: R36.2 (END_2), R37.1 (END_1), R38.2 (END_2), U18.11 (IN4_P)
- new net EV_THRESH_6_VOICE: R40.2 (END_2), R41.1 (END_1), R42.2 (END_2), U19.3 (IN_P)
- new net FAULT_ASSERT_N: R12.2 (END_2), R9.2 (END_2), U3.4 (Y), U4.4 (Y), U5.7 (WDO_N), U6.4 (Y), U7.3 (2A), U8.7 (PRE_N)
- new net RUN_EDGE: U2.19 (PA24), U6.2 (A), U7.6 (1Y), U8.1 (CLK)
- new net RUN_LOOP_RAW: C4.1 (END_1), D3.1 (D1_PLUS), R4.2 (END_2), SW1.1 (THROW_A), U7.1 (1A)
- new net S3_FAULT_RESET_REQUEST: U2.18 (PA23), U4.2 (A)
- new net SAFETY_CONTROLLER_NRST_N: C7.1 (END_1), R7.2 (END_2), U2.5 (PA1_NRST)
- new net SAFETY_ESD_GROUND: D3.3 (GND_3), D3.8 (GND_8)
- new net SAFETY_EVIDENCE_I2C_SCL: R15.2 (END_2), U2.8 (PA2), U20.22 (SCL)
- new net SAFETY_EVIDENCE_I2C_SDA: R16.2 (END_2), U2.9 (PA4), U20.23 (SDA)
- new net SAFETY_FAULT_REQUEST: R8.1 (END_1), U2.20 (PA25), U3.2 (A)
- new net SAFETY_SERVICE_UART_RX: U2.14 (PA18)
- new net SAFETY_SERVICE_UART_TX: U2.13 (PA17)
- new net SAFETY_SWCLK: U2.16 (PA20_SWCLK)
- new net SAFETY_SWDIO: U2.15 (PA19_SWDIO)
- new net SAFETY_WATCHDOG_MR_N: R11.2 (END_2), U5.2 (MR_N)
- new net SAFETY_WATCHDOG_WDI: R10.1 (END_1), U2.10 (PA6), U5.3 (WDI)
- new net SAFE_D_LOW: R13.1 (END_1), U8.2 (D)
- new net VOICE_EVIDENCE_HOLD: C2.1 (END_1), D2.3 (K), R2.1 (END_1), U17.2 (ENBL)
- no-connect marks 63 -> 22
Other:
- title: (none) -> Leshy2 — exact RF-side TX interlock and physical evidence

Commit message: complete exact H2.3.13 RF testpoint sheet
Changed lines of the file:
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@@
 		(effects (font (size 1.27 1.27)))
 	)
-	(label "ANY_TX_AON_N"
+	(hierarchical_label "ANY_TX_AON_N"
+		(shape bidirectional)
 		(at 543.56 78.74 180)
 		(effects (font (size 1.27 1.27)) (justify right bottom))
@@
 		(effects (font (size 1.27 1.27)))
 	)
-	(label "EVIDENCE_MASK_INT_N_TP"
+	(hierarchical_label "EVIDENCE_MASK_INT_N_TP"
+		(shape bidirectional)
 		(at 27.94 190.50 0)
 		(effects (font (size 1.27 1.27)))
@@
 		(effects (font (size 1.27 1.27)) (justify right bottom))
 	)
-	(label "SAFETY_CONTROLLER_NRST_N"
+	(hierarchical_label "SAFETY_CONTROLLER_NRST_N"
+		(shape bidirectional)
 		(at 508.00 73.66 0)
 		(effects (font (size 1.27 1.27)))
@@
 		(effects (font (size 1.27 1.27)) (justify right bottom))
 	)
-	(label "SAFETY_SERVICE_UART_RX"
+	(hierarchical_label "SAFETY_SERVICE_UART_RX"
+		(shape bidirectional)
 		(at 543.56 71.12 180)
 		(effects (font (size 1.27 1.27)) (justify right bottom))
 	)
-	(label "SAFETY_SERVICE_UART_TX"
+	(hierarchical_label "SAFETY_SERVICE_UART_TX"
+		(shape bidirectional)
 		(at 543.56 68.58 180)
 		(effects (font (size 1.27 1.27)) (justify right bottom))
 	)
-	(label "SAFETY_SWCLK"
+	(hierarchical_label "SAFETY_SWCLK"
+		(shape bidirectional)
 		(at 543.56 76.20 180)
 		(effects (font (size 1.27 1.27)) (justify right bottom))
 	)
-	(label "SAFETY_SWDIO"
+	(hierarchical_label "SAFETY_SWDIO"
+		(shape bidirectional)
 		(at 543.56 73.66 180)
 		(effects (font (size 1.27 1.27)) (justify right bottom))

Commit message: complete H2 schematic review package
Parts:
- renumbered C1 to C50001, C2 to C50002, C3 to C50003, C4 to C50004, C5 to C50005, C6 to C50006, C7 to C50007, C8 to C50008, C9 to C50009, C10 to C50010, C11 to C50011, C12 to C50012, C13 to C50013, C14 to C50014, C15 to C50015, C16 to C50016, C17 to C50017, C18 to C50018, C19 to C50019, C20 to C50020, C21 to C50021, C22 to C50022, D1 to D50001, D2 to D50002, D3 to D50003, D4 to D50004, D5 to D50005, D6 to D50006, D7 to D50007, D8 to D50008, Q1 to Q50001, R1 to R50001, R2 to R50002, R3 to R50003, R4 to R50004, R5 to R50005, R6 to R50006, R7 to R50007, R8 to R50008, R9 to R50009, R10 to R50010, R11 to R50011, R12 to R50012, R13 to R50013, R14 to R50014, R15 to R50015, R16 to R50016, R17 to R50017, R18 to R50018, R19 to R50019, R20 to R50020, R21 to R50021, R22 to R50022, R23 to R50023, R24 to R50024, R25 to R50025, R26 to R50026, R27 to R50027, R28 to R50028, R29 to R50029, R30 to R50030, R31 to R50031, R32 to R50032, R33 to R50033, R34 to R50034, R35 to R50035, R36 to R50036, R37 to R50037, R38 to R50038, R39 to R50039, R40 to R50040, R41 to R50041, R42 to R50042, R43 to R50043, R44 to R50044, SW1 to SW50001, U1 to U50001, U2 to U50002, U3 to U50003, U4 to U50004, U5 to U50005, U6 to U50006, U7 to U50007, U8 to U50008, U9 to U50009, U10 to U50010, U11 to U50011, U12 to U50012, U13 to U50013, U14 to U50014, U15 to U50015, U16 to U50016, U17 to U50017, U18 to U50018, U19 to U50019, U20 to U50020, U21 to U50021

Commit message: Complete H3.2 power transition verification
Parts:
- removed R50013: Yageo RC0402FR-0710KL, Resistor_SMD:R_0402_1005Metric, symbol Leshy2:RF50_SAFE_LATCH_D_PULLDOWN
- added C50014: Murata GRM21BR71E225KE11L, Capacitor_SMD:C_0805_2012Metric, symbol Leshy2:RF50_SAFE_REARM_DELAY_CAP
- added C50015: TDK C1005X7R1H104K050BB, Capacitor_SMD:C_0402_1005Metric, symbol Leshy2:RF50_SAFE_REARM_BUFFER_BYPASS
- added R50013: Yageo RC0402FR-07100KL, Resistor_SMD:R_0402_1005Metric, symbol Leshy2:RF50_SAFE_REARM_DELAY_RES
- added R50014: Yageo RC0402FR-0710KL, Resistor_SMD:R_0402_1005Metric, symbol Leshy2:RF50_SAFE_LATCH_D_PULLUP
- added U50008: SN74LVC1G17DCKR, Package_TO_SOT_SMD:SOT-353_SC-70-5, symbol Leshy2:RF50_SAFE_REARM_BUFFER
- renumbered C50014 to C50016, C50015 to C50017, C50016 to C50018, C50017 to C50019, C50018 to C50020, C50019 to C50021, C50020 to C50022, C50021 to C50023, C50022 to C50024, R50014 to R50015, R50015 to R50016, R50016 to R50017, R50017 to R50018, R50018 to R50019, R50019 to R50020, R50020 to R50021, R50021 to R50022, R50022 to R50023, R50023 to R50024, R50024 to R50025, R50025 to R50026, R50026 to R50027, R50027 to R50028, R50028 to R50029, R50029 to R50030, R50030 to R50031, R50031 to R50032, R50032 to R50033, R50033 to R50034, R50034 to R50035, R50035 to R50036, R50036 to R50037, R50037 to R50038, R50038 to R50039, R50039 to R50040, R50040 to R50041, R50041 to R50042, R50042 to R50043, R50043 to R50044, R50044 to R50045, U50008 to U50009, U50009 to U50010, U50010 to U50011, U50011 to U50012, U50012 to U50013, U50013 to U50014, U50014 to U50015, U50015 to U50016, U50016 to U50017, U50017 to U50018, U50018 to U50019, U50019 to U50020, U50020 to U50021, U50021 to U50022
Connections:
- net AON_SAFE_3V3: now also U50009.7 (PRE_N), C50015.1 (END_1), R50014.1 (END_1), U50008.5 (VCC)
- net FAULT_ASSERT_N: now also U50012.10 (3B); no longer U50009.7 (PRE_N)
- net FAULT_LATCH_SENSE_AON: now also U50009.3 (Q_N); no longer U50009.5 (Q)
- net POR_N: now also U50012.9 (3A); no longer U50009.6 (CLR_N)
- net RUN_EDGE: now also R50013.1 (END_1); no longer U50009.1 (CLK)
- net RUN_PERMIT: now also U50009.5 (Q); no longer U50009.3 (Q_N)
- net SAFETY_GROUND: now also C50014.2 (END_2), C50015.2 (END_2), U50008.3 (GND); no longer U50012.10 (3B), U50012.9 (3A)
- net SAFE_CLEAR_N: now reaches U50012.8 (3Y)
- net SAFE_CLEAR_N: now also U50009.6 (CLR_N)
- net SAFE_D_LOW renamed SAFE_D_HIGH
- net SAFE_D_HIGH: now also R50014.2 (END_2)
- new net SAFE_REARM_CLK: U50008.4 (Y), U50009.1 (CLK)
- new net SAFE_REARM_DELAY: C50014.1 (END_1), R50013.2 (END_2), U50008.1 (A)
Other:
- moved on the sheet: C50016, C50017, C50018, C50019, C50020, C50021, C50022, C50023, C50024, D50004, D50005, D50006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

Commit message: review H3.6.2 single-fault containment
Parts:
- removed R50018: Yageo RC0402FR-0710KL, Resistor_SMD:R_0402_1005Metric, symbol Leshy2:RF50_EVIDENCE_MASK_P11_PULLDOWN
- added C50018: TDK C1005X7R1H104K050BB, Capacitor_SMD:C_0402_1005Metric, symbol Leshy2:RF50_SAFE_FAULT_RESET_BUFFER_BYPASS
- added R50013: Yageo RC0402FR-071ML, Resistor_SMD:R_0402_1005Metric, symbol Leshy2:RF50_FAULT_ASSERT_BACKUP_PULLDOWN
- added R50019: Yageo RC0402FR-07100KL, Resistor_SMD:R_0402_1005Metric, symbol Leshy2:RF50_FAULT_ASSERT_SENSE_SERIES
- added U50011: SN74LVC3G07DCUR, Package_SO:VSSOP-8_2.3x2mm_P0.5mm, symbol Leshy2:RF50_SAFE_FAULT_RESET_BUFFER
- renumbered C50018 to C50019, C50019 to C50020, C50020 to C50021, C50021 to C50022, C50022 to C50023, C50023 to C50024, C50024 to C50025, R50013 to R50014, R50014 to R50015, R50015 to R50016, R50016 to R50017, R50017 to R50018, R50019 to R50020, R50020 to R50021, R50021 to R50022, R50022 to R50023, R50023 to R50024, R50024 to R50025, R50025 to R50026, R50026 to R50027, R50027 to R50028, R50028 to R50029, R50029 to R50030, R50030 to R50031, R50031 to R50032, R50032 to R50033, R50033 to R50034, R50034 to R50035, R50035 to R50036, R50036 to R50037, R50037 to R50038, R50038 to R50039, R50039 to R50040, R50040 to R50041, R50041 to R50042, R50042 to R50043, R50043 to R50044, R50044 to R50045, R50045 to R50046, U50011 to U50012, U50012 to U50013, U50013 to U50014, U50014 to U50015, U50015 to U50016, U50016 to U50017, U50017 to U50018, U50018 to U50019, U50019 to U50020, U50020 to U50021, U50021 to U50022, U50022 to U50023
Connections:
- net AON_SAFE_3V3: now also C50018.1 (END_1), U50011.8 (VCC)
- net CC_PWR_EN_SAFE: no longer U50013.3 (1Y)
- net FAULT_ASSERT_N: now also R50013.1 (END_1), R50019.1 (END_1), U50011.1 (1A), U50011.2 (3Y), U50011.3 (2A)
- net POWER_COMMAND_OFF_N: now also U50011.6 (3A)
- net RP_RESET_N: now also U50011.7 (1Y)
- net SAFETY_GROUND: now also C50018.2 (END_2), R50013.2 (END_2), U50011.4 (GND)
- net EVIDENCE_MASK_UNUSED_P11 renamed FAULT_ASSERT_SENSE
- net FAULT_ASSERT_SENSE: now also R50019.2 (END_2)
- net NRF_GROUP_PWR_EN_SAFE renamed NRF_GROUP_PWR_EN_PRIMARY
- new net CC_PWR_EN_PRIMARY: U50013.3 (1Y)
- new net VOICE_EFUSE_BACKUP_EN_N: U50011.5 (2Y)
Other:
- moved on the sheet: C50011, C50012, C50013, C50014, C50015, C50016, C50017, C50019, C50020, C50021, C50022, C50023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

Commit message: Reclose H2 through H4 on dual SA818S architecture
Parts:
- added C50003: TDK C1608X7R1C105K080AC, Capacitor_SMD:C_0603_1608Metric, symbol Leshy2:RF50_VOICE_V_EVIDENCE_HOLD_CAP
- added C50025: TDK C1005X7R1H104K050BB, Capacitor_SMD:C_0402_1005Metric, symbol Leshy2:RF50_EVIDENCE_CMP_VOICE_V_BYPASS
- added D50003: Diodes Incorporated BAT54-7-F, Package_TO_SOT_SMD:SOT-23, symbol Leshy2:RF50_VOICE_V_EVIDENCE_HOLD_DIODE
- added R50003: Yageo RC0402FR-0710KL, Resistor_SMD:R_0402_1005Metric, symbol Leshy2:RF50_VOICE_V_EVIDENCE_HOLD_PULLDOWN
- added R50047: Yageo RC0402FR-07100KL, Resistor_SMD:R_0402_1005Metric, symbol Leshy2:RF50_VOICE_V_EVIDENCE_THRESHOLD_TOP
- added R50048: Yageo RC0402FR-0710KL, Resistor_SMD:R_0402_1005Metric, symbol Leshy2:RF50_VOICE_V_EVIDENCE_THRESHOLD_BOTTOM
- added R50049: Yageo RC0402FR-071ML, Resistor_SMD:R_0402_1005Metric, symbol Leshy2:RF50_VOICE_V_EVIDENCE_HYSTERESIS
- added U50020: Analog Devices AD8314ACPZ-RL7, Package_CSP:LFCSP-8-1EP_3x2mm_P0.5mm_EP1.6x1.65mm, symbol Leshy2:RF50_DET_VOICE_V
- added U50023: TLV1821DCKR, Package_TO_SOT_SMD:SOT-353_SC-70-5, symbol Leshy2:RF50_EVIDENCE_CMP_VOICE_V
- renumbered C50003 to C50004, C50004 to C50005, C50005 to C50006, C50006 to C50007, C50007 to C50008, C50008 to C50009, C50009 to C50010, C50010 to C50011, C50011 to C50012, C50012 to C50013, C50013 to C50014, C50014 to C50015, C50015 to C50016, C50016 to C50017, C50017 to C50018, C50018 to C50019, C50019 to C50020, C50020 to C50021, C50021 to C50022, C50022 to C50023, C50023 to C50024, C50024 to C50026, C50025 to C50027, D50003 to D50004, D50004 to D50005, D50005 to D50006, D50006 to D50007, D50007 to D50008, D50008 to D50009, R50003 to R50004, R50004 to R50005, R50005 to R50006, R50006 to R50007, R50007 to R50008, R50008 to R50009, R50009 to R50010, R50010 to R50011, R50011 to R50012, R50012 to R50013, R50013 to R50014, R50014 to R50015, R50015 to R50016, R50016 to R50017, R50017 to R50018, R50018 to R50019, R50019 to R50020, R50020 to R50021, R50021 to R50022, R50022 to R50023, R50023 to R50024, R50024 to R50025, R50025 to R50026, R50026 to R50027, R50027 to R50028, R50028 to R50029, R50029 to R50030, R50030 to R50031, R50031 to R50032, R50032 to R50033, R50033 to R50034, R50034 to R50035, R50035 to R50036, R50036 to R50037, R50037 to R50038, R50038 to R50039, R50039 to R50040, R50040 to R50041, R50041 to R50042, R50042 to R50043, R50043 to R50044, R50044 to R50045, R50045 to R50046, R50046 to R50050, U50020 to U50021, U50021 to U50022, U50022 to U50024, U50023 to U50025
Connections:
- net AON_SAFE_3V3: now also C50025.1 (END_1), R50047.1 (END_1), U50020.8 (VPOS), U50023.5 (VPLUS)
- net EV_N6_VOICE: now also R50049.1 (END_1), U50023.1 (OUT)
- net SAFETY_GROUND: now also C50003.2 (END_2), C50025.2 (END_2), R50003.2 (END_2), R50048.2 (END_2), U50020.5 (COMM), U50020.9 (EPAD), U50023.2 (VMINUS)
- net VOICE_DOMAIN_EN_SAFE: now also D50003.1 (A)
- net VOICE_RF_SAMPLE renamed VOICE_U_RF_SAMPLE
- new net EV_THRESH_6_VOICE_V: R50047.2 (END_2), R50048.1 (END_1), R50049.2 (END_2), U50023.3 (IN_P)
- new net VOICE_V_DETECT_FILTER: U50020.4 (FLTR)
- new net VOICE_V_DETECT_V: U50020.3 (VSET), U50020.6 (V_UP), U50023.4 (IN_N)
- new net VOICE_V_EVIDENCE_HOLD: C50003.1 (END_1), D50003.3 (K), R50003.1 (END_1), U50020.2 (ENBL)
- new net VOICE_V_RF_SAMPLE: U50020.1 (RFIN)
- no-connect marks 22 -> 24
Other:
- moved on the sheet: C50004, C50005, C50006, C50007, C50008, C50009, C50010, C50011, C50012, C50013, C50014, C50015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

Commit message: Optimize H1 display and stocked BOM routes
Parts:
- C50004, C50005, C50007, C50009, C50010, C50011, C50012, C50013, C50014, C50016, C50017, C50018, C50019, C50020, C50021, C50022, C50023, C50024, C50025, C50026, C50027: value TDK C1005X7R1H104K050BB -> Yageo CC0402KRX7R9BB104
Changed lines of the file:
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@@
 			(effects (font (size 1.27 1.27)))
 		)
-		(property "Value" "TDK C1005X7R1H104K050BB"
+		(property "Value" "Yageo CC0402KRX7R9BB104"
 			(at 251.46 69.85 0)
 			(show_name no)
@@
 			(effects (font (size 1.27 1.27)))
 		)
-		(property "Value" "TDK C1005X7R1H104K050BB"
+		(property "Value" "Yageo CC0402KRX7R9BB104"
 			(at 388.62 69.85 0)
 			(show_name no)
@@
 			(effects (font (size 1.27 1.27)))
 		)
-		(property "Value" "TDK C1005X7R1H104K050BB"
+		(property "Value" "Yageo CC0402KRX7R9BB104"
 			(at 251.46 92.71 0)
 			(show_name no)
@@
 			(effects (font (size 1.27 1.27)))
 		)
-		(property "Value" "TDK C1005X7R1H104K050BB"
+		(property "Value" "Yageo CC0402KRX7R9BB104"
 			(at 525.78 95.25 0)
 			(show_name no)
@@
 			(effects (font (size 1.27 1.27)))
 		)
-		(property "Value" "TDK C1005X7R1H104K050BB"
+		(property "Value" "Yageo CC0402KRX7R9BB104"
 			(at 182.88 115.57 0)
 			(show_name no)
@@
 			(effects (font (size 1.27 1.27)))
 		)
-		(property "Value" "TDK C1005X7R1H104K050BB"
+		(property "Value" "Yageo CC0402KRX7R9BB104"
 			(at 320.04 115.57 0)
 			(show_name no)
@@
 			(effects (font (size 1.27 1.27)))
 		)
-		(property "Value" "TDK C1005X7R1H104K050BB"
+		(property "Value" "Yageo CC0402KRX7R9BB104"
 			(at 182.88 138.43 0)
 			(show_name no)
@@
 			(effects (font (size 1.27 1.27)))
 		)
-		(property "Value" "TDK C1005X7R1H104K050BB"
+		(property "Value" "Yageo CC0402KRX7R9BB104"
 			(at 320.04 138.43 0)
 			(show_name no)
@@
 			(effects (font (size 1.27 1.27)))
 		)
-		(property "Value" "TDK C1005X7R1H104K050BB"
+		(property "Value" "Yageo CC0402KRX7R9BB104"
 			(at 457.20 138.43 0)
 			(show_name no)
@@
 			(effects (font (size 1.27 1.27)))
 		)
-		(property "Value" "TDK C1005X7R1H104K050BB"
+		(property "Value" "Yageo CC0402KRX7R9BB104"
 			(at 45.72 148.59 0)
 			(show_name no)
@@
 			(effects (font (size 1.27 1.27)))
 		)
-		(property "Value" "TDK C1005X7R1H104K050BB"
+		(property "Value" "Yageo CC0402KRX7R9BB104"
 			(at 182.88 161.29 0)
 			(show_name no)
@@
 			(effects (font (size 1.27 1.27)))
 		)
-		(property "Value" "TDK C1005X7R1H104K050BB"
+		(property "Value" "Yageo CC0402KRX7R9BB104"
 			(at 388.62 163.83 0)
 			(show_name no)
@@
 			(effects (font (size 1.27 1.27)))
 		)
-		(property "Value" "TDK C1005X7R1H104K050BB"
+		(property "Value" "Yageo CC0402KRX7R9BB104"
 			(at 594.36 163.83 0)
 			(show_name no)
@@
 			(effects (font (size 1.27 1.27)))
 		)
-		(property "Value" "TDK C1005X7R1H104K050BB"
+		(property "Value" "Yageo CC0402KRX7R9BB104"
 			(at 320.04 184.15 0)
 			(show_name no)
@@
 			(effects (font (size 1.27 1.27)))
 		)
-		(property "Value" "TDK C1005X7R1H104K050BB"
+		(property "Value" "Yageo CC0402KRX7R9BB104"
 			(at 388.62 186.69 0)
 			(show_name no)
@@
 			(effects (font (size 1.27 1.27)))
 		)
-		(property "Value" "TDK C1005X7R1H104K050BB"
+		(property "Value" "Yageo CC0402KRX7R9BB104"
 			(at 114.30 189.23 0)
 			(show_name no)
@@
 			(effects (font (size 1.27 1.27)))
 		)
-		(property "Value" "TDK C1005X7R1H104K050BB"
+		(property "Value" "Yageo CC0402KRX7R9BB104"
 			(at 525.78 222.25 0)
 			(show_name no)
@@
 			(effects (font (size 1.27 1.27)))
 		)
-		(property "Value" "TDK C1005X7R1H104K050BB"
+		(property "Value" "Yageo CC0402KRX7R9BB104"
 			(at 457.20 222.25 0)
 			(show_name no)
@@
 			(effects (font (size 1.27 1.27)))
 		)
-		(property "Value" "TDK C1005X7R1H104K050BB"
+		(property "Value" "Yageo CC0402KRX7R9BB104"
 			(at 45.72 227.33 0)
 			(show_name no)
@@
 			(effects (font (size 1.27 1.27)))
 		)
-		(property "Value" "TDK C1005X7R1H104K050BB"
+		(property "Value" "Yageo CC0402KRX7R9BB104"
 			(at 388.62 240.03 0)
 			(show_name no)
@@
 			(effects (font (size 1.27 1.27)))
 		)
-		(property "Value" "TDK C1005X7R1H104K050BB"
+		(property "Value" "Yageo CC0402KRX7R9BB104"
 			(at 457.20 267.97 0)
 			(show_name no)
