File: hardware/ecad/kicad/LESHY2-RF/RF_01_USB_PD_CHARGE.kicad_sch (KiCad schematic)
At the start: 0 parts

Commit message: complete exact H2.3.1 RF power hierarchy
Connections:
- no-connect marks 0 -> 10
Changed lines of the file:
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@@
 	(generator_version "10.0")
 	(paper "A4")
+	(hierarchical_label "AON_BUCK_EN"
+		(shape bidirectional)
+		(at 20.32 20.32 0)
+		(effects (font (size 1.27 1.27)))
+	)
+	(wire
+		(pts (xy 20.32 20.32) (xy 25.40 20.32))
+		(stroke (width 0) (type default))
+	)
+	(no_connect (at 25.40 20.32)
+	)
+	(hierarchical_label "AON_SAFE_3V3"
+		(shape bidirectional)
+		(at 20.32 25.40 0)
+		(effects (font (size 1.27 1.27)))
+	)
+	(wire
+		(pts (xy 20.32 25.40) (xy 25.40 25.40))
+		(stroke (width 0) (type default))
+	)
+	(no_connect (at 25.40 25.40)
+	)
+	(hierarchical_label "NVDC_SYS"
+		(shape bidirectional)
+		(at 20.32 30.48 0)
+		(effects (font (size 1.27 1.27)))
+	)
+	(wire
+		(pts (xy 20.32 30.48) (xy 25.40 30.48))
+		(stroke (width 0) (type default))
+	)
+	(no_connect (at 25.40 30.48)
+	)
+	(hierarchical_label "POWER_GROUND"
+		(shape bidirectional)
+		(at 20.32 35.56 0)
+		(effects (font (size 1.27 1.27)))
+	)
+	(wire
+		(pts (xy 20.32 35.56) (xy 25.40 35.56))
+		(stroke (width 0) (type default))
+	)
+	(no_connect (at 25.40 35.56)
+	)
+	(hierarchical_label "PROTECTED_PACK_POSITIVE"
+		(shape bidirectional)
+		(at 20.32 40.64 0)
+		(effects (font (size 1.27 1.27)))
+	)
+	(wire
+		(pts (xy 20.32 40.64) (xy 25.40 40.64))
+		(stroke (width 0) (type default))
+	)
+	(no_connect (at 25.40 40.64)
+	)
+	(hierarchical_label "S3_USB_DM"
+		(shape bidirectional)
+		(at 190.50 20.32 180)
+		(effects (font (size 1.27 1.27)) (justify right))
+	)
+	(wire
+		(pts (xy 190.50 20.32) (xy 185.42 20.32))
+		(stroke (width 0) (type default))
+	)
+	(no_connect (at 185.42 20.32)
+	)
+	(hierarchical_label "S3_USB_DP"
+		(shape bidirectional)
+		(at 190.50 25.40 180)
+		(effects (font (size 1.27 1.27)) (justify right))
+	)
+	(wire
+		(pts (xy 190.50 25.40) (xy 185.42 25.40))
+		(stroke (width 0) (type default))
+	)
+	(no_connect (at 185.42 25.40)
+	)
+	(hierarchical_label "SYS_I2C_SCL"
+		(shape bidirectional)
+		(at 190.50 30.48 180)
+		(effects (font (size 1.27 1.27)) (justify right))
+	)
+	(wire
+		(pts (xy 190.50 30.48) (xy 185.42 30.48))
+		(stroke (width 0) (type default))
+	)
+	(no_connect (at 185.42 30.48)
+	)
+	(hierarchical_label "SYS_I2C_SDA"
+		(shape bidirectional)
+		(at 190.50 35.56 180)
+		(effects (font (size 1.27 1.27)) (justify right))
+	)
+	(wire
+		(pts (xy 190.50 35.56) (xy 185.42 35.56))
+		(stroke (width 0) (type default))
+	)
+	(no_connect (at 185.42 35.56)
+	)
+	(hierarchical_label "SYS_INT_N"
+		(shape bidirectional)
+		(at 190.50 40.64 180)
+		(effects (font (size 1.27 1.27)) (justify right))
+	)
+	(wire
+		(pts (xy 190.50 40.64) (xy 185.42 40.64))
+		(stroke (width 0) (type default))
+	)
+	(no_connect (at 185.42 40.64)
+	)
 	(sheet_instances
 		(path "/"

Commit message: complete exact H2.3.2 USB PD charging
Parts:
- added C1: TDK C1608X7S2A104K080AB, Capacitor_SMD:C_0603_1608Metric, symbol Leshy2:RF01_PRODUCT_USB_VBIAS_CAP
- added C10: TDK CGA5L1X7R1E475K160AC, Capacitor_SMD:C_1206_3216Metric, symbol Leshy2:RF01_PD_VBUS_CAP
- added C11: Murata GRM1555C1H221JA01D, Capacitor_SMD:C_0402_1005Metric, symbol Leshy2:RF01_PD_CC1_CAP
- added C12: Murata GRM1555C1H221JA01D, Capacitor_SMD:C_0402_1005Metric, symbol Leshy2:RF01_PD_CC2_CAP
- added C13: TDK C1005X7R1H104K050BB, Capacitor_SMD:C_0402_1005Metric, symbol Leshy2:RF01_PD_EEPROM_BYPASS
- added C14: Murata GRM31CR71E106MA12L, Capacitor_SMD:C_1206_3216Metric, symbol Leshy2:RF01_CHARGER_VBUS_CAP0
- added C15: Murata GRM31CR71E106MA12L, Capacitor_SMD:C_1206_3216Metric, symbol Leshy2:RF01_CHARGER_VBUS_CAP1
- added C16: TDK C1005X7R1H104K050BB, Capacitor_SMD:C_0402_1005Metric, symbol Leshy2:RF01_CHARGER_VBUS_HF_CAP
- added C17: Murata GRM31CR71E106MA12L, Capacitor_SMD:C_1206_3216Metric, symbol Leshy2:RF01_CHARGER_PMID_CAP0
- added C18: Murata GRM31CR71E106MA12L, Capacitor_SMD:C_1206_3216Metric, symbol Leshy2:RF01_CHARGER_PMID_CAP1
- added C19: Murata GRM31CR71E106MA12L, Capacitor_SMD:C_1206_3216Metric, symbol Leshy2:RF01_CHARGER_PMID_CAP2
- added C2: TDK C1608X7R1C105K080AC, Capacitor_SMD:C_0603_1608Metric, symbol Leshy2:RF01_PRODUCT_USB_VPWR_CAP
- added C20: TDK C1005X7R1H104K050BB, Capacitor_SMD:C_0402_1005Metric, symbol Leshy2:RF01_CHARGER_PMID_HF_CAP
- added C21: Murata GRM31CR71E106MA12L, Capacitor_SMD:C_1206_3216Metric, symbol Leshy2:RF01_CHARGER_SYS_CAP0
- added C22: Murata GRM31CR71E106MA12L, Capacitor_SMD:C_1206_3216Metric, symbol Leshy2:RF01_CHARGER_SYS_CAP1
- added C23: Murata GRM31CR71E106MA12L, Capacitor_SMD:C_1206_3216Metric, symbol Leshy2:RF01_CHARGER_SYS_CAP2
- added C24: Murata GRM31CR71E106MA12L, Capacitor_SMD:C_1206_3216Metric, symbol Leshy2:RF01_CHARGER_SYS_CAP3
- added C25: Murata GRM31CR71E106MA12L, Capacitor_SMD:C_1206_3216Metric, symbol Leshy2:RF01_CHARGER_SYS_CAP4
- added C26: TDK C1005X7R1H104K050BB, Capacitor_SMD:C_0402_1005Metric, symbol Leshy2:RF01_CHARGER_SYS_HF_CAP
- added C27: Murata GRM31CR71E106MA12L, Capacitor_SMD:C_1206_3216Metric, symbol Leshy2:RF01_CHARGER_BAT_CAP0
- added C28: Murata GRM31CR71E106MA12L, Capacitor_SMD:C_1206_3216Metric, symbol Leshy2:RF01_CHARGER_BAT_CAP1
- added C29: Murata GRM155R71E473KA88D, Capacitor_SMD:C_0402_1005Metric, symbol Leshy2:RF01_CHARGER_BTST1_CAP
- added C3: Murata GRM188R60J106ME47D, Capacitor_SMD:C_0603_1608Metric, symbol Leshy2:RF01_PD_VIN_CAP
- added C30: Murata GRM155R71E473KA88D, Capacitor_SMD:C_0402_1005Metric, symbol Leshy2:RF01_CHARGER_BTST2_CAP
- added C31: TDK CGA5L1X7R1E475K160AC, Capacitor_SMD:C_1206_3216Metric, symbol Leshy2:RF01_CHARGER_REGN_CAP
- added C32: KEMET C0402C102K5RACTU, Capacitor_SMD:C_0402_1005Metric, symbol Leshy2:RF01_CHARGER_SDRV_CAP
- added C4: Murata GRM188R60J106ME47D, Capacitor_SMD:C_0603_1608Metric, symbol Leshy2:RF01_PD_LDO3V3_CAP
- added C5: Murata GRM188R60J106ME47D, Capacitor_SMD:C_0603_1608Metric, symbol Leshy2:RF01_PD_LDO1V5_CAP
- added C6: Murata GRM32ER71E226KE15L, Capacitor_SMD:C_1210_3225Metric, symbol Leshy2:RF01_PD_PPHV_CAP0
- added C7: Murata GRM32ER71E226KE15L, Capacitor_SMD:C_1210_3225Metric, symbol Leshy2:RF01_PD_PPHV_CAP1
- added C8: Murata GRM32ER71E226KE15L, Capacitor_SMD:C_1210_3225Metric, symbol Leshy2:RF01_PD_PPHV_CAP2
- added C9: Murata GRM32ER71E226KE15L, Capacitor_SMD:C_1210_3225Metric, symbol Leshy2:RF01_PD_PPHV_CAP3
- added D1: Texas Instruments TVS2200DRVR, Package_SON:WSON-6-1EP_2x2mm_P0.65mm_EP1x1.6mm, symbol Leshy2:RF01_PD_VBUS_TVS
- added J1: JAE DX07S016JA1R1500, Connector_USB:USB_C_Receptacle_JAE_DX07S016JA1R1500, symbol Leshy2:RF01_PRODUCT_USB_CONNECTOR
- added L1: Sunlord MWSA0503S-2R2MT, Inductor_SMD:L_Sunlord_MWSA0503S, symbol Leshy2:RF01_CHARGER_INDUCTOR
- added R1: Yageo RC0402FR-0710KL, Resistor_SMD:R_0402_1005Metric, symbol Leshy2:RF01_PRODUCT_USB_FAULT_PULLUP
- added R10: Yageo RC0402FR-07100KL, Resistor_SMD:R_0402_1005Metric, symbol Leshy2:RF01_CHARGER_ILIM_BOTTOM
- added R11: Yageo RC0402FR-0710KL, Resistor_SMD:R_0402_1005Metric, symbol Leshy2:RF01_CHARGER_INT_PULLUP
- added R12: Yageo RC0402FR-0710KL, Resistor_SMD:R_0402_1005Metric, symbol Leshy2:RF01_CHARGER_CE_PULLUP
- added R2: Yageo RC0402FR-0710KL, Resistor_SMD:R_0402_1005Metric, symbol Leshy2:RF01_PD_EEPROM_WP_PULLUP
- added R3: Yageo RC0402FR-072K2L, Resistor_SMD:R_0402_1005Metric, symbol Leshy2:RF01_PD_LOCAL_SCL_PULLUP
- added R4: Yageo RC0402FR-072K2L, Resistor_SMD:R_0402_1005Metric, symbol Leshy2:RF01_PD_LOCAL_SDA_PULLUP
- added R5: Yageo RC0402FR-078K2L, Resistor_SMD:R_0402_1005Metric, symbol Leshy2:RF01_CHARGER_PROG_RES
- added R6: Yageo RC0402FR-07100RL, Resistor_SMD:R_0402_1005Metric, symbol Leshy2:RF01_CHARGER_BATP_RES
- added R7: Yageo RC0402FR-075K23L, Resistor_SMD:R_0402_1005Metric, symbol Leshy2:RF01_CHARGER_TS_TOP
- added R8: Yageo RC0402FR-0730K1L, Resistor_SMD:R_0402_1005Metric, symbol Leshy2:RF01_CHARGER_TS_BOTTOM
- added R9: Yageo RC0402FR-0744K2L, Resistor_SMD:R_0402_1005Metric, symbol Leshy2:RF01_CHARGER_ILIM_TOP
- added TH1: TDK B57332V5103F360, Resistor_SMD:R_0603_1608Metric, symbol Leshy2:RF01_CHARGER_TS_NTC
- added U1: Texas Instruments TPD4S201RUKR, Package_DFN_QFN:Texas_RUK0020B_WQFN-20-1EP_3x3mm_P0.4mm_EP1.7x1.7mm, symbol Leshy2:RF01_PRODUCT_USB_PROTECTOR
- added U2: Texas Instruments TPS25751DREFR, Package_DFN_QFN:Texas_REF0038A_WQFN-38-2EP_6x4mm_P0.4, symbol Leshy2:RF01_PD_CONTROLLER
- added U3: onsemi CAT24C512WI-GT3, Package_SO:SOIC-8_3.9x4.9mm_P1.27mm, symbol Leshy2:RF01_PD_CONFIG_EEPROM
- added U4: Texas Instruments BQ25798RQMR, Package_DFN_QFN:Texas_RQM0029A_VQFN-29_4x4mm_P0.4mm, symbol Leshy2:RF01_NVDC_CHARGER
Connections:
- net AON_SAFE_3V3: now also C3.1 (END_1), U2.38 (VIN_3V3)
- net NVDC_SYS: now also C21.1 (END_1), C22.1 (END_1), C23.1 (END_1), C24.1 (END_1), C25.1 (END_1), C26.1 (END_1), U4.25 (SYS)
- net POWER_GROUND: now also C1.2 (END_2), C10.2 (END_2), C11.2 (END_2), C12.2 (END_2), C13.2 (END_2), C14.2 (END_2), C15.2 (END_2), C16.2 (END_2), C17.2 (END_2), C18.2 (END_2), C19.2 (END_2), C2.2 (END_2), C20.2 (END_2), C21.2 (END_2), C22.2 (END_2), C23.2 (END_2), C24.2 (END_2), C25.2 (END_2), C26.2 (END_2), C27.2 (END_2), C28.2 (END_2), C3.2 (END_2), C31.2 (END_2), C32.2 (END_2), C4.2 (END_2), C5.2 (END_2), C6.2 (END_2), C7.2 (END_2), C8.2 (END_2), C9.2 (END_2), D1.1 (GND_1), D1.2 (GND_2), D1.3 (GND_3), D1.7 (GND_PAD), J1.A1 (A1_GND), J1.A12 (A12_GND), J1.B1 (B1_GND), J1.B12 (B12_GND), J1.SH (SHIELD), R10.2 (END_2), R5.2 (END_2), R8.2 (END_2), TH1.2 (END_2), U1.13 (GND_13), U1.18 (GND_18), U1.21 (GND_PAD), U1.8 (GND_8), U2.11 (GND_11), U2.12 (GND_12), U2.13 (GPIO11), U2.14 (GND_14), U2.19 (GPIO3), U2.26 (GPIO4_USB_P_LD1), U2.27 (GPIO5_USB_N_LD2), U2.3 (ADCIN2), U2.31 (GND_31), U2.34 (PP5V), U2.36 (GPIO7), U2.37 (GPIO6), U2.39 (GND_PAD), U2.7 (GPIO2), U3.1 (A0), U3.2 (A1), U3.3 (A2), U3.4 (VSS), U4.10 (ACDRV2), U4.11 (ACDRV1), U4.27 (GND)
- net PROTECTED_PACK_POSITIVE: now also C27.1 (END_1), C28.1 (END_1), R6.1 (END_1), U4.22 (BAT_22), U4.23 (BAT_23)
- net S3_USB_DM: now also U1.14 (SBU2)
- net S3_USB_DP: now also U1.15 (SBU1)
- net SYS_I2C_SCL: now also U2.9 (I2Ct_SCL)
- net SYS_I2C_SDA: now also U2.8 (I2Ct_SDA)
- net SYS_INT_N: now also U2.10 (I2Ct_IRQ)
- new net CHARGER_BATP_SENSE: R6.2 (END_2), U4.18 (BATP)
- new net CHARGER_BTST1: C29.1 (END_1), U4.4 (BTST1)
- new net CHARGER_BTST2: C30.1 (END_1), U4.19 (BTST2)
- new net CHARGER_ILIM_HIZ: R10.1 (END_1), R9.2 (END_2), U4.17 (ILIM_HIZ)
- new net CHARGER_INT_N: R11.2 (END_2), U2.18 (I2Cc_IRQ), U4.21 (INT)
- new net CHARGER_PMID: C17.1 (END_1), C18.1 (END_1), C19.1 (END_1), C20.1 (END_1), U4.29 (PMID)
- new net CHARGER_PROG_2S_750KHZ: R5.1 (END_1), U4.20 (PROG)
- new net CHARGER_REGN: C31.1 (END_1), R12.1 (END_1), R7.1 (END_1), R9.1 (END_1), U4.5 (REGN)
- new net CHARGER_SDRV_UNUSED: C32.1 (END_1), U4.24 (SDRV)
- new net CHARGER_SW1: C29.2 (END_2), L1.1 (END_1), U4.28 (SW1)
- new net CHARGER_SW2: C30.2 (END_2), L1.2 (END_2), U4.26 (SW2)
- new net CHARGER_TS: R7.2 (END_2), R8.1 (END_1), TH1.1 (END_1), U4.16 (TS)
- new net CHARGE_EN_N: R12.2 (END_2), U2.6 (GPIO1), U4.13 (CE)
- new net PD_DRAIN_COPPER: U2.15 (DRAIN_15), U2.30 (DRAIN_30), U2.40 (DRAIN_PAD)
- new net PD_EEPROM_WP: R2.2 (END_2), U2.5 (GPIO0), U3.7 (WP)
- new net PD_LOCAL_1V5: C5.1 (END_1), U2.4 (LDO_1V5)
- new net PD_LOCAL_3V3: C13.1 (END_1), C2.1 (END_1), C4.1 (END_1), R1.1 (END_1), R11.1 (END_1), R2.1 (END_1), R3.1 (END_1), R4.1 (END_1), U1.10 (VPWR), U2.1 (LDO_3V3), U2.2 (ADCIN1), U3.8 (VCC)
- new net PD_LOCAL_I2C_SCL: R3.2 (END_2), U2.17 (I2Cc_SCL), U3.6 (SCL), U4.14 (SCL)
- new net PD_LOCAL_I2C_SDA: R4.2 (END_2), U2.16 (I2Cc_SDA), U3.5 (SDA), U4.15 (SDA)
- new net PD_NEGOTIATED_VBUS: C14.1 (END_1), C15.1 (END_1), C16.1 (END_1), C6.1 (END_1), C7.1 (END_1), C8.1 (END_1), C9.1 (END_1), U2.20 (PPHV), U4.2 (VBUS_2), U4.3 (VBUS_3), U4.8 (VAC2), U4.9 (VAC1)
- new net USB2_DM_CONNECTOR: J1.A7 (A7_DM), J1.B7 (B7_DM), U1.2 (C_SBU2)
- new net USB2_DP_CONNECTOR: J1.A6 (A6_DP), J1.B6 (B6_DP), U1.1 (C_SBU1)
- new net USB_C_CC1_CONNECTOR: J1.A5 (A5_CC1), U1.4 (C_CC1), U1.7 (RPD_G1)
- new net USB_C_CC1_PROTECTED: C11.1 (END_1), U1.12 (CC1), U2.28 (CC1)
- new net USB_C_CC2_CONNECTOR: J1.B5 (B5_CC2), U1.5 (C_CC2), U1.6 (RPD_G2)
- new net USB_C_CC2_PROTECTED: C12.1 (END_1), U1.11 (CC2), U2.29 (CC2)
- new net USB_C_VBUS_RAW: C10.1 (END_1), D1.4 (IN_4), D1.5 (IN_5), D1.6 (IN_6), J1.A4 (A4_VBUS), J1.A9 (A9_VBUS), J1.B4 (B4_VBUS), J1.B9 (B9_VBUS), U2.23 (VBUS_IN), U2.32 (VBUS)
- new net USB_PROTECTOR_FAULT_N: R1.2 (END_2), U1.9 (FLT)
- new net USB_PROTECTOR_VBIAS: C1.1 (END_1), U1.3 (VBIAS)
Other:
- title: (none) -> Leshy2 — exact sink-only USB-PD and 2S NVDC charging

Commit message: complete H2 schematic review package
Parts:
- renumbered C1 to C1001, C2 to C1002, C3 to C1003, C4 to C1004, C5 to C1005, C6 to C1006, C7 to C1007, C8 to C1008, C9 to C1009, C10 to C1010, C11 to C1011, C12 to C1012, C13 to C1013, C14 to C1014, C15 to C1015, C16 to C1016, C17 to C1017, C18 to C1018, C19 to C1019, C20 to C1020, C21 to C1021, C22 to C1022, C23 to C1023, C24 to C1024, C25 to C1025, C26 to C1026, C27 to C1027, C28 to C1028, C29 to C1029, C30 to C1030, C31 to C1031, C32 to C1032, D1 to D1001, J1 to J1001, L1 to L1001, R1 to R1001, R2 to R1002, R3 to R1003, R4 to R1004, R5 to R1005, R6 to R1006, R7 to R1007, R8 to R1008, R9 to R1009, R10 to R1010, R11 to R1011, R12 to R1012, TH1 to TH1001, U1 to U1001, U2 to U1002, U3 to U1003, U4 to U1004

Commit message: Optimize H1 display and stocked BOM routes
Parts:
- C1013, C1016, C1020, C1026: value TDK C1005X7R1H104K050BB -> Yageo CC0402KRX7R9BB104
Changed lines of the file:
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@@
 			(effects (font (size 1.27 1.27)))
 		)
-		(property "Value" "TDK C1005X7R1H104K050BB"
+		(property "Value" "Yageo CC0402KRX7R9BB104"
 			(at 50.80 120.65 0)
 			(show_name no)
@@
 			(effects (font (size 1.27 1.27)))
 		)
-		(property "Value" "TDK C1005X7R1H104K050BB"
+		(property "Value" "Yageo CC0402KRX7R9BB104"
 			(at 132.08 151.13 0)
 			(show_name no)
@@
 			(effects (font (size 1.27 1.27)))
 		)
-		(property "Value" "TDK C1005X7R1H104K050BB"
+		(property "Value" "Yageo CC0402KRX7R9BB104"
 			(at 457.20 163.83 0)
 			(show_name no)
@@
 			(effects (font (size 1.27 1.27)))
 		)
-		(property "Value" "TDK C1005X7R1H104K050BB"
+		(property "Value" "Yageo CC0402KRX7R9BB104"
 			(at 213.36 189.23 0)
 			(show_name no)

Commit message: Replace six pre-order resistor identities
Parts:
- R1003, R1004: value Yageo RC0402FR-072K2L -> UNI-ROYAL 0402WGF2201TCE
- R1005: value Yageo RC0402FR-078K2L -> UNI-ROYAL 0402WGF8201TCE
- R1007: value Yageo RC0402FR-075K23L -> UNI-ROYAL 0402WGF5231TCE
Changed lines of the file:
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@@
 			(effects (font (size 1.27 1.27)))
 		)
-		(property "Value" "Yageo RC0402FR-072K2L"
+		(property "Value" "UNI-ROYAL 0402WGF2201TCE"
 			(at 294.64 125.73 0)
 			(show_name no)
@@
 			(effects (font (size 1.27 1.27)))
 		)
-		(property "Value" "Yageo RC0402FR-072K2L"
+		(property "Value" "UNI-ROYAL 0402WGF2201TCE"
 			(at 375.92 125.73 0)
 			(show_name no)
@@
 			(effects (font (size 1.27 1.27)))
 		)
-		(property "Value" "Yageo RC0402FR-078K2L"
+		(property "Value" "UNI-ROYAL 0402WGF8201TCE"
 			(at 213.36 214.63 0)
 			(show_name no)
@@
 			(effects (font (size 1.27 1.27)))
 		)
-		(property "Value" "Yageo RC0402FR-075K23L"
+		(property "Value" "UNI-ROYAL 0402WGF5231TCE"
 			(at 50.80 222.25 0)
 			(show_name no)

Commit message: Replace three pre-order passive parts
Parts:
- C1001: value TDK C1608X7S2A104K080AB -> Yageo CC0603KRX7R0BB104
Changed lines of the file:
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@@
 			(effects (font (size 1.27 1.27)))
 		)
-		(property "Value" "TDK C1608X7S2A104K080AB"
+		(property "Value" "Yageo CC0603KRX7R0BB104"
 			(at 213.36 49.53 0)
 			(show_name no)
@@
 			(effects (font (size 1.27 1.27)))
 		)
-		(property "Description" "100nf_10pct_100v_x7s_0603_usb_protector_bias_capacitor"
+		(property "Description" "100nf_10pct_100v_x7r_0603_usb_protector_bias_capacitor"
 			(at 213.36 44.45 0)
 			(show_name no)
