File: hardware/ecad/kicad/LESHY2-UI/LESHY2-UI.kicad_sch (KiCad schematic)
At the start: 0 parts

Commit message: Complete H2.2.2 S3 core schematic
Other:
- sheet UI_10_S3_CORE_MEMORY_BOOT ports: added DISPLAY_SD_SPI_D0, DISPLAY_SD_SPI_SCK, ENCODER_A, ENCODER_B, LCD_BL_PWM, LCD_CS_N, LCD_QSPI_D2, LCD_QSPI_D3, RP_ALERT_N, S3_C5_SDIO_CLK, S3_C5_SDIO_CMD, S3_C5_SDIO_D0, S3_C5_SDIO_D1_IRQ, S3_RP_IPC_CS_N, S3_RP_IPC_MISO, S3_RP_IPC_MOSI, S3_RP_IPC_SCK, SD_SPI_CS_N, UNIT_HOST_SIG0, UNIT_HOST_SIG1; removed none
- sheet UI_11_DISPLAY_TOUCH_STORAGE ports: added DISPLAY_SD_SPI_D0, DISPLAY_SD_SPI_SCK, LCD_BL_PWM, LCD_CS_N, LCD_QSPI_D2, LCD_QSPI_D3, SD_SPI_CS_N; removed none
- sheet UI_20_C5_RADIO_IR_SERVICE ports: added S3_C5_SDIO_CLK, S3_C5_SDIO_CMD, S3_C5_SDIO_D0, S3_C5_SDIO_D1_IRQ; removed none
- sheet UI_40_INTERBOARD_M1 ports: added RP_ALERT_N, S3_RP_IPC_CS_N, S3_RP_IPC_MISO, S3_RP_IPC_MOSI, S3_RP_IPC_SCK, UNIT_HOST_SIG0, UNIT_HOST_SIG1; removed none

Commit message: complete exact H2.2.9 UI TX safety schematic
Other:
- sheet UI_12_CONTROLS_INDICATORS ports: added none; removed S3_RF_TX_EVIDENCE_AON_N
- sheet UI_50_TX_SAFETY_EVIDENCE ports: added none; removed S3_RF_TX_EVIDENCE_AON_N

Commit message: complete exact H2.2.10 UI test points
Other:
- sheet UI_11_DISPLAY_TOUCH_STORAGE ports: added LCD_BACKLIGHT_FAULT_N; removed none
- sheet UI_12_CONTROLS_INDICATORS ports: added SLOW_IO_RESET_N; removed none
- sheet UI_20_C5_RADIO_IR_SERVICE ports: added C5_GPIO27_FIXED_HIGH, C5_SERVICE_VBUS_SENSE_ONLY, IR_TX_CARRIER_SAFE; removed none
- sheet UI_60_TESTPOINTS_MANUFACTURING ports: added C5_GPIO27_FIXED_HIGH, C5_RESET_N, C5_SERVICE_VBUS_SENSE_ONLY, EV_N0_S3, EV_N1_C5, EV_N7_IR, IR_TX_CARRIER_SAFE, LCD_BACKLIGHT_FAULT_N, S3_RESET_N, SLOW_IO_RESET_N, UI_ZONE_TEMP_ADC; removed none

Commit message: review H3.6.2 single-fault containment
Other:
- sheet UI_40_INTERBOARD_M1 ports: added FAULT_ASSERT_N; removed RF_RESET_KILL_GATE
- sheet UI_50_TX_SAFETY_EVIDENCE ports: added FAULT_ASSERT_N, RUN_PERMIT; removed RF_RESET_KILL_GATE

Commit message: Reclose H2 through H4 on dual SA818S architecture
Other:
- sheet UI_13_AUDIO_CODEC_HEADSET ports: added RX_VOICE_AFOUT_SELECTED; removed RX_SA518_AFOUT_ISOLATED
- sheet UI_40_INTERBOARD_M1 ports: added RX_VOICE_AFOUT_SELECTED; removed RX_SA518_AFOUT_ISOLATED
Changed lines of the file:
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@@
 			(effects (font (size 1.27 1.27)))
 		)
-		(pin "RX_SA518_AFOUT_ISOLATED" bidirectional
+		(pin "RX_SI4732_MONO" bidirectional
 			(at 330.20 416.56 0)
 			(effects (font (size 1.27 1.27)))
 		)
-		(pin "RX_SI4732_MONO" bidirectional
+		(pin "RX_VOICE_AFOUT_SELECTED" bidirectional
 			(at 330.20 419.10 0)
 			(effects (font (size 1.27 1.27)))
@@
 			(effects (font (size 1.27 1.27)))
 		)
-		(pin "RX_SA518_AFOUT_ISOLATED" bidirectional
+		(pin "RX_VOICE_AFOUT_SELECTED" bidirectional
 			(at 330.20 660.40 0)
 			(effects (font (size 1.27 1.27)))
@@
 	)
 	(wire
-		(pts (xy 330.20 660.40) (xy 640.08 660.40))
-		(stroke (width 0) (type default))
-	)
-	(junction (at 640.08 660.40)
-		(diameter 0)
-		(color 0 0 0 0)
-	)
-	(wire
-		(pts (xy 640.08 416.56) (xy 640.08 660.40))
-		(stroke (width 0) (type default))
-	)
-	(wire
-		(pts (xy 330.20 419.10) (xy 645.16 419.10))
-		(stroke (width 0) (type default))
-	)
-	(junction (at 645.16 419.10)
-		(diameter 0)
-		(color 0 0 0 0)
-	)
-	(wire
-		(pts (xy 330.20 548.64) (xy 645.16 548.64))
-		(stroke (width 0) (type default))
-	)
-	(junction (at 645.16 548.64)
-		(diameter 0)
-		(color 0 0 0 0)
-	)
-	(wire
-		(pts (xy 645.16 419.10) (xy 645.16 548.64))
-		(stroke (width 0) (type default))
-	)
-	(wire
-		(pts (xy 330.20 299.72) (xy 650.24 299.72))
-		(stroke (width 0) (type default))
-	)
-	(junction (at 650.24 299.72)
-		(diameter 0)
-		(color 0 0 0 0)
-	)
-	(wire
-		(pts (xy 330.20 551.18) (xy 650.24 551.18))
-		(stroke (width 0) (type default))
-	)
-	(junction (at 650.24 551.18)
-		(diameter 0)
-		(color 0 0 0 0)
-	)
-	(wire
-		(pts (xy 650.24 299.72) (xy 650.24 551.18))
-		(stroke (width 0) (type default))
-	)
+		(pts (xy 330.20 548.64) (xy 640.08 548.64))
+		(stroke (width 0) (type default))
+	)
+	(junction (at 640.08 548.64)
+		(diameter 0)
+		(color 0 0 0 0)
+	)
+	(wire
+		(pts (xy 640.08 416.56) (xy 640.08 548.64))
+		(stroke (width 0) (type default))
+	)
+	(wire
+		(pts (xy 330.20 299.72) (xy 645.16 299.72))
+		(stroke (width 0) (type default))
+	)
+	(junction (at 645.16 299.72)
+		(diameter 0)
+		(color 0 0 0 0)
+	)
+	(wire
+		(pts (xy 330.20 551.18) (xy 645.16 551.18))
+		(stroke (width 0) (type default))
+	)
+	(junction (at 645.16 551.18)
+		(diameter 0)
+		(color 0 0 0 0)
+	)
+	(wire
+		(pts (xy 645.16 299.72) (xy 645.16 551.18))
+		(stroke (width 0) (type default))
+	)
+	(wire
+		(pts (xy 330.20 419.10) (xy 650.24 419.10))
+		(stroke (width 0) (type default))
+	)
+	(junction (at 650.24 419.10)
+		(diameter 0)
+		(color 0 0 0 0)
+	)
+	(wire
+		(pts (xy 330.20 660.40) (xy 650.24 660.40))
+		(stroke (width 0) (type default))
+	)
+	(junction (at 650.24 660.40)
+		(diameter 0)
+		(color 0 0 0 0)
+	)
+	(wire
+		(pts (xy 650.24 419.10) (xy 650.24 660.40))
+		(stroke (width 0) (type default))
+	)
