File: hardware/ecad/kicad/LESHY2-UI/UI_12_CONTROLS_INDICATORS.kicad_sch (KiCad schematic)
At the start: 0 parts

Commit message: complete exact H2.2.4 controls schematic
Parts:
- added C1: TDK C1005X7R1H104K050BB, Capacitor_SMD:C_0402_1005Metric, symbol Leshy2:UI12_SLOW_IO_VCCI_BYPASS
- added C2: TDK C1005X7R1H104K050BB, Capacitor_SMD:C_0402_1005Metric, symbol Leshy2:UI12_SLOW_IO_VCCP_BYPASS
- added C3: TDK C1608X7R1C105K080AC, Capacitor_SMD:C_0603_1608Metric, symbol Leshy2:UI12_SLOW_IO_BULK_CAP
- added C4: TDK C1005X7R1H104K050BB, Capacitor_SMD:C_0402_1005Metric, symbol Leshy2:UI12_SLOW_IO_FAULT_SENSE_ISO_BYPASS
- added C5: TDK C1005X7R1H104K050BB, Capacitor_SMD:C_0402_1005Metric, symbol Leshy2:UI12_SLOW_IO_S3_EVIDENCE_ISO_BYPASS
- added C6: TDK C1005X7R1H104K050BB, Capacitor_SMD:C_0402_1005Metric, symbol Leshy2:UI12_UI_MATRIX_IO_BYPASS
- added C7: TDK C1005X7R1H104K050BB, Capacitor_SMD:C_0402_1005Metric, symbol Leshy2:UI12_UI_ZONE_TEMP_FILTER
- added D1: Texas Instruments TPD8E003DQDR, Leshy2:TPD8E003DQDR, symbol Leshy2:UI12_UI_MATRIX_ESD
- added D10: LTST-C190KRKT, LED_SMD:LED_0603_1608Metric, symbol Leshy2:UI12_IR_TX_LED
- added D11: LTST-C190KRKT, LED_SMD:LED_0603_1608Metric, symbol Leshy2:UI12_EXT_TX_LED
- added D12: LTST-C190KFKT, LED_SMD:LED_0603_1608Metric, symbol Leshy2:UI12_FAULT_LED
- added D2: Texas Instruments TPD8E003DQDR, Leshy2:TPD8E003DQDR, symbol Leshy2:UI12_FRONT_FUNCTION_ESD
- added D3: LTST-C190KRKT, LED_SMD:LED_0603_1608Metric, symbol Leshy2:UI12_S3_TX_LED
- added D4: LTST-C190KRKT, LED_SMD:LED_0603_1608Metric, symbol Leshy2:UI12_C5_TX_LED
- added D5: LTST-C190KRKT, LED_SMD:LED_0603_1608Metric, symbol Leshy2:UI12_NRF0_TX_LED
- added D6: LTST-C190KRKT, LED_SMD:LED_0603_1608Metric, symbol Leshy2:UI12_NRF1_TX_LED
- added D7: LTST-C190KRKT, LED_SMD:LED_0603_1608Metric, symbol Leshy2:UI12_NRF2_TX_LED
- added D8: LTST-C190KRKT, LED_SMD:LED_0603_1608Metric, symbol Leshy2:UI12_CC_TX_LED
- added D9: LTST-C190KRKT, LED_SMD:LED_0603_1608Metric, symbol Leshy2:UI12_VOICE_TX_LED
- added R1: Yageo RC0402FR-0710KL, Resistor_SMD:R_0402_1005Metric, symbol Leshy2:UI12_SLOW_IO_RESET_PULLUP
- added R10: Yageo RC0402FR-073K32L, Resistor_SMD:R_0402_1005Metric, symbol Leshy2:UI12_UI_INPUT_OPT_PULLUP
- added R11: Yageo RC0402FR-073K32L, Resistor_SMD:R_0402_1005Metric, symbol Leshy2:UI12_UI_INPUT_F1_PULLUP
- added R12: Yageo RC0402FR-073K32L, Resistor_SMD:R_0402_1005Metric, symbol Leshy2:UI12_UI_INPUT_F2_PULLUP
- added R13: Yageo RC0402FR-073K32L, Resistor_SMD:R_0402_1005Metric, symbol Leshy2:UI12_UI_INPUT_F3_PULLUP
- added R14: Yageo RC0402FR-073K32L, Resistor_SMD:R_0402_1005Metric, symbol Leshy2:UI12_UI_INPUT_F4_PULLUP
- added R15: Yageo RC0402FR-073K32L, Resistor_SMD:R_0402_1005Metric, symbol Leshy2:UI12_UI_INPUT_F5_PULLUP
- added R16: Yageo RC0402FR-073K32L, Resistor_SMD:R_0402_1005Metric, symbol Leshy2:UI12_UI_INPUT_F6_PULLUP
- added R17: Yageo RC0402FR-073K32L, Resistor_SMD:R_0402_1005Metric, symbol Leshy2:UI12_UI_INPUT_F7_PULLUP
- added R18: Yageo RC0402FR-073K32L, Resistor_SMD:R_0402_1005Metric, symbol Leshy2:UI12_UI_INPUT_F8_PULLUP
- added R19: Yageo RC0402FR-073K32L, Resistor_SMD:R_0402_1005Metric, symbol Leshy2:UI12_UI_INPUT_ENCODER_PULLUP
- added R2: Yageo RC0402FR-0710KL, Resistor_SMD:R_0402_1005Metric, symbol Leshy2:UI12_SLOW_IO_FAULT_SENSE_PULLUP
- added R20: Yageo RC0402FR-073K32L, Resistor_SMD:R_0402_1005Metric, symbol Leshy2:UI12_ENCODER_A_PULLUP
- added R21: Yageo RC0402FR-073K32L, Resistor_SMD:R_0402_1005Metric, symbol Leshy2:UI12_ENCODER_B_PULLUP
- added R22: Yageo RC0402FR-0710KL, Resistor_SMD:R_0402_1005Metric, symbol Leshy2:UI12_UI_ZONE_TEMP_PULLUP
- added R23: Yageo RC0402FR-072K2L, Resistor_SMD:R_0402_1005Metric, symbol Leshy2:UI12_S3_TX_LED_SERIES
- added R24: Yageo RC0402FR-072K2L, Resistor_SMD:R_0402_1005Metric, symbol Leshy2:UI12_C5_TX_LED_SERIES
- added R25: Yageo RC0402FR-072K2L, Resistor_SMD:R_0402_1005Metric, symbol Leshy2:UI12_NRF0_TX_LED_SERIES
- added R26: Yageo RC0402FR-072K2L, Resistor_SMD:R_0402_1005Metric, symbol Leshy2:UI12_NRF1_TX_LED_SERIES
- added R27: Yageo RC0402FR-072K2L, Resistor_SMD:R_0402_1005Metric, symbol Leshy2:UI12_NRF2_TX_LED_SERIES
- added R28: Yageo RC0402FR-072K2L, Resistor_SMD:R_0402_1005Metric, symbol Leshy2:UI12_CC_TX_LED_SERIES
- added R29: Yageo RC0402FR-072K2L, Resistor_SMD:R_0402_1005Metric, symbol Leshy2:UI12_VOICE_TX_LED_SERIES
- added R3: Yageo RC0402FR-0710KL, Resistor_SMD:R_0402_1005Metric, symbol Leshy2:UI12_SLOW_IO_S3_EVIDENCE_PULLUP
- added R30: Yageo RC0402FR-072K2L, Resistor_SMD:R_0402_1005Metric, symbol Leshy2:UI12_IR_TX_LED_SERIES
- added R31: Yageo RC0402FR-072K2L, Resistor_SMD:R_0402_1005Metric, symbol Leshy2:UI12_EXT_TX_LED_SERIES
- added R32: Yageo RC0402FR-072K2L, Resistor_SMD:R_0402_1005Metric, symbol Leshy2:UI12_FAULT_LED_SERIES
- added R4: Yageo RC0402FR-0710KL, Resistor_SMD:R_0402_1005Metric, symbol Leshy2:UI12_UI_INPUT_UP_PULLUP
- added R5: Yageo RC0402FR-0710KL, Resistor_SMD:R_0402_1005Metric, symbol Leshy2:UI12_UI_INPUT_DOWN_PULLUP
- added R6: Yageo RC0402FR-0710KL, Resistor_SMD:R_0402_1005Metric, symbol Leshy2:UI12_UI_INPUT_LEFT_PULLUP
- added R7: Yageo RC0402FR-0710KL, Resistor_SMD:R_0402_1005Metric, symbol Leshy2:UI12_UI_INPUT_RIGHT_PULLUP
- added R8: Yageo RC0402FR-0710KL, Resistor_SMD:R_0402_1005Metric, symbol Leshy2:UI12_UI_INPUT_OK_PULLUP
- added R9: Yageo RC0402FR-073K32L, Resistor_SMD:R_0402_1005Metric, symbol Leshy2:UI12_UI_INPUT_BACK_PULLUP
- added RT1: TDK B57332V5103F360, Resistor_SMD:R_0603_1608Metric, symbol Leshy2:UI12_UI_ZONE_NTC
- added SW1: OMRON B3S-1100P, Leshy2:B3S-1100P, symbol Leshy2:UI12_UI_DPAD_UP
- added SW10: OMRON B3S-1100P, Leshy2:B3S-1100P, symbol Leshy2:UI12_UI_SWITCH_F3
- added SW11: OMRON B3S-1100P, Leshy2:B3S-1100P, symbol Leshy2:UI12_UI_SWITCH_F4
- added SW12: OMRON B3S-1100P, Leshy2:B3S-1100P, symbol Leshy2:UI12_UI_SWITCH_F5
- added SW13: OMRON B3S-1100P, Leshy2:B3S-1100P, symbol Leshy2:UI12_UI_SWITCH_F6
- added SW14: OMRON B3S-1100P, Leshy2:B3S-1100P, symbol Leshy2:UI12_UI_SWITCH_F7
- added SW15: OMRON B3S-1100P, Leshy2:B3S-1100P, symbol Leshy2:UI12_UI_SWITCH_F8
- added SW2: OMRON B3S-1100P, Leshy2:B3S-1100P, symbol Leshy2:UI12_UI_DPAD_DOWN
- added SW3: OMRON B3S-1100P, Leshy2:B3S-1100P, symbol Leshy2:UI12_UI_DPAD_LEFT
- added SW4: OMRON B3S-1100P, Leshy2:B3S-1100P, symbol Leshy2:UI12_UI_DPAD_RIGHT
- added SW5: OMRON B3S-1100P, Leshy2:B3S-1100P, symbol Leshy2:UI12_UI_DPAD_OK
- added SW6: OMRON B3S-1100P, Leshy2:B3S-1100P, symbol Leshy2:UI12_UI_SWITCH_BACK
- added SW7: OMRON B3S-1100P, Leshy2:B3S-1100P, symbol Leshy2:UI12_UI_SWITCH_OPT
- added SW8: OMRON B3S-1100P, Leshy2:B3S-1100P, symbol Leshy2:UI12_UI_SWITCH_F1
- added SW9: OMRON B3S-1100P, Leshy2:B3S-1100P, symbol Leshy2:UI12_UI_SWITCH_F2
- added U1: TCA6424ARGJR, Leshy2:TCA6424ARGJR, symbol Leshy2:UI12_SLOW_IO
- added U2: SN74LVC1G07DCKR, Package_TO_SOT_SMD:Texas_R-PDSO-G5_DCK-5, symbol Leshy2:UI12_SLOW_IO_FAULT_SENSE_ISO
- added U3: SN74LVC1G07DCKR, Package_TO_SOT_SMD:Texas_R-PDSO-G5_DCK-5, symbol Leshy2:UI12_SLOW_IO_S3_EVIDENCE_ISO
- added U4: TCA9539PWR, Package_SO:TSSOP-24_4.4x7.8mm_P0.65mm, symbol Leshy2:UI12_UI_MATRIX_IO
Connections:
- net 3V3_MAIN: now also C1.1 (END_1), C2.1 (END_1), C3.1 (END_1), C6.1 (END_1), R1.1 (END_1), R10.1 (END_1), R11.1 (END_1), R12.1 (END_1), R13.1 (END_1), R14.1 (END_1), R15.1 (END_1), R16.1 (END_1), R17.1 (END_1), R18.1 (END_1), R19.1 (END_1), R2.1 (END_1), R20.1 (END_1), R21.1 (END_1), R3.1 (END_1), R4.1 (END_1), R5.1 (END_1), R6.1 (END_1), R7.1 (END_1), R8.1 (END_1), R9.1 (END_1), U1.27 (VCCP), U1.31 (VCCI), U4.24 (VCC)
- net AON_SAFE_3V3: now also C4.1 (END_1), C5.1 (END_1), R22.1 (END_1), R23.1 (END_1), R24.1 (END_1), R25.1 (END_1), R26.1 (END_1), R27.1 (END_1), R28.1 (END_1), R29.1 (END_1), R30.1 (END_1), R31.1 (END_1), U2.5 (VCC), U3.5 (VCC)
- net AUDIO_CAPTURE_MIC_SEL: now also U1.1 (P00)
- net AUDIO_SPK_CODEC_REQ: now also U1.10 (P11)
- net AUDIO_TX_CODEC_REQ: now also U1.11 (P12)
- net CC_BAND_V1_REQ: now also U1.4 (P03)
- net CC_BAND_V2_REQ: now also U1.5 (P04)
- net CODEC_PWR_EN: now also U1.9 (P10)
- net ENCODER_A: now also R20.2 (END_2)
- net ENCODER_B: now also R21.2 (END_2)
- net EV_N0_S3: now also D3.1 (K)
- net EV_N1_C5: now also D4.1 (K)
- net EV_N2_NRF0: now also D5.1 (K)
- net EV_N3_NRF1: now also D6.1 (K)
- net EV_N4_NRF2: now also D7.1 (K)
- net EV_N5_CC: now also D8.1 (K)
- net EV_N6_VOICE: now also D9.1 (K)
- net EV_N7_IR: now also D10.1 (K)
- net EV_N8_LORA_EXT: now also D11.1 (K)
- net FAULT_LATCH_SENSE_AON: now also R32.1 (END_1), U2.2 (A)
- net HEADSET_ABSENT: now also U1.3 (P02)
- net LCD_RST_N: now also U1.7 (P06)
- net POWER_FAULT_N: now also U1.22 (P25)
- net POWER_GROUND: now also C1.2 (END_2), C2.2 (END_2), C3.2 (END_2), C6.2 (END_2), D1.9 (GND), D2.9 (GND), SW1.2 (SIDE_B_1), SW1.4 (SIDE_B_2), SW1.5 (GROUND), SW10.2 (SIDE_B_1), SW10.4 (SIDE_B_2), SW10.5 (GROUND), SW11.2 (SIDE_B_1), SW11.4 (SIDE_B_2), SW11.5 (GROUND), SW12.2 (SIDE_B_1), SW12.4 (SIDE_B_2), SW12.5 (GROUND), SW13.2 (SIDE_B_1), SW13.4 (SIDE_B_2), SW13.5 (GROUND), SW14.2 (SIDE_B_1), SW14.4 (SIDE_B_2), SW14.5 (GROUND), SW15.2 (SIDE_B_1), SW15.4 (SIDE_B_2), SW15.5 (GROUND), SW2.2 (SIDE_B_1), SW2.4 (SIDE_B_2), SW2.5 (GROUND), SW3.2 (SIDE_B_1), SW3.4 (SIDE_B_2), SW3.5 (GROUND), SW4.2 (SIDE_B_1), SW4.4 (SIDE_B_2), SW4.5 (GROUND), SW5.2 (SIDE_B_1), SW5.4 (SIDE_B_2), SW5.5 (GROUND), SW6.2 (SIDE_B_1), SW6.4 (SIDE_B_2), SW6.5 (GROUND), SW7.2 (SIDE_B_1), SW7.4 (SIDE_B_2), SW7.5 (GROUND), SW8.2 (SIDE_B_1), SW8.4 (SIDE_B_2), SW8.5 (GROUND), SW9.2 (SIDE_B_1), SW9.4 (SIDE_B_2), SW9.5 (GROUND), U1.25 (GND), U1.26 (ADDR), U1.33 (EPAD), U4.12 (GND), U4.2 (A1), U4.21 (A0)
- net RX_AUDIO_SOURCE_SEL: now also U1.24 (P27)
- net RX_DOMAIN_EN: now also U1.14 (P15)
- net RX_STATUS_N: now also U1.21 (P24)
- net S3_RESET_N: now also U4.3 (RESET_N)
- net S3_RF_TX_EVIDENCE_AON_N: now also U3.2 (A)
- net SAFETY_GROUND: now also C4.2 (END_2), C5.2 (END_2), C7.2 (END_2), D12.1 (K), RT1.2 (END_2), U2.3 (GND), U3.3 (GND)
- net SD_CARD_DETECT_N: now also U1.18 (P21)
- net SD_PWR_EN: now also U1.17 (P20)
- net SPEAKER_AMP_EN: now also U1.2 (P01)
- net SYS_I2C_SCL: now also U1.29 (SCL), U4.22 (SCL)
- net SYS_I2C_SDA: now also U1.30 (SDA), U4.23 (SDA)
- net SYS_INT_N: now also U1.32 (INT), U4.1 (INT_N)
- net TOUCH_RST_N: now also U1.8 (P07)
- net U214_5V_REQ: now also U1.16 (P17)
- net U214_I2C_READY: now also U1.15 (P16)
- net UI_ENCODER_PUSH_N: now also R19.2 (END_2), U4.15 (P12)
- net UI_ZONE_TEMP_ADC: now also C7.1 (END_1), R22.2 (END_2), RT1.1 (END_1)
- net UNIT_5V_REQ: now also U1.6 (P05)
- net UNIT_READY: now also U1.23 (P26)
- net VOICE_DOMAIN_REQ: now also U1.12 (P13)
- net VOICE_HL_RELEASE_REQ: now also U1.13 (P14)
- new net C5_TX_LED_A: D4.2 (A), R24.2 (END_2)
- new net CC_TX_LED_A: D8.2 (A), R28.2 (END_2)
- new net EXT_TX_LED_A: D11.2 (A), R31.2 (END_2)
- new net FAULT_LATCH_SENSE: R2.2 (END_2), U1.19 (P22), U2.4 (Y)
- new net FAULT_LED_A: D12.2 (A), R32.2 (END_2)
- new net IR_TX_LED_A: D10.2 (A), R30.2 (END_2)
- new net NRF0_TX_LED_A: D5.2 (A), R25.2 (END_2)
- new net NRF1_TX_LED_A: D6.2 (A), R26.2 (END_2)
- new net NRF2_TX_LED_A: D7.2 (A), R27.2 (END_2)
- new net S3_RF_TX_EVIDENCE_N: R3.2 (END_2), U1.20 (P23), U3.4 (Y)
- new net S3_TX_LED_A: D3.2 (A), R23.2 (END_2)
- new net SLOW_IO_RESET_N: R1.2 (END_2), U1.28 (RESET)
- new net UI_BACK_N: D1.6 (IO6), R9.2 (END_2), SW6.1 (SIDE_A_1), SW6.3 (SIDE_A_2), U4.9 (P05)
- new net UI_DPAD_DOWN_N: D1.2 (IO2), R5.2 (END_2), SW2.1 (SIDE_A_1), SW2.3 (SIDE_A_2), U4.5 (P01)
- new net UI_DPAD_LEFT_N: D1.3 (IO3), R6.2 (END_2), SW3.1 (SIDE_A_1), SW3.3 (SIDE_A_2), U4.6 (P02)
- new net UI_DPAD_OK_N: D1.5 (IO5), R8.2 (END_2), SW5.1 (SIDE_A_1), SW5.3 (SIDE_A_2), U4.8 (P04)
- new net UI_DPAD_RIGHT_N: D1.4 (IO4), R7.2 (END_2), SW4.1 (SIDE_A_1), SW4.3 (SIDE_A_2), U4.7 (P03)
- new net UI_DPAD_UP_N: D1.1 (IO1), R4.2 (END_2), SW1.1 (SIDE_A_1), SW1.3 (SIDE_A_2), U4.4 (P00)
- new net UI_F1_N: D2.1 (IO1), R11.2 (END_2), SW8.1 (SIDE_A_1), SW8.3 (SIDE_A_2), U4.13 (P10)
- new net UI_F2_N: D2.2 (IO2), R12.2 (END_2), SW9.1 (SIDE_A_1), SW9.3 (SIDE_A_2), U4.14 (P11)
- new net UI_F3_N: D1.8 (IO8), R13.2 (END_2), SW10.1 (SIDE_A_1), SW10.3 (SIDE_A_2), U4.11 (P07)
- new net UI_F4_N: D2.3 (IO3), R14.2 (END_2), SW11.1 (SIDE_A_1), SW11.3 (SIDE_A_2), U4.16 (P13)
- new net UI_F5_N: D2.4 (IO4), R15.2 (END_2), SW12.1 (SIDE_A_1), SW12.3 (SIDE_A_2), U4.17 (P14)
- new net UI_F6_N: D2.5 (IO5), R16.2 (END_2), SW13.1 (SIDE_A_1), SW13.3 (SIDE_A_2), U4.18 (P15)
- new net UI_F7_N: D2.6 (IO6), R17.2 (END_2), SW14.1 (SIDE_A_1), SW14.3 (SIDE_A_2), U4.19 (P16)
- new net UI_F8_N: D2.7 (IO7), R18.2 (END_2), SW15.1 (SIDE_A_1), SW15.3 (SIDE_A_2), U4.20 (P17)
- new net UI_OPT_N: D1.7 (IO7), R10.2 (END_2), SW7.1 (SIDE_A_1), SW7.3 (SIDE_A_2), U4.10 (P06)
- new net VOICE_TX_LED_A: D9.2 (A), R29.2 (END_2)
- no-connect marks 45 -> 3
Other:
- title: (none) -> Leshy2 — exact controls, safety sensing and front indicators

Commit message: complete exact H2.2.9 UI TX safety schematic
Connections:
- net S3_RF_TX_EVIDENCE_AON_N is gone; now on net EV_N0_S3: U3.2 (A)
Changed lines of the file:
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@@
 	(hierarchical_label "EV_N0_S3"
 		(shape bidirectional)
+		(at 276.86 71.12 0)
+		(effects (font (size 1.27 1.27)))
+	)
+	(label "EV_N0_S3"
 		(at 33.02 271.78 0)
 		(effects (font (size 1.27 1.27)))
@@
 		(effects (font (size 1.27 1.27)))
 	)
-	(hierarchical_label "S3_RF_TX_EVIDENCE_AON_N"
-		(shape bidirectional)
-		(at 276.86 71.12 0)
-		(effects (font (size 1.27 1.27)))
-	)

Commit message: complete exact H2.2.10 UI test points
Changed lines of the file:
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@@
 		(effects (font (size 1.27 1.27)))
 	)
-	(label "SLOW_IO_RESET_N"
+	(hierarchical_label "SLOW_IO_RESET_N"
+		(shape bidirectional)
 		(at 68.58 68.58 180)
 		(effects (font (size 1.27 1.27)) (justify right bottom))

Commit message: complete H2 schematic review package
Parts:
- renumbered C1 to C12001, C2 to C12002, C3 to C12003, C4 to C12004, C5 to C12005, C6 to C12006, C7 to C12007, D1 to D12001, D2 to D12002, D3 to D12003, D4 to D12004, D5 to D12005, D6 to D12006, D7 to D12007, D8 to D12008, D9 to D12009, D10 to D12010, D11 to D12011, D12 to D12012, R1 to R12001, R2 to R12002, R3 to R12003, R4 to R12004, R5 to R12005, R6 to R12006, R7 to R12007, R8 to R12008, R9 to R12009, R10 to R12010, R11 to R12011, R12 to R12012, R13 to R12013, R14 to R12014, R15 to R12015, R16 to R12016, R17 to R12017, R18 to R12018, R19 to R12019, R20 to R12020, R21 to R12021, R22 to R12022, R23 to R12023, R24 to R12024, R25 to R12025, R26 to R12026, R27 to R12027, R28 to R12028, R29 to R12029, R30 to R12030, R31 to R12031, R32 to R12032, RT1 to RT12001, SW1 to SW12001, SW2 to SW12002, SW3 to SW12003, SW4 to SW12004, SW5 to SW12005, SW6 to SW12006, SW7 to SW12007, SW8 to SW12008, SW9 to SW12009, SW10 to SW12010, SW11 to SW12011, SW12 to SW12012, SW13 to SW12013, SW14 to SW12014, SW15 to SW12015, U1 to U12001, U2 to U12002, U3 to U12003, U4 to U12004

Commit message: Optimize H1 display and stocked BOM routes
Parts:
- C12001, C12002, C12004, C12005, C12006, C12007: value TDK C1005X7R1H104K050BB -> Yageo CC0402KRX7R9BB104
Changed lines of the file:
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@@
 			(effects (font (size 1.27 1.27)))
 		)
-		(property "Value" "TDK C1005X7R1H104K050BB"
+		(property "Value" "Yageo CC0402KRX7R9BB104"
 			(at 132.08 49.53 0)
 			(show_name no)
@@
 			(effects (font (size 1.27 1.27)))
 		)
-		(property "Value" "TDK C1005X7R1H104K050BB"
+		(property "Value" "Yageo CC0402KRX7R9BB104"
 			(at 213.36 49.53 0)
 			(show_name no)
@@
 			(effects (font (size 1.27 1.27)))
 		)
-		(property "Value" "TDK C1005X7R1H104K050BB"
+		(property "Value" "Yageo CC0402KRX7R9BB104"
 			(at 132.08 74.93 0)
 			(show_name no)
@@
 			(effects (font (size 1.27 1.27)))
 		)
-		(property "Value" "TDK C1005X7R1H104K050BB"
+		(property "Value" "Yageo CC0402KRX7R9BB104"
 			(at 375.92 74.93 0)
 			(show_name no)
@@
 			(effects (font (size 1.27 1.27)))
 		)
-		(property "Value" "TDK C1005X7R1H104K050BB"
+		(property "Value" "Yageo CC0402KRX7R9BB104"
 			(at 213.36 184.15 0)
 			(show_name no)
@@
 			(effects (font (size 1.27 1.27)))
 		)
-		(property "Value" "TDK C1005X7R1H104K050BB"
+		(property "Value" "Yageo CC0402KRX7R9BB104"
 			(at 457.20 262.89 0)
 			(show_name no)

Commit message: Replace six pre-order resistor identities
Parts:
- R12023, R12024, R12025, R12026, R12027, R12028, R12029, R12030, R12031, R12032: value Yageo RC0402FR-072K2L -> UNI-ROYAL 0402WGF2201TCE
Changed lines of the file:
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@@
 			(effects (font (size 1.27 1.27)))
 		)
-		(property "Value" "Yageo RC0402FR-072K2L"
+		(property "Value" "UNI-ROYAL 0402WGF2201TCE"
 			(at 213.36 285.75 0)
 			(show_name no)
@@
 			(effects (font (size 1.27 1.27)))
 		)
-		(property "Value" "Yageo RC0402FR-072K2L"
+		(property "Value" "UNI-ROYAL 0402WGF2201TCE"
 			(at 132.08 288.29 0)
 			(show_name no)
@@
 			(effects (font (size 1.27 1.27)))
 		)
-		(property "Value" "Yageo RC0402FR-072K2L"
+		(property "Value" "UNI-ROYAL 0402WGF2201TCE"
 			(at 457.20 288.29 0)
 			(show_name no)
@@
 			(effects (font (size 1.27 1.27)))
 		)
-		(property "Value" "Yageo RC0402FR-072K2L"
+		(property "Value" "UNI-ROYAL 0402WGF2201TCE"
 			(at 213.36 311.15 0)
 			(show_name no)
@@
 			(effects (font (size 1.27 1.27)))
 		)
-		(property "Value" "Yageo RC0402FR-072K2L"
+		(property "Value" "UNI-ROYAL 0402WGF2201TCE"
 			(at 132.08 313.69 0)
 			(show_name no)
@@
 			(effects (font (size 1.27 1.27)))
 		)
-		(property "Value" "Yageo RC0402FR-072K2L"
+		(property "Value" "UNI-ROYAL 0402WGF2201TCE"
 			(at 457.20 313.69 0)
 			(show_name no)
@@
 			(effects (font (size 1.27 1.27)))
 		)
-		(property "Value" "Yageo RC0402FR-072K2L"
+		(property "Value" "UNI-ROYAL 0402WGF2201TCE"
 			(at 213.36 336.55 0)
 			(show_name no)
@@
 			(effects (font (size 1.27 1.27)))
 		)
-		(property "Value" "Yageo RC0402FR-072K2L"
+		(property "Value" "UNI-ROYAL 0402WGF2201TCE"
 			(at 132.08 339.09 0)
 			(show_name no)
@@
 			(effects (font (size 1.27 1.27)))
 		)
-		(property "Value" "Yageo RC0402FR-072K2L"
+		(property "Value" "UNI-ROYAL 0402WGF2201TCE"
 			(at 457.20 339.09 0)
 			(show_name no)
@@
 			(effects (font (size 1.27 1.27)))
 		)
-		(property "Value" "Yageo RC0402FR-072K2L"
+		(property "Value" "UNI-ROYAL 0402WGF2201TCE"
 			(at 213.36 361.95 0)
 			(show_name no)
