File: hardware/ecad/kicad/LESHY2-UI/UI_21_FM_AM_RECEIVER.kicad_sch (KiCad schematic)
At the start: 0 parts

Commit message: complete exact H2.2.7 broadcast receiver schematic
Parts:
- added C1: TDK C1608X7R1C105K080AC, Capacitor_SMD:C_0603_1608Metric, symbol Leshy2:UI21_SI_AUDIO_L_COUPLING
- added C10: Murata GRM1555C1H220JA01D, Capacitor_SMD:C_0402_1005Metric, symbol Leshy2:UI21_RECEIVER_CLOCK_CAP_GPO3
- added C11: Murata GRM1555C1H102JA01D, Capacitor_SMD:C_0402_1005Metric, symbol Leshy2:UI21_RECEIVER_FMI_COUPLING_CAP
- added C12: Murata GRM155R71A474KE01D, Capacitor_SMD:C_0402_1005Metric, symbol Leshy2:UI21_RECEIVER_AMI_COUPLING_CAP
- added C2: TDK C1608X7R1C105K080AC, Capacitor_SMD:C_0603_1608Metric, symbol Leshy2:UI21_SI_AUDIO_R_COUPLING
- added C3: TDK C1608X7R1C105K080AC, Capacitor_SMD:C_0603_1608Metric, symbol Leshy2:UI21_RECEIVER_POWER_INPUT_CAP
- added C4: Murata GRM188R60J106ME47D, Capacitor_SMD:C_0603_1608Metric, symbol Leshy2:UI21_RECEIVER_POWER_OUTPUT_CAP
- added C5: TDK C1005X7R1H104K050BB, Capacitor_SMD:C_0402_1005Metric, symbol Leshy2:UI21_RECEIVER_SUPERVISOR_BYPASS
- added C6: TDK C1005X7R1H104K050BB, Capacitor_SMD:C_0402_1005Metric, symbol Leshy2:UI21_RECEIVER_I2C_ISO_BYPASS
- added C7: TDK C1005X7R1H104K050BB, Capacitor_SMD:C_0402_1005Metric, symbol Leshy2:UI21_RECEIVER_IRQ_ISO_BYPASS
- added C8: TDK C1005X7R1H104K050BB, Capacitor_SMD:C_0402_1005Metric, symbol Leshy2:UI21_RECEIVER_VDD_BYPASS
- added C9: Murata GRM1555C1H220JA01D, Capacitor_SMD:C_0402_1005Metric, symbol Leshy2:UI21_RECEIVER_CLOCK_CAP_RCLK
- added D1: Littelfuse SESD0402X1UN-0020-090, Diode_SMD:D_0402_1005Metric, symbol Leshy2:UI21_RECEIVER_FMI_ESD
- added D2: Littelfuse SESD0402X1UN-0020-090, Diode_SMD:D_0402_1005Metric, symbol Leshy2:UI21_RECEIVER_AMI_ESD
- added J1: GCT RFPC-SMA31-FN-175-A, Leshy2:RFPC-SMA31-FN-175-A, symbol Leshy2:UI21_RECEIVER_FMSW_EXTERNAL_SMA
- added J2: GCT RFPC-SMA31-FN-175-A, Leshy2:RFPC-SMA31-FN-175-A, symbol Leshy2:UI21_RECEIVER_AMLW_EXTERNAL_SMA
- added L1: Murata LQW15AN56NJ00D, Inductor_SMD:L_0402_1005Metric, symbol Leshy2:UI21_RECEIVER_FMI_MATCH_INDUCTOR
- added R1: Yageo RC0402FR-0710KL, Resistor_SMD:R_0402_1005Metric, symbol Leshy2:UI21_SI_AUDIO_L_SUM
- added R2: Yageo RC0402FR-0710KL, Resistor_SMD:R_0402_1005Metric, symbol Leshy2:UI21_SI_AUDIO_R_SUM
- added R3: Yageo RC0402FR-07100KL, Resistor_SMD:R_0402_1005Metric, symbol Leshy2:UI21_SI_AUDIO_SUM_BIAS
- added R4: Yageo RC0402FR-0710KL, Resistor_SMD:R_0402_1005Metric, symbol Leshy2:UI21_RECEIVER_POWER_ON_PULLDOWN
- added R5: Yageo RC0402FR-07100KL, Resistor_SMD:R_0402_1005Metric, symbol Leshy2:UI21_RECEIVER_READY_PULLDOWN
- added R6: Yageo RC0402FR-072K2L, Resistor_SMD:R_0402_1005Metric, symbol Leshy2:UI21_RECEIVER_I2C_SCL_PULLUP
- added R7: Yageo RC0402FR-072K2L, Resistor_SMD:R_0402_1005Metric, symbol Leshy2:UI21_RECEIVER_I2C_SDA_PULLUP
- added R8: Yageo RC0402FR-0710KL, Resistor_SMD:R_0402_1005Metric, symbol Leshy2:UI21_RECEIVER_IRQ_PULLUP
- added R9: Yageo RC0402FR-0710KL, Resistor_SMD:R_0402_1005Metric, symbol Leshy2:UI21_RECEIVER_SENB_PULLDOWN
- added U1: Si4732-A10-GSR, Package_SO:SOIC-16_3.9x9.9mm_P1.27mm, symbol Leshy2:UI21_RECEIVER
- added U2: Texas Instruments TPS3839K33DBZR, Package_TO_SOT_SMD:SOT-23, symbol Leshy2:UI21_RECEIVER_SUPERVISOR
- added U3: Texas Instruments SN74LVC2G66DCUR, Package_SO:VSSOP-8_2.3x2mm_P0.5mm, symbol Leshy2:UI21_RECEIVER_I2C_ISO
- added U4: SN74LVC1G07DCKR, Package_TO_SOT_SMD:Texas_R-PDSO-G5_DCK-5, symbol Leshy2:UI21_RECEIVER_IRQ_ISO
- added U5: Texas Instruments TPS22919DCKR, Package_TO_SOT_SMD:SOT-363_SC-70-6, symbol Leshy2:UI21_RECEIVER_POWER_SWITCH
- added Y1: Seiko Epson Q13FC13500005, Leshy2:FC-135-Q13FC13500005, symbol Leshy2:UI21_RECEIVER_CLOCK
Connections:
- net 3V3_MAIN: now also C3.1 (END_1), C6.1 (END_1), R8.1 (END_1), U3.8 (VCC), U5.1 (IN)
- net AUDIO_VMID_MAIN: now also R3.2 (END_2)
- net POWER_GROUND: now also C10.2 (END_2), C3.2 (END_2), C4.2 (END_2), C5.2 (END_2), C6.2 (END_2), C7.2 (END_2), C8.2 (END_2), C9.2 (END_2), D1.2 (A), D2.2 (A), J1.2 (GROUND_TOP_LEFT), J1.3 (GROUND_TOP_RIGHT), J1.4 (GROUND_BOTTOM_LEFT), J1.5 (GROUND_BOTTOM_RIGHT), J2.2 (GROUND_TOP_LEFT), J2.3 (GROUND_TOP_RIGHT), J2.4 (GROUND_BOTTOM_LEFT), J2.5 (GROUND_BOTTOM_RIGHT), R4.2 (END_2), R5.2 (END_2), R9.2 (END_2), U1.15 (GND), U1.7 (RFGND), U2.2 (GND), U3.4 (GND), U4.3 (GND), U5.2 (GND)
- net RX_DOMAIN_EN: now also R4.1 (END_1), U5.3 (ON)
- net RX_SI4732_MONO: now also R1.2 (END_2), R2.2 (END_2), R3.1 (END_1)
- net RX_STATUS_N: now also R8.2 (END_2), U4.4 (Y)
- net SYS_I2C_SCL: now also U3.5 (2A)
- net SYS_I2C_SDA: now also U3.1 (1A)
- new net 3V3_RECEIVER_SWITCHED: C4.1 (END_1), C5.1 (END_1), C7.1 (END_1), C8.1 (END_1), R6.1 (END_1), R7.1 (END_1), U1.14 (VDD), U2.3 (VDD), U4.5 (VCC), U5.5 (QOD), U5.6 (VOUT)
- new net RECEIVER_READY: R5.1 (END_1), U1.9 (RST), U2.1 (RESET_N), U3.3 (2C), U3.7 (1C)
- new net RX_AMI_RF: C12.2 (END_2), U1.8 (AMI)
- new net RX_AMLW_BOUNDARY_RF: C12.1 (END_1), D2.1 (K), J2.1 (RF)
- new net RX_AUDIO_L: C1.1 (END_1), U1.1 (LOUT_DFS)
- new net RX_AUDIO_L_AC: C1.2 (END_2), R1.1 (END_1)
- new net RX_AUDIO_R: C2.1 (END_1), U1.16 (ROUT_DOUT)
- new net RX_AUDIO_R_AC: C2.2 (END_2), R2.1 (END_1)
- new net RX_FMI_RF: C11.2 (END_2), U1.6 (FMI)
- new net RX_FMSW_BOUNDARY_RF: D1.1 (K), J1.1 (RF), L1.1 (END_1)
- new net RX_FMSW_MATCHED_RF: C11.1 (END_1), L1.2 (END_2)
- new net RX_I2C_SCL: R6.2 (END_2), U1.11 (SCLK), U3.6 (2B)
- new net RX_I2C_SDA: R7.2 (END_2), U1.12 (SDIO), U3.2 (1B)
- new net RX_SENB_LOW: R9.1 (END_1), U1.10 (SENB)
- new net RX_STATUS_LOCAL_N: U1.3 (GPO2_INTB), U4.2 (A)
- new net RX_XTAL_GPO3: C10.1 (END_1), U1.2 (GPO3_DCLK), Y1.2 (X2)
- new net RX_XTAL_RCLK: C9.1 (END_1), U1.13 (RCLK), Y1.1 (X1)
- no-connect marks 8 -> 4
Other:
- title: (none) -> Leshy2 — exact FM/AM/SW/LW receive-only frontend

Commit message: complete H2 schematic review package
Parts:
- renumbered C1 to C21001, C2 to C21002, C3 to C21003, C4 to C21004, C5 to C21005, C6 to C21006, C7 to C21007, C8 to C21008, C9 to C21009, C10 to C21010, C11 to C21011, C12 to C21012, D1 to D21001, D2 to D21002, J1 to J21001, J2 to J21002, L1 to L21001, R1 to R21001, R2 to R21002, R3 to R21003, R4 to R21004, R5 to R21005, R6 to R21006, R7 to R21007, R8 to R21008, R9 to R21009, U1 to U21001, U2 to U21002, U3 to U21003, U4 to U21004, U5 to U21005, Y1 to Y21001
Changed lines of the file:
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@@
 		(on_board yes)
 		(dnp no)
-		(property "Reference" "J1"
+		(property "Reference" "J21001"
 			(at 50.80 40.64 0)
 			(show_name no)
@@
 			(project "LESHY2-UI"
 				(path "/b1abf8d4-4004-5a36-a895-3c09708b05a5"
-					(reference "J1")
+					(reference "J21001")
 					(unit 1)
 				)
@@
 		(on_board yes)
 		(dnp no)
-		(property "Reference" "J2"
+		(property "Reference" "J21002"
 			(at 132.08 40.64 0)
 			(show_name no)
@@
 			(project "LESHY2-UI"
 				(path "/b1abf8d4-4004-5a36-a895-3c09708b05a5"
-					(reference "J2")
+					(reference "J21002")
 					(unit 1)
 				)
@@
 		(on_board yes)
 		(dnp no)
-		(property "Reference" "U1"
+		(property "Reference" "U21001"
 			(at 213.36 40.87 0)
 			(show_name no)
@@
 			(project "LESHY2-UI"
 				(path "/b1abf8d4-4004-5a36-a895-3c09708b05a5"
-					(reference "U1")
+					(reference "U21001")
 					(unit 1)
 				)
@@
 		(on_board yes)
 		(dnp no)
-		(property "Reference" "C1"
+		(property "Reference" "C21001"
 			(at 294.64 39.37 0)
 			(show_name no)
@@
 			(project "LESHY2-UI"
 				(path "/b1abf8d4-4004-5a36-a895-3c09708b05a5"
-					(reference "C1")
+					(reference "C21001")
 					(unit 1)
 				)
@@
 		(on_board yes)
 		(dnp no)
-		(property "Reference" "C2"
+		(property "Reference" "C21002"
 			(at 375.92 39.37 0)
 			(show_name no)
@@
 			(project "LESHY2-UI"
 				(path "/b1abf8d4-4004-5a36-a895-3c09708b05a5"
-					(reference "C2")
+					(reference "C21002")
 					(unit 1)
 				)
@@
 		(on_board yes)
 		(dnp no)
-		(property "Reference" "R1"
+		(property "Reference" "R21001"
 			(at 457.20 39.37 0)
 			(show_name no)
@@
 			(project "LESHY2-UI"
 				(path "/b1abf8d4-4004-5a36-a895-3c09708b05a5"
-					(reference "R1")
+					(reference "R21001")
 					(unit 1)
 				)
@@
 		(on_board yes)
 		(dnp no)
-		(property "Reference" "R2"
+		(property "Reference" "R21002"
 			(at 294.64 64.77 0)
 			(show_name no)
@@
 			(project "LESHY2-UI"
 				(path "/b1abf8d4-4004-5a36-a895-3c09708b05a5"
-					(reference "R2")
+					(reference "R21002")
 					(unit 1)
 				)
@@
 		(on_board yes)
 		(dnp no)
-		(property "Reference" "R3"
+		(property "Reference" "R21003"
 			(at 375.92 64.77 0)
 			(show_name no)
@@
 			(project "LESHY2-UI"
 				(path "/b1abf8d4-4004-5a36-a895-3c09708b05a5"
-					(reference "R3")
+					(reference "R21003")
 					(unit 1)
 				)
@@
 		(on_board yes)
 		(dnp no)
-		(property "Reference" "C3"
+		(property "Reference" "C21003"
 			(at 457.20 64.77 0)
 			(show_name no)
@@
 			(project "LESHY2-UI"
 				(path "/b1abf8d4-4004-5a36-a895-3c09708b05a5"
-					(reference "C3")
+					(reference "C21003")
 					(unit 1)
 				)
@@
 		(on_board yes)
 		(dnp no)
-		(property "Reference" "C4"
+		(property "Reference" "C21004"
 			(at 50.80 67.31 0)
 			(show_name no)
@@
 			(project "LESHY2-UI"
 				(path "/b1abf8d4-4004-5a36-a895-3c09708b05a5"
-					(reference "C4")
+					(reference "C21004")
 					(unit 1)
 				)
@@
 		(on_board yes)
 		(dnp no)
-		(property "Reference" "R4"
+		(property "Reference" "R21004"
 			(at 132.08 67.31 0)
 			(show_name no)
@@
 			(project "LESHY2-UI"
 				(path "/b1abf8d4-4004-5a36-a895-3c09708b05a5"
-					(reference "R4")
+					(reference "R21004")
 					(unit 1)
 				)
@@
 		(on_board yes)
 		(dnp no)
-		(property "Reference" "U2"
+		(property "Reference" "U21002"
 			(at 213.36 80.01 0)
 			(show_name no)
@@
 			(project "LESHY2-UI"
 				(path "/b1abf8d4-4004-5a36-a895-3c09708b05a5"
-					(reference "U2")
+					(reference "U21002")
 					(unit 1)
 				)
@@
 		(on_board yes)
 		(dnp no)
-		(property "Reference" "C5"
+		(property "Reference" "C21005"
 			(at 294.64 90.17 0)
 			(show_name no)
@@
 			(project "LESHY2-UI"
 				(path "/b1abf8d4-4004-5a36-a895-3c09708b05a5"
-					(reference "C5")
+					(reference "C21005")
 					(unit 1)
 				)
@@
 		(on_board yes)
 		(dnp no)
-		(property "Reference" "R5"
+		(property "Reference" "R21005"
 			(at 375.92 90.17 0)
 			(show_name no)
@@
 			(project "LESHY2-UI"
 				(path "/b1abf8d4-4004-5a36-a895-3c09708b05a5"
-					(reference "R5")
+					(reference "R21005")
 					(unit 1)
 				)
@@
 		(on_board yes)
 		(dnp no)
-		(property "Reference" "U3"
+		(property "Reference" "U21003"
 			(at 457.20 92.19 0)
 			(show_name no)
@@
 			(project "LESHY2-UI"
 				(path "/b1abf8d4-4004-5a36-a895-3c09708b05a5"
-					(reference "U3")
+					(reference "U21003")
 					(unit 1)
 				)
@@
 		(on_board yes)
 		(dnp no)
-		(property "Reference" "C6"
+		(property "Reference" "C21006"
 			(at 50.80 92.71 0)
 			(show_name no)
@@
 			(project "LESHY2-UI"
 				(path "/b1abf8d4-4004-5a36-a895-3c09708b05a5"
-					(reference "C6")
+					(reference "C21006")
 					(unit 1)
 				)
@@
 		(on_board yes)
 		(dnp no)
-		(property "Reference" "R6"
+		(property "Reference" "R21006"
 			(at 132.08 92.71 0)
 			(show_name no)
@@
 			(project "LESHY2-UI"
 				(path "/b1abf8d4-4004-5a36-a895-3c09708b05a5"
-					(reference "R6")
+					(reference "R21006")
 					(unit 1)
 				)
@@
 		(on_board yes)
 		(dnp no)
-		(property "Reference" "R7"
+		(property "Reference" "R21007"
 			(at 213.36 105.41 0)
 			(show_name no)
@@
 			(project "LESHY2-UI"
 				(path "/b1abf8d4-4004-5a36-a895-3c09708b05a5"
-					(reference "R7")
+					(reference "R21007")
 					(unit 1)
 				)
@@
 		(on_board yes)
 		(dnp no)
-		(property "Reference" "U4"
+		(property "Reference" "U21004"
 			(at 294.64 116.84 0)
 			(show_name no)
@@
 			(project "LESHY2-UI"
 				(path "/b1abf8d4-4004-5a36-a895-3c09708b05a5"
-					(reference "U4")
+					(reference "U21004")
 					(unit 1)
 				)
@@
 		(on_board yes)
 		(dnp no)
-		(property "Reference" "C7"
+		(property "Reference" "C21007"
 			(at 375.92 115.57 0)
 			(show_name no)
@@
 			(project "LESHY2-UI"
 				(path "/b1abf8d4-4004-5a36-a895-3c09708b05a5"
-					(reference "C7")
+					(reference "C21007")
 					(unit 1)
 				)
@@
 		(on_board yes)
 		(dnp no)
-		(property "Reference" "R8"
+		(property "Reference" "R21008"
 			(at 50.80 118.11 0)
 			(show_name no)
@@
 			(project "LESHY2-UI"
 				(path "/b1abf8d4-4004-5a36-a895-3c09708b05a5"
-					(reference "R8")
+					(reference "R21008")
 					(unit 1)
 				)
@@
 		(on_board yes)
 		(dnp no)
-		(property "Reference" "C8"
+		(property "Reference" "C21008"
 			(at 132.08 118.11 0)
 			(show_name no)
@@
 			(project "LESHY2-UI"
 				(path "/b1abf8d4-4004-5a36-a895-3c09708b05a5"
-					(reference "C8")
+					(reference "C21008")
 					(unit 1)
 				)
@@
 		(on_board yes)
 		(dnp no)
-		(property "Reference" "Y1"
+		(property "Reference" "Y21001"
 			(at 457.20 120.65 0)
 			(show_name no)
@@
 			(project "LESHY2-UI"
 				(path "/b1abf8d4-4004-5a36-a895-3c09708b05a5"
-					(reference "Y1")
+					(reference "Y21001")
 					(unit 1)
 				)
@@
 		(on_board yes)
 		(dnp no)
-		(property "Reference" "C9"
+		(property "Reference" "C21009"
 			(at 213.36 130.81 0)
 			(show_name no)
@@
 			(project "LESHY2-UI"
 				(path "/b1abf8d4-4004-5a36-a895-3c09708b05a5"
-					(reference "C9")
+					(reference "C21009")
 					(unit 1)
 				)
@@
 		(on_board yes)
 		(dnp no)
-		(property "Reference" "C10"
+		(property "Reference" "C21010"
 			(at 375.92 140.97 0)
 			(show_name no)
@@
 			(project "LESHY2-UI"
 				(path "/b1abf8d4-4004-5a36-a895-3c09708b05a5"
-					(reference "C10")
+					(reference "C21010")
 					(unit 1)
 				)
@@
 		(on_board yes)
 		(dnp no)
-		(property "Reference" "R9"
+		(property "Reference" "R21009"
 			(at 50.80 143.51 0)
 			(show_name no)
@@
 			(project "LESHY2-UI"
 				(path "/b1abf8d4-4004-5a36-a895-3c09708b05a5"
-					(reference "R9")
+					(reference "R21009")
 					(unit 1)
 				)
@@
 		(on_board yes)
 		(dnp no)
-		(property "Reference" "D1"
+		(property "Reference" "D21001"
 			(at 132.08 143.51 0)
 			(show_name no)
@@
 			(project "LESHY2-UI"
 				(path "/b1abf8d4-4004-5a36-a895-3c09708b05a5"
-					(reference "D1")
+					(reference "D21001")
 					(unit 1)
 				)
@@
 		(on_board yes)
 		(dnp no)
-		(property "Reference" "L1"
+		(property "Reference" "L21001"
 			(at 294.64 143.51 0)
 			(show_name no)
@@
 			(project "LESHY2-UI"
 				(path "/b1abf8d4-4004-5a36-a895-3c09708b05a5"
-					(reference "L1")
+					(reference "L21001")
 					(unit 1)
 				)
@@
 		(on_board yes)
 		(dnp no)
-		(property "Reference" "C11"
+		(property "Reference" "C21011"
 			(at 457.20 146.05 0)
 			(show_name no)
@@
 			(project "LESHY2-UI"
 				(path "/b1abf8d4-4004-5a36-a895-3c09708b05a5"
-					(reference "C11")
+					(reference "C21011")
 					(unit 1)
 				)
@@
 		(on_board yes)
 		(dnp no)
-		(property "Reference" "D2"
+		(property "Reference" "D21002"
 			(at 213.36 156.21 0)
 			(show_name no)
@@
 			(project "LESHY2-UI"
 				(path "/b1abf8d4-4004-5a36-a895-3c09708b05a5"
-					(reference "D2")
+					(reference "D21002")
 					(unit 1)
 				)
@@
 		(on_board yes)
 		(dnp no)
-		(property "Reference" "C12"
+		(property "Reference" "C21012"
 			(at 375.92 166.37 0)
 			(show_name no)
@@
 			(project "LESHY2-UI"
 				(path "/b1abf8d4-4004-5a36-a895-3c09708b05a5"
-					(reference "C12")
+					(reference "C21012")
 					(unit 1)
 				)
@@
 		(on_board yes)
 		(dnp no)
-		(property "Reference" "U5"
+		(property "Reference" "U21005"
 			(at 50.80 170.18 0)
 			(show_name no)
@@
 			(project "LESHY2-UI"
 				(path "/b1abf8d4-4004-5a36-a895-3c09708b05a5"
-					(reference "U5")
-					(unit 1)
-				)
+					(reference "U21005")
+					(unit 1)
+				)

Commit message: Optimize H1 display and stocked BOM routes
Parts:
- C21005, C21006, C21007, C21008: value TDK C1005X7R1H104K050BB -> Yageo CC0402KRX7R9BB104
Changed lines of the file:
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@@
 			(effects (font (size 1.27 1.27)))
 		)
-		(property "Value" "TDK C1005X7R1H104K050BB"
+		(property "Value" "Yageo CC0402KRX7R9BB104"
 			(at 294.64 100.33 0)
 			(show_name no)
@@
 			(effects (font (size 1.27 1.27)))
 		)
-		(property "Value" "TDK C1005X7R1H104K050BB"
+		(property "Value" "Yageo CC0402KRX7R9BB104"
 			(at 50.80 102.87 0)
 			(show_name no)
@@
 			(effects (font (size 1.27 1.27)))
 		)
-		(property "Value" "TDK C1005X7R1H104K050BB"
+		(property "Value" "Yageo CC0402KRX7R9BB104"
 			(at 375.92 125.73 0)
 			(show_name no)
@@
 			(effects (font (size 1.27 1.27)))
 		)
-		(property "Value" "TDK C1005X7R1H104K050BB"
+		(property "Value" "Yageo CC0402KRX7R9BB104"
 			(at 132.08 128.27 0)
 			(show_name no)

Commit message: Replace six pre-order resistor identities
Parts:
- R21006, R21007: value Yageo RC0402FR-072K2L -> UNI-ROYAL 0402WGF2201TCE
Changed lines of the file:
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@@
 			(effects (font (size 1.27 1.27)))
 		)
-		(property "Value" "Yageo RC0402FR-072K2L"
+		(property "Value" "UNI-ROYAL 0402WGF2201TCE"
 			(at 132.08 102.87 0)
 			(show_name no)
@@
 			(effects (font (size 1.27 1.27)))
 		)
-		(property "Value" "Yageo RC0402FR-072K2L"
+		(property "Value" "UNI-ROYAL 0402WGF2201TCE"
 			(at 213.36 115.57 0)
 			(show_name no)

Commit message: Reduce factory BOM cost without functional loss
Parts:
- L21001: value Murata LQW15AN56NJ00D -> Murata LQW15AN56NG00D
Changed lines of the file:
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@@
 			(effects (font (size 1.27 1.27)))
 		)
-		(property "Value" "Murata LQW15AN56NJ00D"
+		(property "Value" "Murata LQW15AN56NG00D"
 			(at 294.64 153.67 0)
 			(show_name no)
@@
 			(effects (font (size 1.27 1.27)))
 		)
-		(property "Description" "56nh_5pct_high_q_rf_inductor_0402"
+		(property "Description" "56nh_2pct_high_q_rf_inductor_0402"
 			(at 294.64 148.59 0)
 			(show_name no)
