File: hardware/ecad/kicad/LESHY2-UI/UI_20_C5_RADIO_IR_SERVICE.kicad_sch (KiCad schematic)
At the start: 61 parts, among them J20001 GCT RFPC-SMA32-FN-175-A, J20002 Hirose U.FL-R-SMT-1(10), J20003 GCT USB4105-GF-A, J20004 Samtec FTSH-105-01-L-DV-K-P-TR, Q20001 Diodes Incorporated DMN2056U-7, SW20001 Alps Alpine SKRTLAE010, SW20002 Alps Alpine SKRTLAE010, U20001 ESP32-C5-WROOM-1U-N8R8, U20002 KYOCERA AVX CP0603Q5425ENTR, U20003 Texas Instruments TPS22919DCKR, U20004 Vishay TSOP75238TT, U20005 Vishay TSMP95000TT, U20006 Nexperia 74LVC2G126DC,125, U20007 onsemi FSUSB42MUX, U20008 SN74LVC1G08DCKR, X20001 ESP32-C5-WROOM-1U-N8R8 factor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

Commit message: Optimize H1 display and stocked BOM routes
Parts:
- C20003, C20006, C20009, C20010, C20011: value TDK C1005X7R1H104K050BB -> Yageo CC0402KRX7R9BB104
- U20006: value Nexperia 74LVC2G126DC,125 -> Nexperia 74LVC2G126DP,125; footprint Package_SO:VSSOP-8_2.3x2mm_P0.5mm -> Package_SO:TSSOP-8_3x3mm_P0.65mm
Changed lines of the file:
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@@
 			(effects (font (size 1.27 1.27)))
 		)
-		(property "Value" "TDK C1005X7R1H104K050BB"
+		(property "Value" "Yageo CC0402KRX7R9BB104"
 			(at 330.20 74.93 0)
 			(show_name no)
@@
 			(effects (font (size 1.27 1.27)))
 		)
-		(property "Value" "TDK C1005X7R1H104K050BB"
+		(property "Value" "Yageo CC0402KRX7R9BB104"
 			(at 116.84 77.47 0)
 			(show_name no)
@@
 			(effects (font (size 1.27 1.27)))
 		)
-		(property "Value" "Nexperia 74LVC2G126DC,125"
+		(property "Value" "Nexperia 74LVC2G126DP,125"
 			(at 187.96 128.79 0)
 			(show_name no)
@@
 			(effects (font (size 1.27 1.27)))
 		)
-		(property "Footprint" "Package_SO:VSSOP-8_2.3x2mm_P0.5mm"
+		(property "Footprint" "Package_SO:TSSOP-8_3x3mm_P0.65mm"
 			(at 187.96 123.19 0)
 			(show_name no)
@@
 			(effects (font (size 1.27 1.27)))
 		)
-		(property "Description" "vssop8_dual_noninverting_three_state_buffer_with_ioff"
+		(property "Description" "tssop8_dual_noninverting_three_state_buffer_with_ioff"
 			(at 187.96 123.19 0)
 			(show_name no)
@@
 			(effects (font (size 1.27 1.27)))
 		)
-		(property "Value" "TDK C1005X7R1H104K050BB"
+		(property "Value" "Yageo CC0402KRX7R9BB104"
 			(at 259.08 125.73 0)
 			(show_name no)
@@
 			(effects (font (size 1.27 1.27)))
 		)
-		(property "Value" "TDK C1005X7R1H104K050BB"
+		(property "Value" "Yageo CC0402KRX7R9BB104"
 			(at 45.72 161.29 0)
 			(show_name no)
@@
 			(effects (font (size 1.27 1.27)))
 		)
-		(property "Value" "TDK C1005X7R1H104K050BB"
+		(property "Value" "Yageo CC0402KRX7R9BB104"
 			(at 401.32 229.87 0)
 			(show_name no)

Commit message: Replace three pre-order passive parts
Parts:
- U20007: renamed from R20012; value Yageo RC1206FR-0747RL -> FH RS-06K47R0FT
- renumbered R20013 to R20012, R20014 to R20013, R20015 to R20014, R20016 to R20015, R20017 to R20016, R20018 to R20017, R20019 to R20018, R20020 to R20019, R20021 to R20020, R20022 to R20021, R20023 to R20022, R20024 to R20023, R20025 to R20024, R20026 to R20025, R20027 to R20026, R20028 to R20027, R20029 to R20028, R20030 to R20029, U20007 to U20008, U20008 to U20009
Changed lines of the file:
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@@
 		(on_board yes)
 		(dnp no)
-		(property "Reference" "R20012"
+		(property "Reference" "U20007"
 			(at 45.72 125.73 0)
 			(show_name no)
@@
 			(effects (font (size 1.27 1.27)))
 		)
-		(property "Value" "Yageo RC1206FR-0747RL"
+		(property "Value" "FH RS-06K47R0FT"
 			(at 45.72 135.89 0)
 			(show_name no)
@@
 			(project "LESHY2-UI"
 				(path "/cfff0690-e8b4-57c0-a4b3-e43b652c1ac8"
-					(reference "R20012")
+					(reference "U20007")
 					(unit 1)
 				)
@@
 		(on_board yes)
 		(dnp no)
-		(property "Reference" "R20013"
+		(property "Reference" "R20012"
 			(at 330.20 140.97 0)
 			(show_name no)
@@
 			(project "LESHY2-UI"
 				(path "/cfff0690-e8b4-57c0-a4b3-e43b652c1ac8"
-					(reference "R20013")
+					(reference "R20012")
 					(unit 1)
 				)
@@
 		(on_board yes)
 		(dnp no)
-		(property "Reference" "R20014"
+		(property "Reference" "R20013"
 			(at 472.44 140.97 0)
 			(show_name no)
@@
 			(project "LESHY2-UI"
 				(path "/cfff0690-e8b4-57c0-a4b3-e43b652c1ac8"
-					(reference "R20014")
+					(reference "R20013")
 					(unit 1)
 				)
@@
 		(on_board yes)
 		(dnp no)
-		(property "Reference" "R20015"
+		(property "Reference" "R20014"
 			(at 543.56 140.97 0)
 			(show_name no)
@@
 			(project "LESHY2-UI"
 				(path "/cfff0690-e8b4-57c0-a4b3-e43b652c1ac8"
-					(reference "R20015")
+					(reference "R20014")
 					(unit 1)
 				)
@@
 		(on_board yes)
 		(dnp no)
-		(property "Reference" "U20007"
+		(property "Reference" "U20008"
 			(at 187.96 147.94 0)
 			(show_name no)
@@
 			(project "LESHY2-UI"
 				(path "/cfff0690-e8b4-57c0-a4b3-e43b652c1ac8"
-					(reference "U20007")
+					(reference "U20008")
 					(unit 1)
 				)
@@
 		(on_board yes)
 		(dnp no)
-		(property "Reference" "R20016"
+		(property "Reference" "R20015"
 			(at 259.08 166.37 0)
 			(show_name no)
@@
 			(project "LESHY2-UI"
 				(path "/cfff0690-e8b4-57c0-a4b3-e43b652c1ac8"
-					(reference "R20016")
+					(reference "R20015")
 					(unit 1)
 				)
@@
 		(on_board yes)
 		(dnp no)
-		(property "Reference" "R20017"
+		(property "Reference" "R20016"
 			(at 330.20 166.37 0)
 			(show_name no)
@@
 			(project "LESHY2-UI"
 				(path "/cfff0690-e8b4-57c0-a4b3-e43b652c1ac8"
-					(reference "R20017")
+					(reference "R20016")
 					(unit 1)
 				)
@@
 		(on_board yes)
 		(dnp no)
-		(property "Reference" "R20018"
+		(property "Reference" "R20017"
 			(at 472.44 166.37 0)
 			(show_name no)
@@
 			(project "LESHY2-UI"
 				(path "/cfff0690-e8b4-57c0-a4b3-e43b652c1ac8"
-					(reference "R20018")
+					(reference "R20017")
 					(unit 1)
 				)
@@
 		(on_board yes)
 		(dnp no)
-		(property "Reference" "R20019"
+		(property "Reference" "R20018"
 			(at 543.56 166.37 0)
 			(show_name no)
@@
 			(project "LESHY2-UI"
 				(path "/cfff0690-e8b4-57c0-a4b3-e43b652c1ac8"
-					(reference "R20019")
+					(reference "R20018")
 					(unit 1)
 				)
@@
 		(on_board yes)
 		(dnp no)
-		(property "Reference" "R20020"
+		(property "Reference" "R20019"
 			(at 401.32 168.91 0)
 			(show_name no)
@@
 			(project "LESHY2-UI"
 				(path "/cfff0690-e8b4-57c0-a4b3-e43b652c1ac8"
-					(reference "R20020")
+					(reference "R20019")
 					(unit 1)
 				)
@@
 		(on_board yes)
 		(dnp no)
-		(property "Reference" "R20021"
+		(property "Reference" "R20020"
 			(at 330.20 191.77 0)
 			(show_name no)
@@
 			(project "LESHY2-UI"
 				(path "/cfff0690-e8b4-57c0-a4b3-e43b652c1ac8"
-					(reference "R20021")
+					(reference "R20020")
 					(unit 1)
 				)
@@
 		(on_board yes)
 		(dnp no)
-		(property "Reference" "R20022"
+		(property "Reference" "R20021"
 			(at 472.44 191.77 0)
 			(show_name no)
@@
 			(project "LESHY2-UI"
 				(path "/cfff0690-e8b4-57c0-a4b3-e43b652c1ac8"
-					(reference "R20022")
+					(reference "R20021")
 					(unit 1)
 				)
@@
 		(on_board yes)
 		(dnp no)
-		(property "Reference" "R20023"
+		(property "Reference" "R20022"
 			(at 543.56 191.77 0)
 			(show_name no)
@@
 			(project "LESHY2-UI"
 				(path "/cfff0690-e8b4-57c0-a4b3-e43b652c1ac8"
-					(reference "R20023")
+					(reference "R20022")
 					(unit 1)
 				)
@@
 		(on_board yes)
 		(dnp no)
-		(property "Reference" "R20024"
+		(property "Reference" "R20023"
 			(at 401.32 194.31 0)
 			(show_name no)
@@
 			(project "LESHY2-UI"
 				(path "/cfff0690-e8b4-57c0-a4b3-e43b652c1ac8"
-					(reference "R20024")
+					(reference "R20023")
 					(unit 1)
 				)
@@
 		(on_board yes)
 		(dnp no)
-		(property "Reference" "R20025"
+		(property "Reference" "R20024"
 			(at 45.72 209.55 0)
 			(show_name no)
@@
 			(project "LESHY2-UI"
 				(path "/cfff0690-e8b4-57c0-a4b3-e43b652c1ac8"
-					(reference "R20025")
+					(reference "R20024")
 					(unit 1)
 				)
@@
 		(on_board yes)
 		(dnp no)
-		(property "Reference" "R20026"
+		(property "Reference" "R20025"
 			(at 116.84 212.09 0)
 			(show_name no)
@@
 			(project "LESHY2-UI"
 				(path "/cfff0690-e8b4-57c0-a4b3-e43b652c1ac8"
-					(reference "R20026")
+					(reference "R20025")
 					(unit 1)
 				)
@@
 		(on_board yes)
 		(dnp no)
-		(property "Reference" "R20027"
+		(property "Reference" "R20026"
 			(at 187.96 212.09 0)
 			(show_name no)
@@
 			(project "LESHY2-UI"
 				(path "/cfff0690-e8b4-57c0-a4b3-e43b652c1ac8"
-					(reference "R20027")
+					(reference "R20026")
 					(unit 1)
 				)
@@
 		(on_board yes)
 		(dnp no)
-		(property "Reference" "R20028"
+		(property "Reference" "R20027"
 			(at 259.08 217.17 0)
 			(show_name no)
@@
 			(project "LESHY2-UI"
 				(path "/cfff0690-e8b4-57c0-a4b3-e43b652c1ac8"
-					(reference "R20028")
+					(reference "R20027")
 					(unit 1)
 				)
@@
 		(on_board yes)
 		(dnp no)
-		(property "Reference" "R20029"
+		(property "Reference" "R20028"
 			(at 330.20 217.17 0)
 			(show_name no)
@@
 			(project "LESHY2-UI"
 				(path "/cfff0690-e8b4-57c0-a4b3-e43b652c1ac8"
-					(reference "R20029")
+					(reference "R20028")
 					(unit 1)
 				)
@@
 		(on_board yes)
 		(dnp no)
-		(property "Reference" "R20030"
+		(property "Reference" "R20029"
 			(at 472.44 217.17 0)
 			(show_name no)
@@
 			(project "LESHY2-UI"
 				(path "/cfff0690-e8b4-57c0-a4b3-e43b652c1ac8"
-					(reference "R20030")
+					(reference "R20029")
 					(unit 1)
 				)
@@
 		(on_board yes)
 		(dnp no)
-		(property "Reference" "U20008"
+		(property "Reference" "U20009"
 			(at 543.56 218.44 0)
 			(show_name no)
@@
 			(project "LESHY2-UI"
 				(path "/cfff0690-e8b4-57c0-a4b3-e43b652c1ac8"
-					(reference "U20008")
-					(unit 1)
-				)
+					(reference "U20009")
+					(unit 1)
+				)

Commit message: Reduce factory BOM cost without functional loss
Parts:
- U20004: value Vishay TSOP75238TT -> Vishay TSOP75238TR
Changed lines of the file:
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@@
 			(effects (font (size 1.27 1.27)))
 		)
-		(property "Value" "Vishay TSOP75238TT"
+		(property "Value" "Vishay TSOP75238TR"
 			(at 259.08 100.33 0)
 			(show_name no)

Commit message: Audit top 20 costs and accept stocked U.FL route
Parts:
- J20002: value Hirose U.FL-R-SMT-1(10) -> Hirose U.FL-R-SMT-1(80)
Changed lines of the file:
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@@
 			(effects (font (size 1.27 1.27)))
 		)
-		(property "Value" "Hirose U.FL-R-SMT-1(10)"
+		(property "Value" "Hirose U.FL-R-SMT-1(80)"
 			(at 259.08 49.53 0)
 			(show_name no)
