File: hardware/ecad/kicad/LESHY2-RF-R2/LESHY2-RF-R2.kicad_sch (KiCad schematic)
At the start: 0 parts

Commit message: Connect RF emergency reset to active RP reset net
Other:
- sheet RF_10_RP2354_CORE_SERVICE ports: added RF_RP_RESET_N; removed none
- sheet RF_50_TX_SAFETY_EVIDENCE ports: added RF_RP_RESET_N; removed none

Commit message: Review R2 startup and fault-display sequencing
Other:
- sheet RF_40_INTERBOARD_M1 ports: added S3_RESET_KILL_GATE; removed none
- sheet RF_50_TX_SAFETY_EVIDENCE ports: added S3_RESET_KILL_GATE; removed none

Commit message: Review R2 power transitions and watchdog
Other:
- sheet RF_40_INTERBOARD_M1 ports: added FAULT_KILL; removed none
- sheet RF_50_TX_SAFETY_EVIDENCE ports: added FAULT_KILL; removed none

Commit message: Complete current R2 schematic and sourcing revalidation
Other:
- sheet RF_10_RP2354_CORE_SERVICE ports: added CAP_PIN10_HOST; removed CAP_PIN10_BUSY_OR_NFC_CS_N
- sheet RF_30_U214_U219_M5_EXT ports: added CAP_PIN10_HOST, EV_N9_U219_NFC; removed CAP_PIN10_BUSY_OR_NFC_CS_N
- sheet RF_50_TX_SAFETY_EVIDENCE ports: added EV_N9_U219_NFC; removed none

Commit message: Bind H6 RF and USB routing geometry
Other:
- sheet RF_01_USB_PD_CHARGE ports: added S3_USB_N, S3_USB_P; removed S3_USB_DM, S3_USB_DP
- sheet RF_40_INTERBOARD_M1 ports: added S3_USB_N, S3_USB_P; removed S3_USB_DM, S3_USB_DP
Changed lines of the file:
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@@
 			(effects (font (size 1.27 1.27)))
 		)
-		(pin "S3_USB_DM" bidirectional
+		(pin "S3_USB_N" bidirectional
 			(at 274.32 35.56 0)
 			(effects (font (size 1.27 1.27)))
 		)
-		(pin "S3_USB_DP" bidirectional
+		(pin "S3_USB_P" bidirectional
 			(at 274.32 36.83 0)
 			(effects (font (size 1.27 1.27)))
@@
 			(effects (font (size 1.27 1.27)))
 		)
-		(pin "S3_USB_DM" bidirectional
+		(pin "S3_USB_N" bidirectional
 			(at 274.32 538.48 0)
 			(effects (font (size 1.27 1.27)))
 		)
-		(pin "S3_USB_DP" bidirectional
+		(pin "S3_USB_P" bidirectional
 			(at 274.32 539.75 0)
 			(effects (font (size 1.27 1.27)))

Commit message: Canonicalize physical ground anchors
Other:
- sheet RF_03_MAIN_RAILS_DOMAIN_GATES ports: added none; removed SAFETY_GROUND
- sheet RF_20_CC1101_VOICE_TX ports: added none; removed SAFETY_GROUND
- sheet RF_30_U214_U219_M5_EXT ports: added none; removed SAFETY_GROUND
- sheet RF_40_INTERBOARD_M1 ports: added none; removed SAFETY_GROUND
- sheet RF_50_TX_SAFETY_EVIDENCE ports: added none; removed SAFETY_GROUND
