File: hardware/ecad/kicad/LESHY2-RF-R2/RF_20_CC1101_VOICE_TX.kicad_sch (KiCad schematic)
At the start: 146 parts, among them J5 GCT RFPC-SMA31-FN-175-A, J6 GCT RFPC-SMA31-FN-175-A, J7 GCT RFPC-SMA31-FN-175-A, Q5 Diodes Incorporated MMBT3904-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, U26 CC1101RGPR, U27 SN74LVC1G08DCKR, U28 TTM Technologies B0310J50100A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, U29 Nexperia 74LVC2G126DP,125, U30 Nexperia 74LVC126APW,118, U31 Texas Instruments TPS22919DCKR, U32 Nexperia 74LVC126APW,118, U33 Infineon BGS13SN8E6327XTSA1, U34 Infineon BGS13SN8E6327XTSA1, U35 Analog Devices AD8314ARMZ-REEL, U36 Analog Devices AD8314ARMZ-REEL, U37 Analog Devices AD8314ARMZ-REEL, U38 G-NiceRF SA818S-U, U39 Texas Instruments TMUX1136DGSR, U40 74LVC2G14GV,125, U41 TCA9534APWR, U42 Texas Instruments TPS564252DR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, U43 Texas Instruments TMUX1136DGSR, U44 Texas Instruments TMUX1136DGSR, U45 Texas Instruments TPS25974LRP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, U46 SN74LVC1G07DCKR, U47 Texas Instruments TPS22919DCKR, U48 Texas Instruments SN74LVC2G08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, U49 TPS3808G33DBVR, U50 G-NiceRF SA818S-V, Y2 Abracon ABM8-26.000MHZ-10-D-1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

Commit message: Complete current R2 schematic and sourcing revalidation
Parts:
- renumbered C101 to C106, C102 to C107, C103 to C108, C104 to C109, C105 to C110, C106 to C111, C107 to C112, C108 to C113, C109 to C114, C110 to C115, C111 to C116, C112 to C117, C113 to C118, C114 to C119, C115 to C120, C116 to C121, C117 to C122, C118 to C123, C119 to C124, C120 to C125, C121 to C126, C122 to C127, C123 to C128, C124 to C129, C125 to C130, C126 to C131, C127 to C132, C128 to C133, C129 to C134, C130 to C135, C131 to C136, C132 to C137, C133 to C138, C134 to C139, C135 to C140, C136 to C141, C137 to C142, C138 to C143, C139 to C144, C140 to C145, C141 to C146, C142 to C147, C143 to C148, C144 to C149, C145 to C150, C146 to C151, C147 to C152, C148 to C153, C149 to C154, L11 to L10, L12 to L11, L13 to L12, L14 to L13, L6 to L5, L7 to L6, L8 to L7, L9 to L8, L10 to L9, R99 to R100, R100 to R101, R101 to R102, R102 to R103, R103 to R104, R104 to R105, R105 to R106, R106 to R107, R107 to R108, R108 to R109, R109 to R110, R110 to R111, R111 to R112, R112 to R113, R113 to R114, R114 to R115, R115 to R116, R116 to R117, R117 to R118, R118 to R119, R119 to R120, R120 to R121, R121 to R122, R122 to R123, R123 to R124, R124 to R125, R125 to R126, R126 to R127, R127 to R128, R128 to R129, R129 to R130, R130 to R131, R131 to R132, R132 to R133, R133 to R134, R134 to R135, R135 to R136, R136 to R137, R137 to R138, R138 to R139, R139 to R140, R140 to R141, R141 to R142, R142 to R143, R143 to R144, R144 to R145, R145 to R146, R91 to R92, R92 to R93, R93 to R94, R94 to R95, R95 to R96, R96 to R97, R97 to R98, R98 to R99, U26 to U27, U27 to U28, U28 to U29, U29 to U30, U30 to U31, U31 to U32, U32 to U33, U33 to U34, U34 to U35, U35 to U36, U36 to U37, U37 to U38, U38 to U39, U39 to U40, U40 to U41, U41 to U42, U42 to U43, U43 to U44, U44 to U45, U45 to U46, U46 to U47, U47 to U48, U48 to U49, U49 to U50, U50 to U51

Commit message: Canonicalize physical ground anchors
Connections:
- net CC_RF_GROUND is gone; now on net POWER_GROUND: C106.2 (END_2), C107.2 (END_2), C108.2 (END_2), C109.2 (END_2), C110.2 (END_2), C111.2 (END_2), C112.2 (END_2), C114.2 (END_2), C115.2 (END_2), C116.2 (END_2), C117.2 (END_2), C121.2 (END_2), C122.2 (END_2), C123.2 (END_2), C124.2 (END_2), C126.2 (END_2), R106.2 (END_2), R110.2 (END_2), R111.2 (END_2), R112.2 (END_2), R113.2 (END_2), U27.16 (GND_16), U27.18 (DGUARD), U27.19 (GND_19), U27.21 (EPAD), U29.2 (GND), U30.4 (GND), U31.7 (GND), U33.7 (GND), U34.8 (GND), U35.8 (GND), Y2.2 (GND_2), Y2.4 (GND_4)
- net CC_SMA_RF_GROUND is gone; now on net POWER_GROUND: J5.2 (GROUND_TOP_LEFT), J5.3 (GROUND_TOP_RIGHT), J5.4 (GROUND_BOTTOM_LEFT), J5.5 (GROUND_BOTTOM_RIGHT)
- net SAFETY_GROUND is gone; now on net POWER_GROUND: C113.2 (END_2), C118.2 (END_2), C131.2 (END_2), C135.2 (END_2), C149.2 (END_2), C150.2 (END_2), C151.2 (END_2), C152.2 (END_2), R139.2 (END_2), U28.3 (GND), U36.5 (COMM), U37.5 (COMM), U38.5 (COMM), U41.2 (GND), U41.3 (2A), U49.4 (GND), U50.2 (GND)
- net VOICE_SMA_RF_GROUND is gone; now on net POWER_GROUND: J6.2 (GROUND_TOP_LEFT), J6.3 (GROUND_TOP_RIGHT), J6.4 (GROUND_BOTTOM_LEFT), J6.5 (GROUND_BOTTOM_RIGHT)
- net VOICE_V_SMA_RF_GROUND is gone; now on net POWER_GROUND: J7.2 (GROUND_TOP_LEFT), J7.3 (GROUND_TOP_RIGHT), J7.4 (GROUND_BOTTOM_LEFT), J7.5 (GROUND_BOTTOM_RIGHT)

Commit message: Correct exact RF lands and reopen native power prerequisites
Parts:
- U29: footprint Leshy2:B0310J50100AHF -> Leshy2_R2:B0310J50100AHF
Changed lines of the file:
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@@
 			(effects (font (size 1.27 1.27)))
 		)
-		(property "Footprint" "Leshy2:B0310J50100AHF"
+		(property "Footprint" "Leshy2_R2:B0310J50100AHF"
 			(at 238.76 407.67 0)
 			(show_name no)
