File: hardware/ecad/kicad/LESHY2-RF-R2/RF_02_PACK_SAFETY_AON.kicad_sch (KiCad schematic)
At the start: 65 parts, among them J2 Samtec FTSH-105-01-L-DV-K-P-TR, Q1 Diodes Incorporated DMN2056U-7, Q2 Diodes Incorporated 2N7002DW-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, Q3 Diodes Incorporated 2N7002DW-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, U10 Texas Instruments CSD87313DMS, U11 onsemi BAV70LT1G, U12 Diodes Incorporated BAT54-7-F, U6 TCA9803DGKR, U7 Texas Instruments MSPM0C1106S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, U8 Texas Instruments TPUL2G223BQ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, U9 Analog Devices MAX17320G20+T

Commit message: Correct second-cell polarity and fuse locality; reopen unproven thermal contact
Parts:
- BT1: footprint Leshy2:Keystone-1048P -> Leshy2_R2:Keystone-1048P-POLARITY-CORRECTED
Changed lines of the file:
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@@
 			(effects (font (size 1.27 1.27)))
 		)
-		(property "Footprint" "Leshy2:Keystone-1048P"
+		(property "Footprint" "Leshy2_R2:Keystone-1048P-POLARITY-CORRECTED"
 			(at 55.88 52.07 0)
 			(show_name no)
