File: hardware/ecad/kicad/LESHY2-RF-R2/RF_01_USB_PD_CHARGE.kicad_sch (KiCad schematic)
At the start: 52 parts, among them J1 JAE DX07S016JA1R1500, U1 Texas Instruments BQ25798RQMR, U2 onsemi CAT24C512WI-GT3, U3 Texas Instruments TPS25751DRE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, U4 Texas Instruments TVS2200DRVR, U5 Texas Instruments TPD4S201RUKR

Commit message: Bind H6 RF and USB routing geometry
Connections:
- net S3_USB_DM renamed S3_USB_N
- net S3_USB_DP renamed S3_USB_P
- net USB2_DM_CONNECTOR renamed USB2_CONNECTOR_N
- net USB2_DP_CONNECTOR renamed USB2_CONNECTOR_P
Changed lines of the file:
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@@
 		(effects (font (size 1.27 1.27)))
 	)
-	(label "USB2_DP_CONNECTOR"
+	(label "USB2_CONNECTOR_P"
 		(at 767.08 127.00 0)
 		(effects (font (size 1.27 1.27)))
 	)
-	(label "USB2_DM_CONNECTOR"
+	(label "USB2_CONNECTOR_N"
 		(at 767.08 129.54 0)
 		(effects (font (size 1.27 1.27)))
@@
 		(effects (font (size 1.27 1.27)) (justify right bottom))
 	)
-	(label "USB2_DP_CONNECTOR"
+	(label "USB2_CONNECTOR_P"
 		(at 807.72 124.46 180)
 		(effects (font (size 1.27 1.27)) (justify right bottom))
 	)
-	(label "USB2_DM_CONNECTOR"
+	(label "USB2_CONNECTOR_N"
 		(at 807.72 127.00 180)
 		(effects (font (size 1.27 1.27)) (justify right bottom))
@@
 		)
 	)
-	(label "USB2_DP_CONNECTOR"
+	(label "USB2_CONNECTOR_P"
 		(at 309.88 190.50 0)
 		(effects (font (size 1.27 1.27)))
 	)
-	(label "USB2_DM_CONNECTOR"
+	(label "USB2_CONNECTOR_N"
 		(at 309.88 193.04 0)
 		(effects (font (size 1.27 1.27)))
@@
 		(effects (font (size 1.27 1.27)) (justify right bottom))
 	)
-	(hierarchical_label "S3_USB_DM"
+	(hierarchical_label "S3_USB_N"
 		(shape bidirectional)
 		(at 350.52 195.58 180)
 		(effects (font (size 1.27 1.27)) (justify right bottom))
 	)
-	(hierarchical_label "S3_USB_DP"
+	(hierarchical_label "S3_USB_P"
 		(shape bidirectional)
 		(at 350.52 198.12 180)

Commit message: Audit native interfaces and correct connector poses and user silkscreen
Parts:
- J1: footprint Connector_USB:USB_C_Receptacle_JAE_DX07S016JA1R1500 -> Leshy2_R2:USB_C_Receptacle_JAE_DX07S016JA1R1500_EdgeSilk
Changed lines of the file:
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@@
 			(effects (font (size 1.27 1.27)))
 		)
-		(property "Footprint" "Connector_USB:USB_C_Receptacle_JAE_DX07S016JA1R1500"
+		(property "Footprint" "Leshy2_R2:USB_C_Receptacle_JAE_DX07S016JA1R1500_EdgeSilk"
 			(at 787.40 129.54 0)
 			(show_name no)

Commit message: Unify four USB-C ports on exact GCT and verify native preservation
Parts:
- J1: value JAE DX07S016JA1R1500 -> GCT USB4105-GF-A; footprint Leshy2_R2:USB_C_Receptacle_JAE_DX07S016JA1R1500_EdgeSilk -> Connector_USB:USB_C_Receptacle_GCT_USB4105-xx-A_16P_TopMnt_Horizontal; symbol Leshy2_R2:jae_dx07s016ja1r1500 -> Leshy2_R2:gct_usb4105_gf_a
Changed lines of the file:
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@@
 	)
 	(symbol
-		(lib_id "Leshy2_R2:jae_dx07s016ja1r1500")
+		(lib_id "Leshy2_R2:gct_usb4105_gf_a")
 		(at 787.40 129.54 0)
 		(unit 1)
@@
 			(effects (font (size 1.27 1.27)))
 		)
-		(property "Value" "JAE DX07S016JA1R1500"
+		(property "Value" "GCT USB4105-GF-A"
 			(at 787.40 143.51 0)
 			(show_name no)
@@
 			(effects (font (size 1.27 1.27)))
 		)
-		(property "Footprint" "Leshy2_R2:USB_C_Receptacle_JAE_DX07S016JA1R1500_EdgeSilk"
+		(property "Footprint" "Connector_USB:USB_C_Receptacle_GCT_USB4105-xx-A_16P_TopMnt_Horizontal"
 			(at 787.40 129.54 0)
 			(show_name no)
@@
 			(effects (font (size 1.27 1.27)))
 		)
-		(property "Description" "jae_dx07s016ja1r1500"
+		(property "Description" "gct_usb4105_gf_a"
 			(at 787.40 129.54 0)
 			(show_name no)
