File: hardware/ecad/kicad/LESHY2-UI-R2/UI_31_NRF24_X3_TX_EVIDENCE.kicad_sch (KiCad schematic)
At the start: 107 parts, among them J12 GCT RFPC-SMA31-FN-175-A, J13 Hirose U.FL-R-SMT-1(80), J14 GCT RFPC-SMA31-FN-175-A, J15 Hirose U.FL-R-SMT-1(80), J16 GCT RFPC-SMA31-FN-175-A, J17 Hirose U.FL-R-SMT-1(80), U32 Analog Devices AD8314ARMZ-REEL, U33 Analog Devices AD8314ARMZ-REEL, U34 Analog Devices AD8314ARMZ-REEL, U35 Ebyte E01-ML01SP4, U36 TTM Technologies DC2337J5010A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, U37 Nexperia 74LVC126APW,118, U38 Nexperia 74LVC2G126DP,125, U39 Ebyte E01-ML01SP4, U40 TTM Technologies DC2337J5010A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, U41 Nexperia 74LVC126APW,118, U42 Nexperia 74LVC2G126DP,125, U43 Ebyte E01-ML01SP4, U44 TTM Technologies DC2337J5010A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, U45 Nexperia 74LVC126APW,118, U46 Nexperia 74LVC2G126DP,125, U47 SN74LVC1G08DCKR, U48 Diodes Incorporated BAT54-7-F, U49 Texas Instruments TPS22919DCKR

Commit message: Canonicalize physical ground anchors
Connections:
- net NRF0_RF_GROUND is gone; now on net POWER_GROUND: C62.2 (END_2), C63.2 (END_2), J13.2 (SHELL), R147.2 (END_2), R149.2 (END_2), R158.2 (END_2), R161.2 (END_2), R162.2 (END_2), R163.2 (END_2), U35.10 (GND_10), U35.8 (GND), U35.9 (GND_9), U36.3 (GND_3), U36.4 (GND_4)
- net NRF0_SMA_RF_GROUND is gone; now on net POWER_GROUND: J12.2 (GROUND_TOP_LEFT), J12.3 (GROUND_TOP_RIGHT), J12.4 (GROUND_BOTTOM_LEFT), J12.5 (GROUND_BOTTOM_RIGHT)
- net NRF1_RF_GROUND is gone; now on net POWER_GROUND: C68.2 (END_2), C69.2 (END_2), J15.2 (SHELL), R167.2 (END_2), R169.2 (END_2), R178.2 (END_2), R181.2 (END_2), R182.2 (END_2), R183.2 (END_2), U39.10 (GND_10), U39.8 (GND), U39.9 (GND_9), U40.3 (GND_3), U40.4 (GND_4)
- net NRF1_SMA_RF_GROUND is gone; now on net POWER_GROUND: J14.2 (GROUND_TOP_LEFT), J14.3 (GROUND_TOP_RIGHT), J14.4 (GROUND_BOTTOM_LEFT), J14.5 (GROUND_BOTTOM_RIGHT)
- net NRF2_RF_GROUND is gone; now on net POWER_GROUND: C74.2 (END_2), C75.2 (END_2), J17.2 (SHELL), R187.2 (END_2), R189.2 (END_2), R198.2 (END_2), R201.2 (END_2), R202.2 (END_2), R203.2 (END_2), U43.10 (GND_10), U43.8 (GND), U43.9 (GND_9), U44.3 (GND_3), U44.4 (GND_4)
- net NRF2_SMA_RF_GROUND is gone; now on net POWER_GROUND: J16.2 (GROUND_TOP_LEFT), J16.3 (GROUND_TOP_RIGHT), J16.4 (GROUND_BOTTOM_LEFT), J16.5 (GROUND_BOTTOM_RIGHT)
- net SAFETY_GROUND is gone; now on net POWER_GROUND: C59.2 (END_2), C65.2 (END_2), C71.2 (END_2), C77.2 (END_2), C78.2 (END_2), R206.2 (END_2), U32.5 (COMM), U33.5 (COMM), U34.5 (COMM), U47.3 (GND)

Commit message: Correct exact RF lands and reopen native power prerequisites
Parts:
- U36, U40, U44: footprint Leshy2:DC2337J5010AHF -> Leshy2_R2:DC2337J5010AHF
Changed lines of the file:
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@@
 			(effects (font (size 1.27 1.27)))
 		)
-		(property "Footprint" "Leshy2:DC2337J5010AHF"
+		(property "Footprint" "Leshy2_R2:DC2337J5010AHF"
 			(at 878.84 300.99 0)
 			(show_name no)
@@
 			(effects (font (size 1.27 1.27)))
 		)
-		(property "Footprint" "Leshy2:DC2337J5010AHF"
+		(property "Footprint" "Leshy2_R2:DC2337J5010AHF"
 			(at 147.32 336.55 0)
 			(show_name no)
@@
 			(effects (font (size 1.27 1.27)))
 		)
-		(property "Footprint" "Leshy2:DC2337J5010AHF"
+		(property "Footprint" "Leshy2_R2:DC2337J5010AHF"
 			(at 513.08 336.55 0)
 			(show_name no)
